File: audio/CM4_docker.kicad_sch (KiCad schematic)
At the start: 0 parts

Commit message: .
.
Parts:
- added J6, J7: Conn_01x10, Connector_PinHeader_2.54mm:PinHeader_1x10_P2.54mm_Vertical, symbol Connector_Generic:Conn_01x10
Connections:
- net +5V: now also J6.1 (Pin_1), J6.2 (Pin_2)
- net GND: now also J6.10 (Pin_10), J6.4 (Pin_4), J6.6 (Pin_6), J6.8 (Pin_8), J7.1 (Pin_1), J7.10 (Pin_10), J7.2 (Pin_2), J7.3 (Pin_3), J7.4 (Pin_4), J7.5 (Pin_5), J7.6 (Pin_6), J7.8 (Pin_8)
- new net 3.3V: J6.3 (Pin_3)
- new net I2C1_SCL: J7.9 (Pin_9)
- new net I2C1_SDA: J7.7 (Pin_7)
- new net I2S_ADC: J6.7 (Pin_7)
- new net I2S_BCLK: J6.9 (Pin_9)
- new net I2S_LRCK: J6.5 (Pin_5)
Other:
- sheet CM4_LOW_SPEED ports: added 3.3V, GND, I2C1_SCL, I2C1_SDA, I2S_ADC, I2S_BCLK, I2S_LRCK; removed none

Commit message: .
.
Parts:
- added J10: Conn_01x10, Connector_PinHeader_2.54mm:PinHeader_1x10_P2.54mm_Vertical, symbol Connector_Generic:Conn_01x10
Connections:
- net +5V: now also J10.1 (Pin_1)
- net 3.3V: now also J10.3 (Pin_3), J10.4 (Pin_4)
- net GND: now also J10.2 (Pin_2)
- new net SD_CLK: J10.10 (Pin_10)
- new net SD_CMD: J10.9 (Pin_9)
- new net SD_DAT0: J10.8 (Pin_8)
- new net SD_DAT1: J10.7 (Pin_7)
- new net SD_DAT2: J10.6 (Pin_6)
- new net SD_DAT3: J10.5 (Pin_5)
Other:
- sheet CM4_LOW_SPEED ports: added SD_CLK, SD_CMD, SD_DAT0, SD_DAT1, SD_DAT2, SD_DAT3; removed none
Changed lines of the file:
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@@
 (kicad_sch (version 20211123) (generator eeschema)
   (paper "A4")
+  (wire (pts (xy 30.48 41.91) (xy 45.72 41.91))
+    (stroke (width 0) (type default) (color 0 0 0 0))
+  )
+  (wire (pts (xy 30.48 49.53) (xy 45.72 49.53))
+    (stroke (width 0) (type default) (color 0 0 0 0))
+  )
   (wire (pts (xy 165.1 72.39) (xy 177.8 72.39))
     (stroke (width 0) (type default) (color 0 0 0 0))
@@
     (stroke (width 0) (type default) (color 0 0 0 0))
   )
+  (wire (pts (xy 30.48 44.45) (xy 45.72 44.45))
+    (stroke (width 0) (type default) (color 0 0 0 0))
+  )
   (wire (pts (xy 119.38 66.04) (xy 133.35 66.04))
     (stroke (width 0) (type default) (color 0 0 0 0))
@@
     (stroke (width 0) (type default) (color 0 0 0 0))
   )
+  (wire (pts (xy 30.48 34.29) (xy 45.72 34.29))
+    (stroke (width 0) (type default) (color 0 0 0 0))
+  )
   (wire (pts (xy 72.39 88.9) (xy 87.63 88.9))
     (stroke (width 0) (type default) (color 0 0 0 0))
@@
     (stroke (width 0) (type default) (color 0 0 0 0))
   )
+  (wire (pts (xy 30.48 36.83) (xy 45.72 36.83))
+    (stroke (width 0) (type default) (color 0 0 0 0))
+  )
   (wire (pts (xy 165.1 64.77) (xy 177.8 64.77))
     (stroke (width 0) (type default) (color 0 0 0 0))
@@
     (stroke (width 0) (type default) (color 0 0 0 0))
   )
+  (wire (pts (xy 30.48 31.75) (xy 45.72 31.75))
+    (stroke (width 0) (type default) (color 0 0 0 0))
+  )
   (wire (pts (xy 30.48 99.06) (xy 45.72 99.06))
     (stroke (width 0) (type default) (color 0 0 0 0))
   )
+  (wire (pts (xy 30.48 46.99) (xy 45.72 46.99))
+    (stroke (width 0) (type default) (color 0 0 0 0))
+  )
   (wire (pts (xy 165.1 53.34) (xy 177.8 53.34))
     (stroke (width 0) (type default) (color 0 0 0 0))
@@
     (stroke (width 0) (type default) (color 0 0 0 0))
   )
+  (wire (pts (xy 30.48 39.37) (xy 45.72 39.37))
+    (stroke (width 0) (type default) (color 0 0 0 0))
+  )
   (wire (pts (xy 30.48 86.36) (xy 45.72 86.36))
     (stroke (width 0) (type default) (color 0 0 0 0))
   )
+  (wire (pts (xy 30.48 52.07) (xy 45.72 52.07))
+    (stroke (width 0) (type default) (color 0 0 0 0))
+  )
   (wire (pts (xy 119.38 63.5) (xy 133.35 63.5))
     (stroke (width 0) (type default) (color 0 0 0 0))
@@
     (stroke (width 0) (type default) (color 0 0 0 0))
   )
+  (wire (pts (xy 30.48 29.21) (xy 45.72 29.21))
+    (stroke (width 0) (type default) (color 0 0 0 0))
+  )
   (wire (pts (xy 30.48 121.92) (xy 45.72 121.92))
     (stroke (width 0) (type default) (color 0 0 0 0))
@@
     (effects (font (size 1.27 1.27)) (justify left bottom))
   )
-  (text "Connectors\n-------\nEthernet\nUSB 2.0" (at 90.17 48.26 0)
+  (text "Connectors\n-------\nEthernet\nUSB 2.0" (at 106.68 46.99 0)
     (effects (font (size 1.27 1.27)) (justify left bottom))
   )
@@
     (effects (font (size 1.27 1.27)) (justify left bottom))
   )
+  (label "SD_DAT1" (at 40.64 36.83 180)
+    (effects (font (size 1.27 1.27)) (justify right bottom))
+  )
   (label "GND" (at 34.29 78.74 0)
     (effects (font (size 1.27 1.27)) (justify left bottom))
   )
+  (label "+5V" (at 33.02 52.07 0)
+    (effects (font (size 1.27 1.27)) (justify left bottom))
+  )
+  (label "SD_DAT0" (at 40.64 34.29 180)
+    (effects (font (size 1.27 1.27)) (justify right bottom))
+  )
   (label "GND" (at 79.6172 118.11 0)
     (effects (font (size 1.27 1.27)) (justify left bottom))
@@
     (effects (font (size 1.27 1.27)) (justify left bottom))
   )
+  (label "SD_DAT2" (at 40.64 39.37 180)
+    (effects (font (size 1.27 1.27)) (justify right bottom))
+  )
   (label "+5V" (at 34.29 86.36 0)
     (effects (font (size 1.27 1.27)) (justify left bottom))
@@
     (effects (font (size 1.27 1.27)) (justify left bottom))
   )
+  (label "3.3V" (at 33.02 46.99 0)
+    (effects (font (size 1.27 1.27)) (justify left bottom))
+  )
   (label "I2C1_SCL" (at 76.2 77.47 0)
     (effects (font (size 1.27 1.27)) (justify left bottom))
@@
     (effects (font (size 1.27 1.27)) (justify left bottom))
   )
+  (label "3.3V" (at 33.02 44.45 0)
+    (effects (font (size 1.27 1.27)) (justify left bottom))
+  )
   (label "GND" (at 34.29 63.5 0)
     (effects (font (size 1.27 1.27)) (justify left bottom))
@@
     (effects (font (size 1.27 1.27)) (justify left bottom))
   )
+  (label "GND" (at 32.8475 49.53 0)
+    (effects (font (size 1.27 1.27)) (justify left bottom))
+  )
   (label "GND" (at 34.29 121.92 0)
     (effects (font (size 1.27 1.27)) (justify left bottom))
@@
     (effects (font (size 1.27 1.27)) (justify left bottom))
   )
+  (label "SD_DAT3" (at 40.64 41.91 180)
+    (effects (font (size 1.27 1.27)) (justify right bottom))
+  )
   (label "3.3V" (at 34.29 81.28 0)
     (effects (font (size 1.27 1.27)) (justify left bottom))
@@
   (label "I2S_BCLK" (at 34.29 66.04 0)
     (effects (font (size 1.27 1.27)) (justify left bottom))
+  )
+  (label "SD_CLK" (at 40.64 29.21 180)
+    (effects (font (size 1.27 1.27)) (justify right bottom))
+  )
+  (label "SD_CMD" (at 40.64 31.75 180)
+    (effects (font (size 1.27 1.27)) (justify right bottom))
   )
   (hierarchical_label "I2C1_SDA" (shape output) (at 72.39 80.01 180)
@@
     (pin "9")
   )
-  (symbol (lib_id "Connector_Generic:Conn_01x10") (at 25.4 111.76 180) (unit 1)
+  (symbol (lib_id "Connector_Generic:Conn_01x10") (at 25.4 41.91 180) (unit 1)
     (in_bom yes) (on_board yes) (fields_autoplaced)
-    (property "Reference" "J7" (id 0) (at 25.4 92.71 0))
-    (property "Value" "Conn_01x10" (id 1) (at 25.4 95.25 0))
-    (property "Footprint" "Connector_PinHeader_2.54mm:PinHeader_1x10_P2.54mm_Vertical" (id 2) (at 25.4 111.76 0)
-      (effects (font (size 1.27 1.27)) hide)
-    )
-    (property "Datasheet" "~" (id 3) (at 25.4 111.76 0)
+    (property "Reference" "J10" (id 0) (at 25.4 22.86 0))
+    (property "Value" "Conn_01x10" (id 1) (at 25.4 25.4 0))
+    (property "Footprint" "Connector_PinHeader_2.54mm:PinHeader_1x10_P2.54mm_Vertical" (id 2) (at 25.4 41.91 0)
+      (effects (font (size 1.27 1.27)) hide)
+    )
+    (property "Datasheet" "~" (id 3) (at 25.4 41.91 0)
       (effects (font (size 1.27 1.27)) hide)
     )
@@
     (pin "9")
   )
+  (symbol (lib_id "Connector_Generic:Conn_01x10") (at 25.4 111.76 180) (unit 1)
+    (in_bom yes) (on_board yes) (fields_autoplaced)
+    (property "Reference" "J7" (id 0) (at 25.4 92.71 0))
+    (property "Value" "Conn_01x10" (id 1) (at 25.4 95.25 0))
+    (property "Footprint" "Connector_PinHeader_2.54mm:PinHeader_1x10_P2.54mm_Vertical" (id 2) (at 25.4 111.76 0)
+      (effects (font (size 1.27 1.27)) hide)
+    )
+    (property "Datasheet" "~" (id 3) (at 25.4 111.76 0)
+      (effects (font (size 1.27 1.27)) hide)
+    )
+    (pin "1")
+    (pin "10")
+    (pin "2")
+    (pin "3")
+    (pin "4")
+    (pin "5")
+    (pin "6")
+    (pin "7")
+    (pin "8")
+    (pin "9")
+  )
   (sheet (at 177.8 38.1) (size 29.21 57.15)
     (stroke (width 0.152) (type solid) (color 132 0 132 1))
@@
       (effects (font (size 1.27 1.27)) (justify left))
     )
+    (pin "SD_CLK" input (at 87.63 49.53 180)
+      (effects (font (size 1.27 1.27)) (justify left))
+    )
+    (pin "SD_DAT3" input (at 87.63 46.99 180)
+      (effects (font (size 1.27 1.27)) (justify left))
+    )
+    (pin "SD_DAT0" input (at 87.63 44.45 180)
+      (effects (font (size 1.27 1.27)) (justify left))
+    )
+    (pin "SD_DAT1" input (at 87.63 41.91 180)
+      (effects (font (size 1.27 1.27)) (justify left))
+    )
+    (pin "SD_DAT2" input (at 87.63 52.07 180)
+      (effects (font (size 1.27 1.27)) (justify left))
+    )
+    (pin "SD_CMD" input (at 87.63 54.61 180)
+      (effects (font (size 1.27 1.27)) (justify left))
+    )

Commit message: .
.
Changed lines of the file:
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@@
+    (stroke (width 0) (type default) (color 0 0 0 0))
+  )
+  (wire (pts (xy 72.39 45.72) (xy 87.63 45.72))
     (stroke (width 0) (type default) (color 0 0 0 0))
   )
@@
     (stroke (width 0) (type default) (color 0 0 0 0))
   )
+  (wire (pts (xy 72.39 40.64) (xy 87.63 40.64))
+    (stroke (width 0) (type default) (color 0 0 0 0))
+  )
   (wire (pts (xy 30.48 36.83) (xy 45.72 36.83))
     (stroke (width 0) (type default) (color 0 0 0 0))
@@
     (stroke (width 0) (type default) (color 0 0 0 0))
   )
+  (wire (pts (xy 72.39 50.8) (xy 87.63 50.8))
+    (stroke (width 0) (type default) (color 0 0 0 0))
+  )
   (wire (pts (xy 30.48 99.06) (xy 45.72 99.06))
     (stroke (width 0) (type default) (color 0 0 0 0))
@@
     (stroke (width 0) (type default) (color 0 0 0 0))
   )
+  (wire (pts (xy 72.39 43.18) (xy 87.63 43.18))
+    (stroke (width 0) (type default) (color 0 0 0 0))
+  )
+  (wire (pts (xy 72.39 53.34) (xy 87.63 53.34))
+    (stroke (width 0) (type default) (color 0 0 0 0))
+  )
   (wire (pts (xy 119.38 63.5) (xy 133.35 63.5))
     (stroke (width 0) (type default) (color 0 0 0 0))
@@
     (stroke (width 0) (type default) (color 0 0 0 0))
   )
+  (wire (pts (xy 72.39 48.26) (xy 87.63 48.26))
+    (stroke (width 0) (type default) (color 0 0 0 0))
+  )
   (wire (pts (xy 30.48 119.38) (xy 45.72 119.38))
     (stroke (width 0) (type default) (color 0 0 0 0))
@@
     (effects (font (size 1.27 1.27)) (justify left bottom))
   )
+  (label "SD_DAT3" (at 82.55 53.34 180)
+    (effects (font (size 1.27 1.27)) (justify right bottom))
+  )
   (label "I2C1_SCL" (at 34.29 101.6 0)
     (effects (font (size 1.27 1.27)) (justify left bottom))
@@
     (effects (font (size 1.27 1.27)) (justify left bottom))
   )
+  (label "SD_CMD" (at 82.55 43.18 180)
+    (effects (font (size 1.27 1.27)) (justify right bottom))
+  )
   (label "+5V" (at 33.02 52.07 0)
     (effects (font (size 1.27 1.27)) (justify left bottom))
@@
     (effects (font (size 1.27 1.27)) (justify left bottom))
   )
+  (label "SD_DAT0" (at 82.55 45.72 180)
+    (effects (font (size 1.27 1.27)) (justify right bottom))
+  )
+  (label "SD_DAT1" (at 82.55 48.26 180)
+    (effects (font (size 1.27 1.27)) (justify right bottom))
+  )
   (label "I2S_LRCK" (at 34.29 76.2 0)
     (effects (font (size 1.27 1.27)) (justify left bottom))
@@
     (effects (font (size 1.27 1.27)) (justify left bottom))
   )
+  (label "SD_DAT2" (at 82.55 50.8 180)
+    (effects (font (size 1.27 1.27)) (justify right bottom))
+  )
   (label "3.3V" (at 76.2 86.36 0)
     (effects (font (size 1.27 1.27)) (justify left bottom))
@@
   (label "GND" (at 34.29 68.58 0)
     (effects (font (size 1.27 1.27)) (justify left bottom))
+  )
+  (label "SD_CLK" (at 82.55 40.64 180)
+    (effects (font (size 1.27 1.27)) (justify right bottom))
   )
   (label "I2S_BCLK" (at 34.29 66.04 0)
@@
       (effects (font (size 1.27 1.27)) (justify left))
     )
-    (pin "SD_CLK" input (at 87.63 49.53 180)
-      (effects (font (size 1.27 1.27)) (justify left))
-    )
-    (pin "SD_DAT3" input (at 87.63 46.99 180)
-      (effects (font (size 1.27 1.27)) (justify left))
-    )
-    (pin "SD_DAT0" input (at 87.63 44.45 180)
-      (effects (font (size 1.27 1.27)) (justify left))
-    )
-    (pin "SD_DAT1" input (at 87.63 41.91 180)
-      (effects (font (size 1.27 1.27)) (justify left))
-    )
-    (pin "SD_DAT2" input (at 87.63 52.07 180)
-      (effects (font (size 1.27 1.27)) (justify left))
-    )
-    (pin "SD_CMD" input (at 87.63 54.61 180)
-      (effects (font (size 1.27 1.27)) (justify left))
-    )
+    (pin "SD_CLK" input (at 87.63 40.64 180)
+      (effects (font (size 1.27 1.27)) (justify left))
+    )
+    (pin "SD_DAT3" input (at 87.63 53.34 180)
+      (effects (font (size 1.27 1.27)) (justify left))
+    )
+    (pin "SD_DAT0" input (at 87.63 45.72 180)
+      (effects (font (size 1.27 1.27)) (justify left))
+    )
+    (pin "SD_DAT1" input (at 87.63 48.26 180)
+      (effects (font (size 1.27 1.27)) (justify left))
+    )
+    (pin "SD_DAT2" input (at 87.63 50.8 180)
+      (effects (font (size 1.27 1.27)) (justify left))
+    )
+    (pin "SD_CMD" input (at 87.63 43.18 180)
+      (effects (font (size 1.27 1.27)) (justify left))
+    )

Commit message: .
.
Changed lines of the file:
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@@
     (effects (font (size 1.27 1.27)) (justify left bottom))
   )
-  (label "SD_CMD" (at 82.55 43.18 180)
+  (label "SD_CMD" (at 81.915 43.18 180)
     (effects (font (size 1.27 1.27)) (justify right bottom))
   )
@@
     (effects (font (size 1.27 1.27)) (justify left bottom))
   )
-  (label "SD_CLK" (at 82.55 40.64 180)
+  (label "SD_CLK" (at 81.915 40.64 180)
     (effects (font (size 1.27 1.27)) (justify right bottom))
   )
@@
     (effects (font (size 1.27 1.27)) (justify left bottom))
   )
-  (label "SD_CLK" (at 40.64 29.21 180)
+  (label "SD_CLK" (at 39.37 29.21 180)
     (effects (font (size 1.27 1.27)) (justify right bottom))
   )
-  (label "SD_CMD" (at 40.64 31.75 180)
+  (label "SD_CMD" (at 40.005 31.75 180)
     (effects (font (size 1.27 1.27)) (justify right bottom))
   )
-  (hierarchical_label "I2C1_SDA" (shape output) (at 72.39 80.01 180)
-    (effects (font (size 1.27 1.27)) (justify right))
+  (hierarchical_label "I2S_LRCK" (shape bidirectional) (at 45.72 76.2 0)
+    (effects (font (size 1.27 1.27)) (justify left))
   )
-  (hierarchical_label "I2S_LRCK" (shape bidirectional) (at 72.39 60.96 180)
-    (effects (font (size 1.27 1.27)) (justify right))
+  (hierarchical_label "+5V" (shape output) (at 45.72 86.36 0)
+    (effects (font (size 1.27 1.27)) (justify left))
   )
-  (hierarchical_label "I2S_ADC" (shape input) (at 72.39 66.04 180)
-    (effects (font (size 1.27 1.27)) (justify right))
+  (hierarchical_label "I2C1_SDA" (shape output) (at 45.72 106.68 0)
+    (effects (font (size 1.27 1.27)) (justify left))
   )
-  (hierarchical_label "3.3V" (shape output) (at 72.39 86.36 180)
-    (effects (font (size 1.27 1.27)) (justify right))
+  (hierarchical_label "I2S_ADC" (shape input) (at 45.72 71.12 0)
+    (effects (font (size 1.27 1.27)) (justify left))
   )
-  (hierarchical_label "+5V" (shape output) (at 74.93 121.92 180)
-    (effects (font (size 1.27 1.27)) (justify right))
+  (hierarchical_label "I2S_BCLK" (shape bidirectional) (at 45.72 66.04 0)
+    (effects (font (size 1.27 1.27)) (justify left))
   )
-  (hierarchical_label "I2C1_SCL" (shape output) (at 72.39 77.47 180)
-    (effects (font (size 1.27 1.27)) (justify right))
+  (hierarchical_label "3.3V" (shape output) (at 45.72 81.28 0)
+    (effects (font (size 1.27 1.27)) (justify left))
   )
-  (hierarchical_label "I2S_BCLK" (shape bidirectional) (at 72.39 63.5 180)
-    (effects (font (size 1.27 1.27)) (justify right))
+  (hierarchical_label "I2C1_SCL" (shape output) (at 45.72 101.6 0)
+    (effects (font (size 1.27 1.27)) (justify left))
   )
-  (hierarchical_label "GND" (shape output) (at 74.93 118.11 180)
-    (effects (font (size 1.27 1.27)) (justify right))
+  (hierarchical_label "GND" (shape output) (at 45.72 78.74 0)
+    (effects (font (size 1.27 1.27)) (justify left))
   )
   (symbol (lib_id "Connector_Generic:Conn_01x10") (at 25.4 76.2 180) (unit 1)

Commit message: .
.
Connections:
- net SD_CLK: now also J10.6 (Pin_6); no longer J10.10 (Pin_10)
- net SD_CMD: now also J10.5 (Pin_5); no longer J10.9 (Pin_9)
- net SD_DAT0: now also J10.10 (Pin_10); no longer J10.8 (Pin_8)
- net SD_DAT1: now also J10.9 (Pin_9); no longer J10.7 (Pin_7)
- net SD_DAT2: now also J10.8 (Pin_8); no longer J10.6 (Pin_6)
- net SD_DAT3: now also J10.7 (Pin_7); no longer J10.5 (Pin_5)
Changed lines of the file:
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@@
     (effects (font (size 1.27 1.27)) (justify left bottom))
   )
-  (label "SD_DAT1" (at 40.64 36.83 180)
+  (label "SD_DAT1" (at 41.91 31.75 180)
     (effects (font (size 1.27 1.27)) (justify right bottom))
   )
@@
     (effects (font (size 1.27 1.27)) (justify left bottom))
   )
-  (label "SD_DAT0" (at 40.64 34.29 180)
+  (label "SD_DAT0" (at 41.91 29.21 180)
     (effects (font (size 1.27 1.27)) (justify right bottom))
   )
@@
     (effects (font (size 1.27 1.27)) (justify left bottom))
   )
-  (label "SD_DAT2" (at 40.64 39.37 180)
+  (label "SD_DAT2" (at 41.91 34.29 180)
     (effects (font (size 1.27 1.27)) (justify right bottom))
   )
@@
     (effects (font (size 1.27 1.27)) (justify left bottom))
   )
-  (label "SD_DAT3" (at 40.64 41.91 180)
+  (label "SD_DAT3" (at 41.91 36.83 180)
     (effects (font (size 1.27 1.27)) (justify right bottom))
   )
@@
     (effects (font (size 1.27 1.27)) (justify left bottom))
   )
-  (label "SD_CLK" (at 39.37 29.21 180)
+  (label "SD_CLK" (at 40.64 39.37 180)
     (effects (font (size 1.27 1.27)) (justify right bottom))
   )
-  (label "SD_CMD" (at 40.005 31.75 180)
+  (label "SD_CMD" (at 40.64 41.91 180)
     (effects (font (size 1.27 1.27)) (justify right bottom))
   )

Commit message: .
.
Changed lines of the file:
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@@
     (effects (font (size 1.27 1.27)) (justify right bottom))
   )
-  (label "GND" (at 79.6172 118.11 0)
+  (label "GND" (at 78.74 121.92 0)
     (effects (font (size 1.27 1.27)) (justify left bottom))
   )
@@
     (effects (font (size 1.27 1.27)) (justify left bottom))
   )
-  (label "+5V" (at 78.74 121.92 0)
+  (label "+5V" (at 78.74 118.11 0)
     (effects (font (size 1.27 1.27)) (justify left bottom))
   )

Commit message: .
.
Connections:
- net +5V: now also J10.2 (Pin_2), J7.1 (Pin_1), J7.2 (Pin_2), J7.3 (Pin_3), J7.4 (Pin_4); no longer J6.1 (Pin_1), J6.2 (Pin_2)
- net 3.3V: now also J7.10 (Pin_10); no longer J10.3 (Pin_3), J6.3 (Pin_3)
- net GND: now also J10.3 (Pin_3), J6.3 (Pin_3); no longer J10.2 (Pin_2), J7.1 (Pin_1), J7.10 (Pin_10), J7.2 (Pin_2), J7.3 (Pin_3), J7.4 (Pin_4)
- new net USB_DEBUG_N: J6.1 (Pin_1)
- new net USB_DEBUG_P: J6.2 (Pin_2)
Changed lines of the file:
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@@
-    (effects (font (size 1.27 1.27)) (justify left bottom))
-  )
-  (label "GND" (at 34.29 119.38 0)
     (effects (font (size 1.27 1.27)) (justify left bottom))
   )
@@
     (effects (font (size 1.27 1.27)) (justify left bottom))
   )
-  (label "GND" (at 34.29 99.06 0)
+  (label "USB_DEBUG_P" (at 119.38 63.5 0)
     (effects (font (size 1.27 1.27)) (justify left bottom))
   )
@@
     (effects (font (size 1.27 1.27)) (justify right bottom))
   )
+  (label "+5V" (at 33.02 49.53 0)
+    (effects (font (size 1.27 1.27)) (justify left bottom))
+  )
   (label "I2C1_SCL" (at 34.29 101.6 0)
     (effects (font (size 1.27 1.27)) (justify left bottom))
   )
   (label "I2S_BCLK" (at 76.2 63.5 0)
+    (effects (font (size 1.27 1.27)) (justify left bottom))
+  )
+  (label "+5V" (at 34.29 114.3 0)
     (effects (font (size 1.27 1.27)) (justify left bottom))
   )
@@
     (effects (font (size 1.27 1.27)) (justify left bottom))
   )
-  (label "+5V" (at 34.29 83.82 0)
+  (label "+5V" (at 34.29 116.84 0)
+    (effects (font (size 1.27 1.27)) (justify left bottom))
+  )
+  (label "+5V" (at 34.29 119.38 0)
     (effects (font (size 1.27 1.27)) (justify left bottom))
   )
@@
     (effects (font (size 1.27 1.27)) (justify right bottom))
   )
+  (label "GND" (at 34.29 81.28 0)
+    (effects (font (size 1.27 1.27)) (justify left bottom))
+  )
   (label "I2S_LRCK" (at 34.29 76.2 0)
     (effects (font (size 1.27 1.27)) (justify left bottom))
@@
     (effects (font (size 1.27 1.27)) (justify right bottom))
   )
-  (label "+5V" (at 34.29 86.36 0)
+  (label "+5V" (at 34.29 121.92 0)
     (effects (font (size 1.27 1.27)) (justify left bottom))
   )
   (label "GND" (at 34.29 111.76 0)
-    (effects (font (size 1.27 1.27)) (justify left bottom))
-  )
-  (label "3.3V" (at 33.02 46.99 0)
     (effects (font (size 1.27 1.27)) (justify left bottom))
   )
@@
     (effects (font (size 1.27 1.27)) (justify left bottom))
   )
-  (label "GND" (at 32.8475 49.53 0)
+  (label "USB_DEBUG_N" (at 31.75 86.36 0)
     (effects (font (size 1.27 1.27)) (justify left bottom))
   )
-  (label "GND" (at 34.29 121.92 0)
+  (label "GND" (at 33.02 46.99 0)
     (effects (font (size 1.27 1.27)) (justify left bottom))
   )
@@
     (effects (font (size 1.27 1.27)) (justify left bottom))
   )
-  (label "GND" (at 34.29 116.84 0)
-    (effects (font (size 1.27 1.27)) (justify left bottom))
-  )
-  (label "GND" (at 34.29 114.3 0)
-    (effects (font (size 1.27 1.27)) (justify left bottom))
-  )
   (label "SD_DAT3" (at 41.91 36.83 180)
     (effects (font (size 1.27 1.27)) (justify right bottom))
-  )
-  (label "3.3V" (at 34.29 81.28 0)
-    (effects (font (size 1.27 1.27)) (justify left bottom))
   )
   (label "GND" (at 34.29 68.58 0)
@@
     (effects (font (size 1.27 1.27)) (justify right bottom))
   )
+  (label "USB_DEBUG_N" (at 119.38 60.96 0)
+    (effects (font (size 1.27 1.27)) (justify left bottom))
+  )
   (label "I2S_BCLK" (at 34.29 66.04 0)
     (effects (font (size 1.27 1.27)) (justify left bottom))
@@
   (label "SD_CLK" (at 40.64 39.37 180)
     (effects (font (size 1.27 1.27)) (justify right bottom))
+  )
+  (label "USB_DEBUG_P" (at 31.75 83.82 0)
+    (effects (font (size 1.27 1.27)) (justify left bottom))
+  )
+  (label "3.3V" (at 34.29 99.06 0)
+    (effects (font (size 1.27 1.27)) (justify left bottom))
   )
   (label "SD_CMD" (at 40.64 41.91 180)
@@
     (effects (font (size 1.27 1.27)) (justify left))
   )
-  (hierarchical_label "+5V" (shape output) (at 45.72 86.36 0)
+  (hierarchical_label "I2C1_SDA" (shape output) (at 45.72 106.68 0)
     (effects (font (size 1.27 1.27)) (justify left))
   )
-  (hierarchical_label "I2C1_SDA" (shape output) (at 45.72 106.68 0)
+  (hierarchical_label "3.3V" (shape output) (at 45.72 99.06 0)
     (effects (font (size 1.27 1.27)) (justify left))
   )
@@
     (effects (font (size 1.27 1.27)) (justify left))
   )
-  (hierarchical_label "3.3V" (shape output) (at 45.72 81.28 0)
+  (hierarchical_label "I2C1_SCL" (shape output) (at 45.72 101.6 0)
     (effects (font (size 1.27 1.27)) (justify left))
   )
-  (hierarchical_label "I2C1_SCL" (shape output) (at 45.72 101.6 0)
+  (hierarchical_label "+5V" (shape output) (at 45.72 121.92 0)
     (effects (font (size 1.27 1.27)) (justify left))
   )
@@
     (effects (font (size 1.27 1.27)) (justify left))
   )
+  (hierarchical_label "+5V" (shape output) (at 45.72 119.38 0)
+    (effects (font (size 1.27 1.27)) (justify left))
+  )
