File: audio/CM4_docker.kicad_sch (KiCad schematic)
At the start: 3 parts, among them J10 Conn_01x10, J6 Conn_01x10, J7 Conn_01x10

Commit message: .
.
Connections:
- net +5V: now also J6.3 (Pin_3); no longer J7.1 (Pin_1)
- net 3.3V: now also J7.1 (Pin_1)
- net GND: no longer J6.3 (Pin_3)
- net I2C1_SCL: now also J7.7 (Pin_7); no longer J7.9 (Pin_9)
- net I2C1_SDA: now also J7.9 (Pin_9); no longer J7.7 (Pin_7)
Changed lines of the file:
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@@
     (effects (font (size 1.27 1.27)) (justify left bottom))
   )
-  (label "I2C1_SCL" (at 34.29 101.6 0)
+  (label "I2C1_SCL" (at 34.29 106.68 0)
     (effects (font (size 1.27 1.27)) (justify left bottom))
   )
@@
     (effects (font (size 1.27 1.27)) (justify right bottom))
   )
+  (label "+5V" (at 34.29 81.28 0)
+    (effects (font (size 1.27 1.27)) (justify left bottom))
+  )
   (label "GND" (at 34.29 109.22 0)
     (effects (font (size 1.27 1.27)) (justify left bottom))
   )
-  (label "I2C1_SDA" (at 34.29 106.68 0)
+  (label "I2C1_SDA" (at 34.29 101.6 0)
     (effects (font (size 1.27 1.27)) (justify left bottom))
   )
@@
     (effects (font (size 1.27 1.27)) (justify right bottom))
   )
-  (label "GND" (at 34.29 81.28 0)
-    (effects (font (size 1.27 1.27)) (justify left bottom))
-  )
   (label "I2S_LRCK" (at 34.29 76.2 0)
     (effects (font (size 1.27 1.27)) (justify left bottom))
@@
     (effects (font (size 1.27 1.27)) (justify right bottom))
   )
-  (label "+5V" (at 34.29 121.92 0)
+  (label "3.3V" (at 34.29 121.92 0)
     (effects (font (size 1.27 1.27)) (justify left bottom))
   )
@@
     (effects (font (size 1.27 1.27)) (justify left))
   )
-  (hierarchical_label "I2C1_SDA" (shape output) (at 45.72 106.68 0)
-    (effects (font (size 1.27 1.27)) (justify left))
-  )
   (hierarchical_label "3.3V" (shape output) (at 45.72 99.06 0)
     (effects (font (size 1.27 1.27)) (justify left))
@@
     (effects (font (size 1.27 1.27)) (justify left))
   )
-  (hierarchical_label "I2C1_SCL" (shape output) (at 45.72 101.6 0)
-    (effects (font (size 1.27 1.27)) (justify left))
-  )
-  (hierarchical_label "+5V" (shape output) (at 45.72 121.92 0)
+  (hierarchical_label "I2C1_SDA" (shape output) (at 45.72 101.6 0)
     (effects (font (size 1.27 1.27)) (justify left))
   )
@@
     (effects (font (size 1.27 1.27)) (justify left))
   )
+  (hierarchical_label "I2C1_SCL" (shape output) (at 45.72 106.68 0)
+    (effects (font (size 1.27 1.27)) (justify left))
+  )
+  (hierarchical_label "3.3V" (shape output) (at 45.72 121.92 0)
+    (effects (font (size 1.27 1.27)) (justify left))
+  )
