File: audio/CM4_docker.kicad_sch (KiCad schematic)
At the start: 3 parts, among them J10 Conn_01x10, J6 Conn_01x10, J7 Conn_01x10

Commit message: .
.
Connections:
- net +5V: now also J6.4 (Pin_4)
- net 3.3V: now also J6.10 (Pin_10)
- net GND: no longer J6.10 (Pin_10), J6.4 (Pin_4)
Changed lines of the file:
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@@
+    (effects (font (size 1.27 1.27)) (justify left bottom))
+  )
+  (label "3.3V" (at 34.29 63.5 0)
     (effects (font (size 1.27 1.27)) (justify left bottom))
   )
@@
   (label "SD_DAT1" (at 41.91 31.75 180)
     (effects (font (size 1.27 1.27)) (justify right bottom))
-  )
-  (label "GND" (at 34.29 78.74 0)
-    (effects (font (size 1.27 1.27)) (justify left bottom))
   )
   (label "SD_CMD" (at 81.915 43.18 180)
@@
     (effects (font (size 1.27 1.27)) (justify left bottom))
   )
+  (label "+5V" (at 34.29 78.74 0)
+    (effects (font (size 1.27 1.27)) (justify left bottom))
+  )
   (label "I2C1_SCL" (at 76.2 77.47 0)
     (effects (font (size 1.27 1.27)) (justify left bottom))
@@
   )
   (label "3.3V" (at 33.02 44.45 0)
-    (effects (font (size 1.27 1.27)) (justify left bottom))
-  )
-  (label "GND" (at 34.29 63.5 0)
     (effects (font (size 1.27 1.27)) (justify left bottom))
   )
@@
     (effects (font (size 1.27 1.27)) (justify left))
   )
+  (hierarchical_label "3.3V" (shape output) (at 45.72 63.5 0)
+    (effects (font (size 1.27 1.27)) (justify left))
+  )
   (hierarchical_label "3.3V" (shape output) (at 45.72 99.06 0)
     (effects (font (size 1.27 1.27)) (justify left))
@@
     (effects (font (size 1.27 1.27)) (justify left))
   )
-  (hierarchical_label "GND" (shape output) (at 45.72 78.74 0)
-    (effects (font (size 1.27 1.27)) (justify left))
-  )
   (hierarchical_label "I2C1_SCL" (shape output) (at 45.72 106.68 0)
     (effects (font (size 1.27 1.27)) (justify left))
   )
+  (hierarchical_label "+5V" (shape output) (at 45.72 78.74 0)
+    (effects (font (size 1.27 1.27)) (justify left))
+  )

Commit message: .
.
Connections:
- net +5V: no longer J7.2 (Pin_2), J7.3 (Pin_3), J7.4 (Pin_4)
- net 3.3V: no longer J7.1 (Pin_1)
- net GND renamed GND_I2C
- net GND_I2C: now also J7.1 (Pin_1), J7.2 (Pin_2), J7.3 (Pin_3), J7.4 (Pin_4); no longer J6.8 (Pin_8)
- new net nRPIBOOT: J6.8 (Pin_8)
Other:
- sheet CM4_LOW_SPEED ports: added +5V, nRPIBOOT; removed none

Commit message: .
.
Connections:
- net +5V: now also J7.1 (Pin_1), J7.2 (Pin_2), J7.3 (Pin_3), J7.4 (Pin_4); no longer J6.4 (Pin_4)
- net GND_I2C: now also J6.10 (Pin_10), J6.4 (Pin_4), J7.10 (Pin_10); no longer J6.6 (Pin_6), J7.1 (Pin_1), J7.2 (Pin_2), J7.3 (Pin_3), J7.4 (Pin_4)
- removed net 3.3V: J10.4 (Pin_4), J6.10 (Pin_10), J7.10 (Pin_10)
- new net 3.3V_I2C: J10.4 (Pin_4)
- new net GLOBAL_EN: J6.6 (Pin_6)
Other:
- sheet CM4_LOW_SPEED ports: added GLOBAL_EN, nEXTRST; removed none
Changed lines of the file:
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@@
+    (stroke (width 0) (type default) (color 0 0 0 0))
+  )
+  (wire (pts (xy 119.38 53.34) (xy 129.54 53.34))
     (stroke (width 0) (type default) (color 0 0 0 0))
   )
@@
     (stroke (width 0) (type default) (color 0 0 0 0))
   )
+  (wire (pts (xy 129.54 50.8) (xy 119.38 50.8))
+    (stroke (width 0) (type default) (color 0 0 0 0))
+  )
   (wire (pts (xy 30.48 121.92) (xy 45.72 121.92))
     (stroke (width 0) (type default) (color 0 0 0 0))
@@
     (stroke (width 0) (type default) (color 0 0 0 0))
   )
+  (wire (pts (xy 207.01 57.785) (xy 222.25 57.785))
+    (stroke (width 0) (type default) (color 0 0 0 0))
+  )
   (wire (pts (xy 124.46 87.63) (xy 133.35 87.63))
     (stroke (width 0) (type default) (color 0 0 0 0))
@@
     (effects (font (size 1.27 1.27)) (justify left bottom))
   )
-  (label "GND" (at 34.29 73.66 0)
+  (label "GND" (at 34.29 78.74 0)
     (effects (font (size 1.27 1.27)) (justify left bottom))
   )
@@
     (effects (font (size 1.27 1.27)) (justify left bottom))
   )
+  (label "+5V" (at 34.29 114.3 0)
+    (effects (font (size 1.27 1.27)) (justify left bottom))
+  )
   (label "USB_DEBUG_P" (at 119.38 63.5 0)
     (effects (font (size 1.27 1.27)) (justify left bottom))
@@
     (effects (font (size 1.27 1.27)) (justify left bottom))
   )
-  (label "3.3V" (at 34.29 63.5 0)
-    (effects (font (size 1.27 1.27)) (justify left bottom))
-  )
-  (label "GND_I2C" (at 34.29 114.3 0)
-    (effects (font (size 1.27 1.27)) (justify left bottom))
-  )
   (label "I2S_BCLK" (at 76.2 63.5 0)
     (effects (font (size 1.27 1.27)) (justify left bottom))
@@
     (effects (font (size 1.27 1.27)) (justify right bottom))
   )
-  (label "GND_I2C" (at 34.29 116.84 0)
+  (label "GLOBAL_EN" (at 120.65 53.34 0)
     (effects (font (size 1.27 1.27)) (justify left bottom))
   )
@@
     (effects (font (size 1.27 1.27)) (justify right bottom))
   )
-  (label "GND_I2C" (at 34.29 121.92 0)
-    (effects (font (size 1.27 1.27)) (justify left bottom))
-  )
   (label "GND" (at 78.74 121.92 0)
     (effects (font (size 1.27 1.27)) (justify left bottom))
@@
     (effects (font (size 1.27 1.27)) (justify left bottom))
   )
+  (label "GND_I2C" (at 34.29 111.76 0)
+    (effects (font (size 1.27 1.27)) (justify left bottom))
+  )
+  (label "GND_I2C" (at 34.29 99.06 0)
+    (effects (font (size 1.27 1.27)) (justify left bottom))
+  )
+  (label "+5V" (at 34.29 116.84 0)
+    (effects (font (size 1.27 1.27)) (justify left bottom))
+  )
+  (label "GND" (at 48.26 129.54 0)
+    (effects (font (size 1.27 1.27)) (justify left bottom))
+  )
+  (label "I2C1_SDA" (at 76.2 80.01 0)
+    (effects (font (size 1.27 1.27)) (justify left bottom))
+  )
+  (label "I2S_LRCK" (at 76.2 60.96 0)
+    (effects (font (size 1.27 1.27)) (justify left bottom))
+  )
+  (label "+5V" (at 78.74 118.11 0)
+    (effects (font (size 1.27 1.27)) (justify left bottom))
+  )
+  (label "GLOBAL_EN" (at 34.29 73.66 0)
+    (effects (font (size 1.27 1.27)) (justify left bottom))
+  )
+  (label "I2S_ADC" (at 34.29 71.12 0)
+    (effects (font (size 1.27 1.27)) (justify left bottom))
+  )
+  (label "SD_DAT0" (at 82.55 45.72 180)
+    (effects (font (size 1.27 1.27)) (justify right bottom))
+  )
+  (label "I2C1_SDA" (at 34.29 101.6 0)
+    (effects (font (size 1.27 1.27)) (justify left bottom))
+  )
+  (label "3.3V_I2C" (at 53.34 93.98 0)
+    (effects (font (size 1.27 1.27)) (justify left bottom))
+  )
+  (label "SD_DAT1" (at 82.55 48.26 180)
+    (effects (font (size 1.27 1.27)) (justify right bottom))
+  )
+  (label "I2S_LRCK" (at 34.29 76.2 0)
+    (effects (font (size 1.27 1.27)) (justify left bottom))
+  )
+  (label "GND_I2C" (at 34.29 104.14 0)
+    (effects (font (size 1.27 1.27)) (justify left bottom))
+  )
+  (label "GND" (at 76.2 88.9 0)
+    (effects (font (size 1.27 1.27)) (justify left bottom))
+  )
+  (label "SD_DAT2" (at 41.91 34.29 180)
+    (effects (font (size 1.27 1.27)) (justify right bottom))
+  )
+  (label "+5V" (at 34.253 119.38 0)
+    (effects (font (size 1.27 1.27)) (justify left bottom))
+  )
   (label "+5V" (at 34.29 81.28 0)
     (effects (font (size 1.27 1.27)) (justify left bottom))
   )
-  (label "GND_I2C" (at 34.29 111.76 0)
-    (effects (font (size 1.27 1.27)) (justify left bottom))
-  )
-  (label "GND" (at 48.26 129.54 0)
-    (effects (font (size 1.27 1.27)) (justify left bottom))
-  )
-  (label "I2C1_SDA" (at 76.2 80.01 0)
-    (effects (font (size 1.27 1.27)) (justify left bottom))
-  )
-  (label "I2S_LRCK" (at 76.2 60.96 0)
-    (effects (font (size 1.27 1.27)) (justify left bottom))
-  )
-  (label "+5V" (at 78.74 118.11 0)
-    (effects (font (size 1.27 1.27)) (justify left bottom))
-  )
-  (label "I2S_ADC" (at 34.29 71.12 0)
-    (effects (font (size 1.27 1.27)) (justify left bottom))
-  )
-  (label "SD_DAT0" (at 82.55 45.72 180)
-    (effects (font (size 1.27 1.27)) (justify right bottom))
-  )
-  (label "I2C1_SDA" (at 34.29 101.6 0)
-    (effects (font (size 1.27 1.27)) (justify left bottom))
-  )
-  (label "3.3V_I2C" (at 53.34 93.98 0)
-    (effects (font (size 1.27 1.27)) (justify left bottom))
-  )
-  (label "SD_DAT1" (at 82.55 48.26 180)
-    (effects (font (size 1.27 1.27)) (justify right bottom))
-  )
-  (label "I2S_LRCK" (at 34.29 76.2 0)
-    (effects (font (size 1.27 1.27)) (justify left bottom))
-  )
-  (label "GND_I2C" (at 34.29 104.14 0)
-    (effects (font (size 1.27 1.27)) (justify left bottom))
-  )
-  (label "GND" (at 76.2 88.9 0)
-    (effects (font (size 1.27 1.27)) (justify left bottom))
-  )
-  (label "SD_DAT2" (at 41.91 34.29 180)
-    (effects (font (size 1.27 1.27)) (justify right bottom))
-  )
-  (label "+5V" (at 34.29 78.74 0)
-    (effects (font (size 1.27 1.27)) (justify left bottom))
-  )
   (label "GND_I2C" (at 34.29 129.54 0)
     (effects (font (size 1.27 1.27)) (justify left bottom))
@@
     (effects (font (size 1.27 1.27)) (justify left bottom))
   )
+  (label "+5V" (at 34.29 121.92 0)
+    (effects (font (size 1.27 1.27)) (justify left bottom))
+  )
   (label "3.3V" (at 33.02 44.45 0)
     (effects (font (size 1.27 1.27)) (justify left bottom))
@@
     (effects (font (size 1.27 1.27)) (justify left bottom))
   )
-  (label "3.3V_I2C" (at 34.29 99.06 0)
-    (effects (font (size 1.27 1.27)) (justify left bottom))
-  )
   (label "USB_DEBUG_N" (at 31.75 86.36 0)
     (effects (font (size 1.27 1.27)) (justify left bottom))
@@
     (effects (font (size 1.27 1.27)) (justify left bottom))
   )
-  (label "GND_I2C" (at 34.2573 119.38 0)
-    (effects (font (size 1.27 1.27)) (justify left bottom))
-  )
   (label "3.3V" (at 210.82 76.2 0)
     (effects (font (size 1.27 1.27)) (justify left bottom))
@@
     (effects (font (size 1.27 1.27)) (justify right bottom))
   )
+  (label "GND" (at 34.29 63.5 0)
+    (effects (font (size 1.27 1.27)) (justify left bottom))
+  )
   (label "SD_CLK" (at 81.915 40.64 180)
     (effects (font (size 1.27 1.27)) (justify right bottom))
   )
+  (label "nEXTRST" (at 210.82 57.785 0)
+    (effects (font (size 1.27 1.27)) (justify left bottom))
+  )
   (label "USB_DEBUG_N" (at 119.38 60.96 0)
     (effects (font (size 1.27 1.27)) (justify left bottom))
@@
     (effects (font (size 1.27 1.27)) (justify right bottom))
   )
+  (label "nEXTRST" (at 129.54 50.8 180)
+    (effects (font (size 1.27 1.27)) (justify right bottom))
+  )
   (hierarchical_label "I2S_LRCK" (shape bidirectional) (at 45.72 76.2 0)
     (effects (font (size 1.27 1.27)) (justify left))
   )
-  (hierarchical_label "3.3V" (shape output) (at 45.72 63.5 0)
+  (hierarchical_label "+5V" (shape output) (at 45.72 119.38 0)
+    (effects (font (size 1.27 1.27)) (justify left))
+  )
+  (hierarchical_label "+5V" (shape output) (at 45.72 81.28 0)
     (effects (font (size 1.27 1.27)) (justify left))
   )
@@
     (effects (font (size 1.27 1.27)) (justify left))
   )
-  (hierarchical_label "GND_I2C" (shape output) (at 45.72 121.92 0)
-    (effects (font (size 1.27 1.27)) (justify left))
-  )
   (hierarchical_label "I2S_ADC" (shape input) (at 45.72 71.12 0)
     (effects (font (size 1.27 1.27)) (justify left))
@@
     (effects (font (size 1.27 1.27)) (justify left))
   )
-  (hierarchical_label "3.3V_I2C" (shape output) (at 45.72 99.06 0)
+  (hierarchical_label "GND_I2C" (shape output) (at 45.72 111.76 0)
     (effects (font (size 1.27 1.27)) (justify left))
   )
@@
     (effects (font (size 1.27 1.27)) (justify left))
   )
-  (hierarchical_label "+5V" (shape output) (at 45.72 78.74 0)
+  (hierarchical_label "+5V" (shape output) (at 45.72 116.84 0)
+    (effects (font (size 1.27 1.27)) (justify left))
+  )
+  (hierarchical_label "+5V" (shape output) (at 45.72 114.3 0)
+    (effects (font (size 1.27 1.27)) (justify left))
+  )
+  (hierarchical_label "+5V" (shape output) (at 45.72 121.92 0)
     (effects (font (size 1.27 1.27)) (justify left))
   )
@@
       (effects (font (size 1.27 1.27)) (justify right))
     )
+    (pin "nEXTRST" output (at 119.38 50.8 0)
+      (effects (font (size 1.27 1.27)) (justify right))
+    )
+    (pin "GLOBAL_EN" input (at 119.38 53.34 0)
+      (effects (font (size 1.27 1.27)) (justify right))
+    )

Commit message: .
.
Parts:
- removed J10: Conn_01x10, Connector_PinHeader_2.54mm:PinHeader_1x10_P2.54mm_Vertical, symbol Connector_Generic:Conn_01x10
Other:
- removed sheet xHCI-USB3
- note removed: "Connectors ------- USB 3.0 DUAL"

Commit message: .
.
Parts:
- added R1, R2: NC, Resistor_SMD:R_0402_1005Metric, symbol Device:R_Small_US
Connections:
- net USB_DEBUG_N: now also R2.2; no longer J6.1 (Pin_1)
- net USB_DEBUG_P: now also R1.2; no longer J6.2 (Pin_2)
- new net POWER/USB2_N: R2.1
- new net POWER/USB2_P: R1.1
Other:
- sheet POWER ports: added USB2_N, USB2_P, USBOTG; removed none
Changed lines of the file:
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@@
+    (stroke (width 0) (type default) (color 0 0 0 0))
+  )
+  (wire (pts (xy 119.38 124.46) (xy 125.73 124.46))
     (stroke (width 0) (type default) (color 0 0 0 0))
   )
@@
     (stroke (width 0) (type default) (color 0 0 0 0))
   )
+  (wire (pts (xy 119.38 130.81) (xy 138.43 130.81))
+    (stroke (width 0) (type default) (color 0 0 0 0))
+  )
   (wire (pts (xy 30.48 121.92) (xy 45.72 121.92))
     (stroke (width 0) (type default) (color 0 0 0 0))
   )
+  (wire (pts (xy 130.81 124.46) (xy 148.59 124.46))
+    (stroke (width 0) (type default) (color 0 0 0 0))
+  )
   (wire (pts (xy 74.93 121.92) (xy 87.63 121.92))
     (stroke (width 0) (type default) (color 0 0 0 0))
   )
+  (wire (pts (xy 119.38 118.11) (xy 125.73 118.11))
+    (stroke (width 0) (type default) (color 0 0 0 0))
+  )
   (wire (pts (xy 72.39 83.82) (xy 87.63 83.82))
     (stroke (width 0) (type default) (color 0 0 0 0))
@@
     (stroke (width 0) (type default) (color 0 0 0 0))
   )
+  (wire (pts (xy 130.81 118.11) (xy 148.59 118.11))
+    (stroke (width 0) (type default) (color 0 0 0 0))
+  )
   (wire (pts (xy 30.48 71.12) (xy 45.72 71.12))
     (stroke (width 0) (type default) (color 0 0 0 0))
@@
     (effects (font (size 1.27 1.27)) (justify left bottom))
   )
+  (label "USB_OTG" (at 121.92 66.04 0)
+    (effects (font (size 1.27 1.27)) (justify left bottom))
+  )
   (label "SD_CMD" (at 81.915 43.18 180)
     (effects (font (size 1.27 1.27)) (justify right bottom))
@@
     (effects (font (size 1.27 1.27)) (justify left bottom))
   )
+  (label "USB_DEBUG_N" (at 133.35 124.46 0)
+    (effects (font (size 1.27 1.27)) (justify left bottom))
+  )
+  (label "USB_OTG" (at 123.19 130.81 0)
+    (effects (font (size 1.27 1.27)) (justify left bottom))
+  )
+  (label "USB_DEBUG_P" (at 133.35 118.11 0)
+    (effects (font (size 1.27 1.27)) (justify left bottom))
+  )
   (label "GND" (at 127 87.63 0)
     (effects (font (size 1.27 1.27)) (justify left bottom))
@@
     (effects (font (size 1.27 1.27)) (justify left bottom))
   )
-  (label "USB_DEBUG_N" (at 31.75 86.36 0)
-    (effects (font (size 1.27 1.27)) (justify left bottom))
-  )
   (label "GND" (at 34.29 63.5 0)
     (effects (font (size 1.27 1.27)) (justify left bottom))
@@
     (effects (font (size 1.27 1.27)) (justify right bottom))
   )
-  (label "USB_DEBUG_P" (at 31.75 83.82 0)
-    (effects (font (size 1.27 1.27)) (justify left bottom))
-  )
   (label "nEXTRST" (at 129.54 50.8 180)
     (effects (font (size 1.27 1.27)) (justify right bottom))
@@
   (hierarchical_label "+5V" (shape output) (at 45.72 121.92 0)
     (effects (font (size 1.27 1.27)) (justify left))
+  )
+  (symbol (lib_id "Device:R_Small_US") (at 128.27 124.46 90) (unit 1)
+    (in_bom yes) (on_board yes)
+    (property "Reference" "R2" (id 0) (at 127 121.92 90))
+    (property "Value" "NC" (id 1) (at 130.81 121.92 90))
+    (property "Footprint" "Resistor_SMD:R_0402_1005Metric" (id 2) (at 128.27 124.46 0)
+      (effects (font (size 1.27 1.27)) hide)
+    )
+    (property "Datasheet" "~" (id 3) (at 128.27 124.46 0)
+      (effects (font (size 1.27 1.27)) hide)
+    )
+    (pin "1")
+    (pin "2")
   )
   (symbol (lib_id "Connector_Generic:Conn_01x10") (at 25.4 76.2 180) (unit 1)
@@
     (pin "9")
   )
+  (symbol (lib_id "Device:R_Small_US") (at 128.27 118.11 90) (unit 1)
+    (in_bom yes) (on_board yes)
+    (property "Reference" "R1" (id 0) (at 127 115.57 90))
+    (property "Value" "NC" (id 1) (at 130.81 115.57 90))
+    (property "Footprint" "Resistor_SMD:R_0402_1005Metric" (id 2) (at 128.27 118.11 0)
+      (effects (font (size 1.27 1.27)) hide)
+    )
+    (property "Datasheet" "~" (id 3) (at 128.27 118.11 0)
+      (effects (font (size 1.27 1.27)) hide)
+    )
+    (pin "1")
+    (pin "2")
+  )
   (symbol (lib_id "Connector_Generic:Conn_01x10") (at 25.4 111.76 180) (unit 1)
     (in_bom yes) (on_board yes) (fields_autoplaced)
@@
       (effects (font (size 1.27 1.27)) (justify left))
     )
-  )
+    (pin "USB2_P" output (at 119.38 118.11 0)
+      (effects (font (size 1.27 1.27)) (justify right))
+    )
+    (pin "USB2_N" output (at 119.38 124.46 0)
+      (effects (font (size 1.27 1.27)) (justify right))
+    )
+    (pin "USBOTG" output (at 119.38 130.81 0)
+      (effects (font (size 1.27 1.27)) (justify right))
+    )
+  )
