File: audio/CM4_HIGH_SPEED.kicad_sch (KiCad schematic)
At the start: 5 parts, among them J1 HDMI, U1 RT9742SNGV

Commit message: .
.
Parts:
- J1: footprint CM4IO:EDAC 690-019-298-412 -> CM4IO:CUI_HD02-19-M-MSMT-TR
Changed lines of the file:
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@@
       (effects (font (size 1.27 1.27)) (justify left))
     )
-    (property "Footprint" "CM4IO:EDAC 690-019-298-412" (id 2) (at 252.095 54.61 0)
+    (property "Footprint" "CM4IO:CUI_HD02-19-M-MSMT-TR" (id 2) (at 252.095 54.61 0)
       (effects (font (size 1.27 1.27)) hide)
     )

Commit message: .
.
Parts:
- J1: footprint CM4IO:CUI_HD02-19-M-MSMT-TR -> CM4IO:685119134923
Changed lines of the file:
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@@
       (effects (font (size 1.27 1.27)) (justify left))
     )
-    (property "Footprint" "CM4IO:CUI_HD02-19-M-MSMT-TR" (id 2) (at 252.095 54.61 0)
+    (property "Footprint" "CM4IO:685119134923" (id 2) (at 252.095 54.61 0)
       (effects (font (size 1.27 1.27)) hide)
     )

Commit message: .
.
Parts:
- added J?: 1054500101, CM4IO:MOLEX_105450-0101, symbol CM4IO:1054500101
- added U?: TPD4EUSB30, Package_SON:USON-10_2.5x1.0mm_P0.5mm, symbol CM4IO:TPD4EUSB30
Connections:
- net +5v: now also J?.A4 (VBUS_A), J?.A9 (VBUS_A), J?.B4 (VBUS_B), J?.B9 (VBUS_B)
- net GND: now also J1.20 (SH), J1.21 (SH), J1.22 (SH), J1.23 (SH), J?.A1 (GND_A), J?.A12 (GND_A), J?.B1 (GND_B), J?.B12 (GND_B), J?.S1 (SHIELD), J?.S2 (SHIELD), J?.S3 (SHIELD), J?.S4 (SHIELD), U?.3 (GND), U?.8 (GND); no longer J1.SH1 (SH), J1.SH2 (SH), J1.SH3 (SH), J1.SH4 (SH)
- net USB2_N: now reaches CM4_MODULE1.103 (USB2_N)
- net USB2_N: now also J?.A7 (D1-), J?.B7 (D2-)
- net USB2_P: now reaches CM4_MODULE1.105 (USB2_P)
- net USB2_P: now also J?.A6 (D1+), J?.B6 (D2+)
- new net: U?.1 (D1+), U?.10
- new net: U?.2 (D1-), U?.9
- new net USBD_N: U?.4 (D2+), U?.7
- new net USBD_P: U?.5 (D2-), U?.6
Other:
- note added: "Micro USB ESD protection"

Commit message: .
.
Parts:
- removed J?: 1054500101, CM4IO:MOLEX_105450-0101, symbol CM4IO:1054500101
- removed U?: TPD4EUSB30, Package_SON:USON-10_2.5x1.0mm_P0.5mm, symbol CM4IO:TPD4EUSB30
Connections:
- net GND: now also CM4_MODULE1.107 (GND), CM4_MODULE1.108 (GND), CM4_MODULE1.113 (GND), CM4_MODULE1.114 (GND), CM4_MODULE1.119 (GND), CM4_MODULE1.120 (GND), CM4_MODULE1.125 (GND), CM4_MODULE1.126 (GND), CM4_MODULE1.131 (GND), CM4_MODULE1.132 (GND), CM4_MODULE1.137 (GND), CM4_MODULE1.138 (GND), CM4_MODULE1.144 (GND), CM4_MODULE1.150 (GND), CM4_MODULE1.155 (GND), CM4_MODULE1.156 (GND), CM4_MODULE1.161 (GND), CM4_MODULE1.162 (GND), CM4_MODULE1.167 (GND), CM4_MODULE1.168 (GND), CM4_MODULE1.173 (GND), CM4_MODULE1.174 (GND), CM4_MODULE1.179 (GND), CM4_MODULE1.185 (GND), CM4_MODULE1.186 (GND), CM4_MODULE1.191 (GND), CM4_MODULE1.192 (GND), CM4_MODULE1.197 (GND), CM4_MODULE1.198 (GND)
- net USB_OTG_ID: now reaches CM4_MODULE1.101 (USB_OTG_ID)
Other:
- note removed: "Micro USB ESD protection"

Commit message: .
.
Changed lines of the file:
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@@
     (effects (font (size 1.27 1.27)) (justify right))
   )
-  (hierarchical_label "USB_OTG_ID" (shape output) (at 106.68 34.29 0)
+  (hierarchical_label "USB_OTG_ID" (shape input) (at 106.68 34.29 0)
     (effects (font (size 1.27 1.27)) (justify left))
   )
