File: audio/CM4_docker1_sch.kicad_sch (KiCad schematic)
At the start: 0 parts

Commit message: .
.
Changed lines of the file:
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@@
     (effects (font (size 1.27 1.27)) (justify left bottom))
   )
-  (hierarchical_label "+5V" (shape output) (at 132.08 118.11 0)
+  (hierarchical_label "+5V" (shape input) (at 132.08 118.11 0)
     (effects (font (size 1.27 1.27)) (justify left))
   )
-  (hierarchical_label "GND" (shape output) (at 132.08 120.65 0)
+  (hierarchical_label "GND" (shape input) (at 132.08 120.65 0)
     (effects (font (size 1.27 1.27)) (justify left))
   )
