File: audio/audio.kicad_pcb (KiCad board)
At the start: 2 copper layers, 70 x 60 mm, 67 parts, among them J1 HDMI, J2 Conn_02x05_Odd_Even, J3 USB3_A, J4 THD-02-R, Q1 DMG1012T, U1 RT9742SNGV, U2 AP3429KTTR-G1, U3 VL805, U4 AP22653W6, U5 TPD4EUSB30, U6 TPD4EUSB30, U7 MagJack-A70-112-331N126, Y1 25MHz

Commit message: .
.
Parts:
- removed J4: THD-02-R, Connector_PinHeader_2.54mm:PinHeader_2x02_P2.54mm_Vertical
- removed U7: MagJack-A70-112-331N126, CM4IO:TRJG0926HENL
- added J5: 1054500101, CM4IO:MOLEX_105450-0101, F.Cu at (24.9, 3.09)
- J1: footprint CM4IO:EDAC 690-019-298-412 -> CM4IO:CUI_HD02-19-M-MSMT-TR
- J2: value Conn_02x05_Odd_Even -> JK00177; footprint Connector_PinHeader_2.54mm:PinHeader_2x05_P2.54mm_Vertical -> Connector_RJ:RJ45_Pulse_JK00177NL_Horizontal
- moved C5 96.5 mm to (19.0, 41.0), turned to 90 degrees
- moved C30 94.5 mm to (23.0, 45.0)
- moved C18 93.7 mm to (17.0, 21.0)
- moved C22 92.7 mm to (19.0, 38.0), turned to 90 degrees
- moved C33 89.9 mm to (22.0, 33.0)
- moved C10 89.5 mm to (19.0, 35.0), turned to 90 degrees
- moved C36 89.3 mm to (31.0, 44.0), turned to -90 degrees
- moved C31 88.3 mm to (31.0, 41.0), turned to -90 degrees
- moved R2 87.1 mm to (25.0, 33.0)
- moved R4 86.5 mm to (16.0, 32.0), turned to 90 degrees
- moved C9 86.4 mm to (19.0, 33.0)
- moved C32 84.9 mm to (31.0, 38.0), turned to -90 degrees
- moved C11 84.9 mm to (16.5, 30.0)
- moved C13 84.8 mm to (24.0, 20.0)
- moved C12 84.1 mm to (31.0, 35.0), turned to -90 degrees
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Connections:
- C39 pad 1: Net-(C39-Pad1) -> Net-(J2-Pad12)
- J2 pad 1: /CM4_docker1/xHCI-USB3/VBUS -> Net-(J2-Pad12)
- J2 pad 10: unconnected-(J2-Pad10) -> /CM4_docker1/CM4_LOW_SPEED/TRD0_N
- J2 pad 2: /CM4_docker1/xHCI-USB3/VBUS -> /CM4_docker1/CM4_LOW_SPEED/TRD2_N
- J2 pad 3: /CM4_docker1/xHCI-USB3/PD3_N -> /CM4_docker1/CM4_LOW_SPEED/TRD2_P
- J2 pad 4: /CM4_docker1/xHCI-USB3/PD4_N -> /CM4_docker1/CM4_LOW_SPEED/TRD1_P
- J2 pad 5: /CM4_docker1/xHCI-USB3/PD3_P -> /CM4_docker1/CM4_LOW_SPEED/TRD1_N
- J2 pad 6: /CM4_docker1/xHCI-USB3/PD4_P -> Net-(J2-Pad12)
- J2 pad 7: GND -> Net-(J2-Pad12)
- J2 pad 8: GND -> /CM4_docker1/CM4_LOW_SPEED/TRD3_P
- J2 pad 9: unconnected-(J2-Pad9) -> /CM4_docker1/CM4_LOW_SPEED/TRD3_N
- R10 pad 1: Net-(R10-Pad1) -> Net-(J2-Pad15)
- R10 pad 2: /CM4_docker1/CM4_LOW_SPEED/ETH_LEDG -> /CM4_docker1/CM4_LOW_SPEED/ETH_LEDY
- R11 pad 1: Net-(R11-Pad1) -> Net-(J2-Pad14)
- R11 pad 2: /CM4_docker1/CM4_LOW_SPEED/ETH_LEDY -> /CM4_docker1/CM4_LOW_SPEED/ETH_LEDG
Routing:
- net (no net): vias 0 -> 4
Other:
- board size 70 x 60 mm -> 75 x 75 mm

Commit message: .
.
Parts:
- added J5: 1054500101, CM4IO:MOLEX_105450-0101, F.Cu at (53.5, 71.2)
- J1: footprint CM4IO:CUI_HD02-19-M-MSMT-TR -> CM4IO:685119134923
- moved U1 114.6 mm to (127.1, 42.4)
- moved C1 114.0 mm to (131.0, 41.1)
- moved C2 114.0 mm to (131.0, 43.1)
- moved R6 99.2 mm to (106.3, 47.2), turned to 0 degrees
- moved Q1 98.6 mm to (111.3, 41.7)
- moved C22 97.6 mm to (116.5, 43.1), turned to 0 degrees
- moved C10 95.0 mm to (113.6, 44.3), turned to 0 degrees
- moved C11 94.9 mm to (108.3, 54.1)
- moved R7 93.6 mm to (100.9, 52.2), turned to 0 degrees
- moved C15 93.3 mm to (114.9, 46.3)
- moved C28 91.9 mm to (112.0, 48.3)
- moved C21 91.2 mm to (117.3, 41.1)
- moved C29 89.3 mm to (104.7, 58.1)
- moved R8 89.2 mm to (87.2, 58.9), turned to 0 degrees
- moved C32 88.5 mm to (119.3, 43.1), turned to 0 degrees
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Routing:
- net /CM4_docker1/xHCI-USB3/SSRX2_P: track 0.00 -> 34.0 mm
- net /CM4_docker1/xHCI-USB3/SSRX2_N: track 0.00 -> 34.0 mm
- net /CM4_docker1/CM4_HIGH_SPEED/HDMI0_D1_P: track 0.00 -> 25.6 mm
- net /CM4_docker1/CM4_HIGH_SPEED/HDMI0_D0_P: track 0.00 -> 25.6 mm
- net /CM4_docker1/CM4_HIGH_SPEED/HDMI0_D0_N: track 0.00 -> 25.6 mm
- net /CM4_docker1/CM4_HIGH_SPEED/HDMI0_D1_N: track 0.00 -> 25.5 mm
- net /CM4_docker1/CM4_HIGH_SPEED/HDMI0_D2_P: track 0.00 -> 25.4 mm
- net /CM4_docker1/CM4_HIGH_SPEED/HDMI0_D2_N: track 0.00 -> 25.3 mm
- net /CM4_docker1/CM4_HIGH_SPEED/HDMI0_CK_N: track 0.00 -> 25.3 mm
- net /CM4_docker1/CM4_HIGH_SPEED/HDMI0_CK_P: track 0.00 -> 25.1 mm
- net /CM4_docker1/xHCI-USB3/SSTX2_N: track 0.00 -> 23.3 mm
- net /CM4_docker1/xHCI-USB3/SSTX2_P: track 0.00 -> 23.2 mm
- net /CM4_docker1/xHCI-USB3/SSRX1_N: track 0.00 -> 9.38 mm
- net /CM4_docker1/xHCI-USB3/SSRX1_P: track 0.00 -> 9.36 mm
- net /CM4_docker1/CM4_HIGH_SPEED/PCIE_CLK_P: track 0.00 -> 5.04 mm
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Other:
- outline, holes or cut-outs redrawn
- copper layers 2 -> 4
- board text added: "Board thickness : 1.56mm Finished copper weight inners : 1oz Finished copper weight outers : 1oz Board finish : OSP Material type : FR4 Colour of solder resists : Green Colour of silk screens : White Only on the top side Board to : UL94-V0 TG >=130 50R trace width 0.13mm@ 3GHz 90R diff pair width 0.147 spacing 0.253mm @ 2.5GHz 100R diff pair width 0.127 spacing 0.253mm @ 2GHz"

Commit message: .
.
Parts:
- moved C37 10.3 mm to (19.5, 38.4)
- moved C38 10.3 mm to (19.5, 39.5)
Routing:
- net /CM4_docker1/CM4_LOW_SPEED/TRD2_N: track 0.00 -> 56.6 mm
- net /CM4_docker1/CM4_LOW_SPEED/TRD2_P: track 0.00 -> 55.9 mm
- net /CM4_docker1/CM4_LOW_SPEED/TRD3_P: track 0.00 -> 54.1 mm
- net /CM4_docker1/CM4_LOW_SPEED/TRD3_N: track 0.00 -> 53.5 mm
- net /CM4_docker1/CM4_LOW_SPEED/TRD1_N: track 0.00 -> 52.1 mm
- net /CM4_docker1/CM4_LOW_SPEED/TRD0_N: track 0.00 -> 52.0 mm
- net /CM4_docker1/CM4_LOW_SPEED/TRD1_P: track 0.00 -> 51.4 mm
- net /CM4_docker1/CM4_LOW_SPEED/TRD0_P: track 0.00 -> 50.4 mm
- net /CM4_docker1/xHCI-USB3/SSTX2_N: track 23.3 -> 38.3 mm, vias 0 -> 1
- net /CM4_docker1/xHCI-USB3/SSTX2_P: track 23.2 -> 37.2 mm, vias 0 -> 1
- net /CM4_docker1/CM4_HIGH_SPEED/PCIE_CLK_P: track 5.04 -> 0.00 mm
- net /CM4_docker1/CM4_HIGH_SPEED/PCIE_CLK_N: track 4.88 -> 0.00 mm
- net /CM4_docker1/xHCI-USB3/PEXTX_N: track 2.51 -> 0.00 mm
- net /CM4_docker1/xHCI-USB3/C2_N: track 0.00 -> 2.46 mm
- net /CM4_docker1/xHCI-USB3/C2_P: track 0.00 -> 2.45 mm
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
Commit message: .
.
Parts:
- removed J5 (x2): 1054500101, CM4IO:MOLEX_105450-0101
Connections:
- J1 pad 20: (no net) -> GND
- J1 pad 21: (no net) -> GND
- J1 pad 22: (no net) -> GND
- J1 pad 23: (no net) -> GND

Commit message: .
.
Parts:
- removed U2: AP3429KTTR-G1, Package_TO_SOT_SMD:TSOT-23-5
- added C40: 22u, Capacitor_SMD:C_0805_2012Metric, F.Cu at (29.0, 71.9)
- added J4: 1054500101, CM4IO:MOLEX_105450-0101, F.Cu at (17.8, 3.77)
- added J5: 1054500101, CM4IO:MOLEX_105450-0101, F.Cu at (62.8, 3.73)
- added R12: 5.1K 5%, Resistor_SMD:R_0402_1005Metric, F.Cu at (7.77, 3.19)
- added R13: 5.1K 5%, Resistor_SMD:R_0402_1005Metric, F.Cu at (10.8, 1.39)
- added R14: 5.1K 5%, Resistor_SMD:R_0402_1005Metric, F.Cu at (10.7, 3.19)
- added R15: 5.1K 5%, Resistor_SMD:R_0402_1005Metric, F.Cu at (7.77, 1.20)
- added U7: TPD4EUSB30, Package_SON:USON-10_2.5x1.0mm_P0.5mm, F.Cu at (17.8, 9.58)
- added U8: AP3402, Package_TO_SOT_SMD:TSOT-23-6, F.Cu at (14.4, 71.5)
- C17, C7: value 10u -> 22u
- L2: value 2.2uH -> 1.0uH
- moved C1 115.9 mm to (18.6, 13.0)
- moved C2 115.9 mm to (18.6, 15.0)
- moved U1 115.9 mm to (14.7, 14.2)
- moved R2 106.1 mm to (8.49, 72.8)
- moved C7 101.0 mm to (10.9, 71.4), turned to 90 degrees
- moved R1 95.4 mm to (8.55, 70.3)
- moved C21 91.3 mm to (31.4, 72.0), turned to 90 degrees
- moved C3 87.2 mm to (25.1, 1.55)
- moved R6 86.1 mm to (23.4, 70.4), turned to 90 degrees
- moved C16 84.9 mm to (21.4, 31.5), turned to 90 degrees
- moved R5 84.4 mm to (30.2, 4.32), turned to 90 degrees
- moved C18 84.3 mm to (28.9, 1.55)
- moved C11 83.9 mm to (27.5, 31.4), turned to -90 degrees
- moved C17 81.8 mm to (25.8, 71.7), turned to 90 degrees
- moved U4 81.5 mm to (25.7, 5.25)
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Connections:
- net /CM4_docker1/CM4_HIGH_SPEED/+5v renamed /CM4_docker1/CM4_HIGH_SPEED/5V
- CM4_MODULE1 pad 103: unconnected-(CM4_MODULE1-Pad103) -> /CM4_docker1/CM4_LOW_SPEED/USB2_N
- CM4_MODULE1 pad 105: unconnected-(CM4_MODULE1-Pad105) -> /CM4_docker1/CM4_LOW_SPEED/USB2_P
Routing:
- net /CM4_docker1/CM4_LOW_SPEED/TRD0_N: track 52.0 -> 112.5 mm
- net /CM4_docker1/CM4_LOW_SPEED/TRD0_P: track 50.4 -> 0.00 mm
- net /CM4_docker1/CM4_LOW_SPEED/TRD2_N: track 56.6 -> 50.4 mm
- net /CM4_docker1/CM4_LOW_SPEED/TRD2_P: track 55.9 -> 52.0 mm
- net /CM4_docker1/xHCI-USB3/SSRX1_P: track 9.06 -> 11.2 mm
- net /CM4_docker1/xHCI-USB3/SSTX2_P: track 37.2 -> 39.2 mm
- net /CM4_docker1/xHCI-USB3/SSTX2_N: track 38.3 -> 40.2 mm
- net /CM4_docker1/xHCI-USB3/SSRX2_N: track 34.4 -> 35.2 mm
- net /CM4_docker1/xHCI-USB3/SSRX1_N: track 10.6 -> 11.1 mm

Commit message: .
.
Parts:
- added R16: 2.2K 1%, Resistor_SMD:R_0402_1005Metric, F.Cu at (7.60, 5.84)
- added R17: 2.2K 1%, Resistor_SMD:R_0402_1005Metric, F.Cu at (10.4, 7.70)
- added R18: 2.2K 1%, Resistor_SMD:R_0402_1005Metric, F.Cu at (10.6, 5.71)
- added R19: 5.1K 5%, Resistor_SMD:R_0402_1005Metric, F.Cu at (55.7, 2.00)
- added R20: 5.1K 5%, Resistor_SMD:R_0402_1005Metric, F.Cu at (52.8, 2.00)
- added R21: 5.1K 5%, Resistor_SMD:R_0402_1005Metric, F.Cu at (52.8, 3.99)
- added R22: 5.1K 5%, Resistor_SMD:R_0402_1005Metric, F.Cu at (55.7, 3.99)
Connections:
- C1 pad 1: /CM4_docker1/CM4_HIGH_SPEED/5V -> /CM4_docker1/+5V
- C3 pad 1: /CM4_docker1/xHCI-USB3/+5v -> /CM4_docker1/+5V
- C7 pad 1: /CM4_docker1/xHCI-USB3/+5v -> /CM4_docker1/+5V
- CM4_MODULE1 pad 101: unconnected-(CM4_MODULE1-Pad101) -> /CM4_docker1/CM4_HIGH_SPEED/USB_OTG_ID
- CM4_MODULE1 pad 107: unconnected-(CM4_MODULE1-Pad107) -> GND
- CM4_MODULE1 pad 108: unconnected-(CM4_MODULE1-Pad108) -> GND
- CM4_MODULE1 pad 113: unconnected-(CM4_MODULE1-Pad113) -> GND
- CM4_MODULE1 pad 114: unconnected-(CM4_MODULE1-Pad114) -> GND
- CM4_MODULE1 pad 119: unconnected-(CM4_MODULE1-Pad119) -> GND
- CM4_MODULE1 pad 120: unconnected-(CM4_MODULE1-Pad120) -> GND
- CM4_MODULE1 pad 125: unconnected-(CM4_MODULE1-Pad125) -> GND
- CM4_MODULE1 pad 126: unconnected-(CM4_MODULE1-Pad126) -> GND
- CM4_MODULE1 pad 131: unconnected-(CM4_MODULE1-Pad131) -> GND
- CM4_MODULE1 pad 132: unconnected-(CM4_MODULE1-Pad132) -> GND
- CM4_MODULE1 pad 137: unconnected-(CM4_MODULE1-Pad137) -> GND
- CM4_MODULE1 pad 138: unconnected-(CM4_MODULE1-Pad138) -> GND
- CM4_MODULE1 pad 144: unconnected-(CM4_MODULE1-Pad144) -> GND
- CM4_MODULE1 pad 150: unconnected-(CM4_MODULE1-Pad150) -> GND
- CM4_MODULE1 pad 155: unconnected-(CM4_MODULE1-Pad155) -> GND
- CM4_MODULE1 pad 156: unconnected-(CM4_MODULE1-Pad156) -> GND
- CM4_MODULE1 pad 161: unconnected-(CM4_MODULE1-Pad161) -> GND
- CM4_MODULE1 pad 162: unconnected-(CM4_MODULE1-Pad162) -> GND
- CM4_MODULE1 pad 167: unconnected-(CM4_MODULE1-Pad167) -> GND
- CM4_MODULE1 pad 168: unconnected-(CM4_MODULE1-Pad168) -> GND
- CM4_MODULE1 pad 173: unconnected-(CM4_MODULE1-Pad173) -> GND
- CM4_MODULE1 pad 174: unconnected-(CM4_MODULE1-Pad174) -> GND
- CM4_MODULE1 pad 179: unconnected-(CM4_MODULE1-Pad179) -> GND
- CM4_MODULE1 pad 185: unconnected-(CM4_MODULE1-Pad185) -> GND
- CM4_MODULE1 pad 186: unconnected-(CM4_MODULE1-Pad186) -> GND
- CM4_MODULE1 pad 191: unconnected-(CM4_MODULE1-Pad191) -> GND
- CM4_MODULE1 pad 192: unconnected-(CM4_MODULE1-Pad192) -> GND
- CM4_MODULE1 pad 197: unconnected-(CM4_MODULE1-Pad197) -> GND
- CM4_MODULE1 pad 198: unconnected-(CM4_MODULE1-Pad198) -> GND
- J4 pad A4: /CM4_docker1/CM4_LOW_SPEED/5V -> /CM4_docker1/CM4_LOW_SPEED/VBUS
- J4 pad A9: /CM4_docker1/CM4_LOW_SPEED/5V -> /CM4_docker1/CM4_LOW_SPEED/VBUS
- J4 pad B4: /CM4_docker1/CM4_LOW_SPEED/5V -> /CM4_docker1/CM4_LOW_SPEED/VBUS
- J4 pad B9: /CM4_docker1/CM4_LOW_SPEED/5V -> /CM4_docker1/CM4_LOW_SPEED/VBUS
- J5 pad A1: unconnected-(J5-PadA1) -> GND
- J5 pad A12: unconnected-(J5-PadA12) -> GND
- J5 pad A4: unconnected-(J5-PadA4) -> /CM4_docker1/+5V
- J5 pad A5: unconnected-(J5-PadA5) -> /CM4_docker1/POWER/CC1
- J5 pad A9: unconnected-(J5-PadA9) -> /CM4_docker1/+5V
- J5 pad B1: unconnected-(J5-PadB1) -> GND
- J5 pad B12: unconnected-(J5-PadB12) -> GND
- J5 pad B4: unconnected-(J5-PadB4) -> /CM4_docker1/+5V
- J5 pad B5: unconnected-(J5-PadB5) -> /CM4_docker1/POWER/CC2
- J5 pad B9: unconnected-(J5-PadB9) -> /CM4_docker1/+5V
- J5 pad S1: unconnected-(J5-PadS1) -> GND
- J5 pad S2: unconnected-(J5-PadS2) -> GND
- J5 pad S3: unconnected-(J5-PadS3) -> GND
- J5 pad S4: unconnected-(J5-PadS4) -> GND
- U1 pad 1: /CM4_docker1/CM4_HIGH_SPEED/5V -> /CM4_docker1/+5V
- U4 pad 1: /CM4_docker1/xHCI-USB3/+5v -> /CM4_docker1/+5V
- U8 pad 4: /CM4_docker1/xHCI-USB3/+5v -> /CM4_docker1/+5V

Commit message: .
.
Parts:
- added J6: Conn_01x10, Connector_PinHeader_2.54mm:PinHeader_1x10_P2.54mm_Vertical, F.Cu at (31.0, 3.00)
- added J7: Conn_01x10, Connector_PinHeader_2.54mm:PinHeader_1x10_P2.54mm_Vertical, F.Cu at (40.0, 71.0)
- added J8: Conn_01x10, Connector_PinSocket_2.54mm:PinSocket_1x10_P2.54mm_Vertical, B.Cu at (131.0, 3.00)
- added J9: Conn_01x10, Connector_PinSocket_2.54mm:PinSocket_1x10_P2.54mm_Vertical, B.Cu at (140.0, 71.0)
- added PS1: R05CTE05S-R, CM4IO:SOIC127P1030X265-16N, F.Cu at (132.0, 17.5)
- moved C34 17.8 mm to (31.5, 69.5)
- moved C33 17.6 mm to (30.0, 72.5)
- moved C32 16.2 mm to (30.0, 69.5)
- moved C10 15.8 mm to (43.8, 67.3)
- moved C13 15.8 mm to (42.5, 67.2)
- moved C15 15.8 mm to (41.2, 67.3)
- moved C19 15.8 mm to (39.9, 67.3)
- moved C22 15.8 mm to (38.5, 67.5)
- moved C23 15.8 mm to (37.4, 67.5)
- moved C27 15.8 mm to (36.2, 67.5)
- moved C4 15.8 mm to (51.5, 67.0)
- moved C8 15.8 mm to (47.2, 67.2)
- moved C9 15.8 mm to (45.1, 67.2)
- moved L1 15.8 mm to (49.3, 67.3)
- moved C31 15.7 mm to (28.5, 72.5)
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Connections:
- C4 pad 1: /CM4_docker1/xHCI-USB3/+3.3v -> /CM4_docker1/3.3V
- CM4_MODULE1 pad 26: unconnected-(CM4_MODULE1-Pad26) -> /CM4_docker1/I2S_LRCK
- CM4_MODULE1 pad 27: unconnected-(CM4_MODULE1-Pad27) -> /CM4_docker1/I2S_ADC
- CM4_MODULE1 pad 49: unconnected-(CM4_MODULE1-Pad49) -> /CM4_docker1/I2S_BCLK
- CM4_MODULE1 pad 56: unconnected-(CM4_MODULE1-Pad56) -> /CM4_docker1/I2C1_SCL
- CM4_MODULE1 pad 58: unconnected-(CM4_MODULE1-Pad58) -> /CM4_docker1/I2C1_SDA
- CM4_MODULE1 pad 84: unconnected-(CM4_MODULE1-Pad84) -> /CM4_docker1/3.3V
- CM4_MODULE1 pad 86: unconnected-(CM4_MODULE1-Pad86) -> /CM4_docker1/3.3V
- CM4_MODULE1 pad 98: unconnected-(CM4_MODULE1-Pad98) -> GND
- J5 pad A1: GND -> /CM4_docker1/+5V
- J5 pad A12: GND -> /CM4_docker1/+5V
- J5 pad A4: /CM4_docker1/+5V -> GND
- J5 pad A9: /CM4_docker1/+5V -> GND
- J5 pad B1: GND -> /CM4_docker1/+5V
- J5 pad B12: GND -> /CM4_docker1/+5V
- J5 pad B4: /CM4_docker1/+5V -> GND
- J5 pad B9: /CM4_docker1/+5V -> GND
- J5 pad S1: GND -> /CM4_docker1/+5V
- J5 pad S2: GND -> /CM4_docker1/+5V
- J5 pad S3: GND -> /CM4_docker1/+5V
- J5 pad S4: GND -> /CM4_docker1/+5V
- L1 pad 1: /CM4_docker1/xHCI-USB3/+3.3v -> /CM4_docker1/3.3V
- R1 pad 1: /CM4_docker1/xHCI-USB3/+3.3v -> /CM4_docker1/3.3V
- R16 pad 2: /CM4_docker1/CM4_HIGH_SPEED/USB_OTG_ID -> Net-(R16-Pad2)
- R18 pad 2: /CM4_docker1/CM4_HIGH_SPEED/USB_OTG_ID -> Net-(R16-Pad2)
- R19 pad 1: /CM4_docker1/+5V -> GND
- R20 pad 2: GND -> /CM4_docker1/+5V
- R21 pad 1: /CM4_docker1/+5V -> GND
- R22 pad 2: GND -> /CM4_docker1/+5V
Routing:
- net GND: track 0.00 -> 76.7 mm
- net /CM4_docker1/I2S_BCLK: track 0.00 -> 50.4 mm
- net /CM4_docker1/CM4_HIGH_SPEED/HDMI0_D0_P: track 25.6 -> 0.00 mm
- net /CM4_docker1/CM4_HIGH_SPEED/HDMI0_D0_N: track 25.6 -> 0.00 mm
- net /CM4_docker1/CM4_HIGH_SPEED/HDMI0_D1_N: track 25.5 -> 0.00 mm
- net /CM4_docker1/CM4_HIGH_SPEED/HDMI0_CK_N: track 25.3 -> 0.00 mm
- net /CM4_docker1/CM4_HIGH_SPEED/HDMI0_CK_P: track 25.1 -> 0.00 mm
- net (no net): vias 4 -> 7
Other:
- board size 75 x 75 mm -> 175 x 75 mm
- board text added: "0"
- board text added: "1"
- board text added: "2"
- board text added: "3"
- board text added: "4"
- board text added: "5"
- board text added: "6"
- board text added: "7"
- board text added: "8"
- board text added: "9"
- board text added: "ISOLATION"

Commit message: .
.
Parts:
- added PS2: R05CTE05S-R, CM4IO:SOIC127P1030X265-16N, F.Cu at (154.0, 26.5)
- added U10: ac108, CM4IO:AC108, F.Cu at (162.5, 45.0)
- added U2: ISO1540, Package_SO:SOIC-8_3.9x4.9mm_P1.27mm, F.Cu at (135.0, 36.0)
- added U9: SI8663BB-B-IS1, CM4IO:SI8663BB-B-IS1, F.Cu at (135.0, 14.5)
- moved PS1 9.01 mm to (132.5, 26.5)
