File: audio/audio.kicad_pcb (KiCad board)
At the start: 4 copper layers, 175 x 75 mm, 132 parts, among them J1 HDMI, J10 Conn_01x10, J11 MIC1, J12 MIC2, J13 MIC3, J14 MIC4, J2 JK00177, J3 USB3_A, J4 1054500101, J5 1054500101, J6 Conn_01x10, J7 Conn_01x10, J8 Conn_01x10, J9 Conn_01x10, Q1 DMG1012T, U1 RT9742SNGV, U10 ac108, U11 TCR3RM33, U12 TCR3RM33, U2 ISO1540, U3 VL805, U4 AP22653W6, U5 TPD4EUSB30, U6 TPD4EUSB30, U7 TPD4EUSB30, U8 AP3402, U9 SI8663BB-B-IS1, Y1 25MHz

Commit message: .
.
Other:
- outline, holes or cut-outs redrawn
Changed lines of the file:
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@@
   (gr_line (start 257.75 -1.5) (end 250.75 -8.5) (layer "F.SilkS") (width 0.15))
   (gr_line (start 100 0) (end 175 0) (layer "Edge.Cuts") (width 0.15))
-  (gr_line (start 75 0.25) (end 75 75) (layer "Edge.Cuts") (width 0.1))
-  (gr_line (start 75 0.25) (end 100 0.25) (layer "Edge.Cuts") (width 0.1))
-  (gr_line (start 100 28) (end 100 0.25) (layer "Edge.Cuts") (width 0.15))
+  (gr_line (start 75 0) (end 75 74.75) (layer "Edge.Cuts") (width 0.1))
+  (gr_line (start 100 28) (end 100 0) (layer "Edge.Cuts") (width 0.15))
   (gr_line (start 100 28) (end 118 28) (layer "Edge.Cuts") (width 0.15))
   (gr_line (start 118 46) (end 135 46) (layer "Edge.Cuts") (width 0.15))
   (gr_line (start 0 75) (end 0 0) (layer "Edge.Cuts") (width 0.1))
-  (gr_line (start 75 0) (end 100 0) (layer "Edge.Cuts") (width 0.1))
   (gr_line (start 175 0) (end 175 75) (layer "Edge.Cuts") (width 0.15))
   (gr_line (start 75 0) (end 0 0) (layer "Edge.Cuts") (width 0.1))

Commit message: .
.
Parts:
- added C58: 1uF, Capacitor_SMD:C_0402_1005Metric, F.Cu at (114.3, 19.7)
- added C59: 0.1uF, Capacitor_SMD:C_0402_1005Metric, F.Cu at (115.5, 15.2)
- added C60: 10uF, Capacitor_SMD:C_0402_1005Metric, F.Cu at (107.4, 22.8)
- added C61: 0.1uF, Capacitor_SMD:C_0402_1005Metric, F.Cu at (111.4, 21.7)
- added C62: 0.1uF, Capacitor_SMD:C_0402_1005Metric, F.Cu at (114.3, 17.7)
- added C63: 10uF, Capacitor_SMD:C_0402_1005Metric, F.Cu at (119.5, 12.7)
- added C64: 0.1uF, Capacitor_SMD:C_0402_1005Metric, F.Cu at (121.2, 14.7)
- added C65: 0.1uF, Capacitor_SMD:C_0402_1005Metric, F.Cu at (118.3, 15.2)
- added C66: 0.1uF, Capacitor_SMD:C_0402_1005Metric, F.Cu at (122.3, 12.7)
- added C67: 1uF, Capacitor_SMD:C_0402_1005Metric, F.Cu at (114.3, 21.7)
- added C68: 10uF, Capacitor_SMD:C_0402_1005Metric, F.Cu at (117.2, 17.2)
- added C69: 0.1uF, Capacitor_SMD:C_0402_1005Metric, F.Cu at (111.4, 19.7)
- added C70: 10uF, Capacitor_SMD:C_0402_1005Metric, F.Cu at (111.4, 17.7)
- added C71: 0.1uF, Capacitor_SMD:C_0402_1005Metric, F.Cu at (117.2, 19.2)
- added R42: 0, Resistor_SMD:R_0603_1608Metric, F.Cu at (104.0, 15.5)
- added R43: 0, Resistor_SMD:R_0603_1608Metric, F.Cu at (112.0, 13.0)
- added R44: 0, Resistor_SMD:R_0603_1608Metric, F.Cu at (104.0, 13.0)
- added R45: 0, Resistor_SMD:R_0603_1608Metric, F.Cu at (108.0, 15.5)
- added R46: 1k, Resistor_SMD:R_0603_1608Metric, F.Cu at (108.0, 18.0)
- added R47: 1k, Resistor_SMD:R_0603_1608Metric, F.Cu at (108.0, 20.5)
- added R48: 1k, Resistor_SMD:R_0603_1608Metric, F.Cu at (104.0, 20.5)
- added R49: 1k, Resistor_SMD:R_0603_1608Metric, F.Cu at (104.0, 18.0)
- added R50: 0, Resistor_SMD:R_0603_1608Metric, F.Cu at (112.0, 15.5)
- added R51: 0, Resistor_SMD:R_0603_1608Metric, F.Cu at (108.0, 13.0)
- added R52: 0, Resistor_SMD:R_0603_1608Metric, F.Cu at (104.0, 23.0)
- added R53: 0, Resistor_SMD:R_0603_1608Metric, F.Cu at (116.0, 13.0)
Connections:
- PS1 pad 1: unconnected-(PS1-Pad1) -> /isolation_module/GND
- PS1 pad 11: unconnected-(PS1-Pad11) -> /4ch_mic/VDD_GND
- PS1 pad 12: unconnected-(PS1-Pad12) -> /4ch_mic/VDD_GND
- PS1 pad 13: unconnected-(PS1-Pad13) -> /4ch_mic/VDD_5V
- PS1 pad 14: unconnected-(PS1-Pad14) -> /4ch_mic/VDD_5V
- PS1 pad 15: unconnected-(PS1-Pad15) -> /4ch_mic/VDD_GND
- PS1 pad 16: unconnected-(PS1-Pad16) -> /4ch_mic/VDD_GND
- PS1 pad 2: unconnected-(PS1-Pad2) -> /isolation_module/GND
- PS1 pad 3: unconnected-(PS1-Pad3) -> /isolation_module/+5V
- PS1 pad 4: unconnected-(PS1-Pad4) -> /isolation_module/+5V
- PS1 pad 5: unconnected-(PS1-Pad5) -> /isolation_module/GND
- PS1 pad 6: unconnected-(PS1-Pad6) -> /isolation_module/GND
- PS1 pad 7: unconnected-(PS1-Pad7) -> /isolation_module/GND
- PS1 pad 8: unconnected-(PS1-Pad8) -> /isolation_module/GND
- PS1 pad 9: unconnected-(PS1-Pad9) -> /4ch_mic/VDD_GND
- PS2 pad 1: unconnected-(PS2-Pad1) -> /4ch_mic/VDD_GND
- PS2 pad 11: unconnected-(PS2-Pad11) -> /4ch_mic/AVCC_GND
- PS2 pad 12: unconnected-(PS2-Pad12) -> /4ch_mic/AVCC_GND
- PS2 pad 13: unconnected-(PS2-Pad13) -> /4ch_mic/AVCC_5V
- PS2 pad 14: unconnected-(PS2-Pad14) -> /4ch_mic/AVCC_5V
- PS2 pad 15: unconnected-(PS2-Pad15) -> /4ch_mic/AVCC_GND
- PS2 pad 16: unconnected-(PS2-Pad16) -> /4ch_mic/AVCC_GND
- PS2 pad 2: unconnected-(PS2-Pad2) -> /4ch_mic/VDD_GND
- PS2 pad 3: unconnected-(PS2-Pad3) -> /4ch_mic/VDD_5V
- PS2 pad 4: unconnected-(PS2-Pad4) -> /4ch_mic/VDD_5V
- PS2 pad 5: unconnected-(PS2-Pad5) -> /4ch_mic/VDD_GND
- PS2 pad 6: unconnected-(PS2-Pad6) -> /4ch_mic/VDD_GND
- PS2 pad 7: unconnected-(PS2-Pad7) -> /4ch_mic/VDD_GND
- PS2 pad 8: unconnected-(PS2-Pad8) -> /4ch_mic/VDD_GND
- PS2 pad 9: unconnected-(PS2-Pad9) -> /4ch_mic/AVCC_GND
- R30 pad 1: /4ch_mic/ISO_SDOUT -> /4ch_mic/ISO_ADC
- U10 pad 10: /4ch_mic/SDA -> /4ch_mic/ISO_SDA
- U10 pad 9: /4ch_mic/SCK -> /4ch_mic/ISO_SCK
- U2 pad 1: unconnected-(U2-Pad1) -> /isolation_module/3.3V
- U2 pad 2: unconnected-(U2-Pad2) -> /isolation_module/I2C1_SDA
- U2 pad 3: unconnected-(U2-Pad3) -> /isolation_module/I2C1_SCL
- U2 pad 4: unconnected-(U2-Pad4) -> /isolation_module/GND
- U2 pad 5: unconnected-(U2-Pad5) -> /4ch_mic/VDD_GND
- U2 pad 6: unconnected-(U2-Pad6) -> /4ch_mic/ISO_SCK
- U2 pad 7: unconnected-(U2-Pad7) -> /4ch_mic/ISO_SDA
- U2 pad 8: unconnected-(U2-Pad8) -> /4ch_mic/VDD_3.3V
- U9 pad 1: unconnected-(U9-Pad1) -> /isolation_module/3.3V
- U9 pad 10: unconnected-(U9-Pad10) -> /4ch_mic/ISO_ADC
- U9 pad 11: unconnected-(U9-Pad11) -> /isolation_module/ISO_LRCK_TX
- U9 pad 12: unconnected-(U9-Pad12) -> /isolation_module/ISO_BCLK_TX
- U9 pad 13: unconnected-(U9-Pad13) -> /isolation_module/ISO_LRCK_RX
- U9 pad 14: unconnected-(U9-Pad14) -> /isolation_module/ISO_BCLK_RX
- U9 pad 16: unconnected-(U9-Pad16) -> /4ch_mic/VDD_3.3V
- U9 pad 3: unconnected-(U9-Pad3) -> /isolation_module/I2S_BCLK_TX
- U9 pad 4: unconnected-(U9-Pad4) -> /isolation_module/I2S_LRCK_TX
- U9 pad 5: unconnected-(U9-Pad5) -> /isolation_module/I2S_BCLK_RX
- U9 pad 6: unconnected-(U9-Pad6) -> /isolation_module/I2S_LRCK_RX
- U9 pad 7: unconnected-(U9-Pad7) -> /isolation_module/I2S_ADC
- U9 pad 8: unconnected-(U9-Pad8) -> /isolation_module/GND
- U9 pad 9: unconnected-(U9-Pad9) -> /4ch_mic/VDD_GND
Routing:
- net /CM4_docker1/CM4_LOW_SPEED/TRD2_N: track 162.8 -> 50.4 mm
- net /CM4_docker1/CM4_LOW_SPEED/TRD0_N: track 0.00 -> 112.5 mm
Other:
- outline, holes or cut-outs redrawn

Commit message: .
.
Routing:
- net GND: track 76.7 -> 0.00 mm
- net /CM4_docker1/I2S_BCLK: track 50.4 -> 0.00 mm
- net /CM4_docker1/CM4_HIGH_SPEED/HDMI0_CK_P: track 0.00 -> 30.2 mm
- net /CM4_docker1/CM4_HIGH_SPEED/HDMI0_CK_N: track 0.00 -> 30.2 mm
- net /CM4_docker1/CM4_HIGH_SPEED/HDMI0_D0_N: track 0.00 -> 30.1 mm
- net /CM4_docker1/CM4_HIGH_SPEED/HDMI0_D0_P: track 0.00 -> 30.1 mm
- net /CM4_docker1/CM4_HIGH_SPEED/HDMI0_D1_N: track 0.00 -> 30.0 mm
- net /CM4_docker1/CM4_HIGH_SPEED/HDMI0_D2_N: track 25.3 -> 29.8 mm
- net /CM4_docker1/CM4_HIGH_SPEED/HDMI0_D2_P: track 25.4 -> 29.8 mm
- net /CM4_docker1/CM4_HIGH_SPEED/HDMI0_D1_P: track 25.6 -> 30.0 mm
Changed lines of the file:
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@@
 (kicad_pcb (version 20211014) (generator pcbnew)
   (general
-    (thickness 1.6)
+    (thickness 1.608)
   )
   (paper "A4")
@@
       (layer "F.SilkS" (type "Top Silk Screen"))
       (layer "F.Paste" (type "Top Solder Paste"))
-      (layer "F.Mask" (type "Top Solder Mask") (thickness 0.01))
-      (layer "F.Cu" (type "copper") (thickness 0.035))
-      (layer "dielectric 1" (type "core") (thickness 0.48) (material "FR4") (epsilon_r 4.5) (loss_tangent 0.02))
-      (layer "In1.Cu" (type "copper") (thickness 0.035))
-      (layer "dielectric 2" (type "prepreg") (thickness 0.48) (material "FR4") (epsilon_r 4.5) (loss_tangent 0.02))
-      (layer "In2.Cu" (type "copper") (thickness 0.035))
-      (layer "dielectric 3" (type "core") (thickness 0.48) (material "FR4") (epsilon_r 4.5) (loss_tangent 0.02))
-      (layer "B.Cu" (type "copper") (thickness 0.035))
-      (layer "B.Mask" (type "Bottom Solder Mask") (thickness 0.01))
+      (layer "F.Mask" (type "Top Solder Mask") (thickness 0.012))
+      (layer "F.Cu" (type "copper") (thickness 0.04))
+      (layer "dielectric 1" (type "prepreg") (thickness 0.2) (material "FR4") (epsilon_r 4.18) (loss_tangent 0.02))
+      (layer "In1.Cu" (type "copper") (thickness 0.032))
+      (layer "dielectric 2" (type "core") (thickness 1.04) (material "FR4") (epsilon_r 4.3) (loss_tangent 0.02))
+      (layer "In2.Cu" (type "copper") (thickness 0.032))
+      (layer "dielectric 3" (type "prepreg") (thickness 0.2) (material "FR4") (epsilon_r 4.18) (loss_tangent 0.02))
+      (layer "B.Cu" (type "copper") (thickness 0.04))
+      (layer "B.Mask" (type "Bottom Solder Mask") (thickness 0.012))
       (layer "B.Paste" (type "Bottom Solder Paste"))
       (layer "B.SilkS" (type "Bottom Silk Screen"))
       (copper_finish "None")
-      (dielectric_constraints no)
+      (dielectric_constraints yes)
     )
     (pad_to_mask_clearance 0)
@@
   (via (at 3.5 71.5) (size 5) (drill 3.2) (layers "F.Cu" "B.Cu") (free) (net 0))
   (via (at 171.5 3.5) (size 5) (drill 3.2) (layers "F.Cu" "B.Cu") (free) (net 0))
-  (segment (start 34.42 26.17) (end 32.674314 26.17) (width 0.2) (layer "F.Cu") (net 46))
-  (segment (start 34.42 25.77) (end 32.84 25.77) (width 0.2) (layer "F.Cu") (net 46))
-  (segment (start 24.064314 17.56) (end 12.89 17.56) (width 0.2) (layer "F.Cu") (net 46))
-  (segment (start 32.84 25.77) (end 24.23 17.16) (width 0.2) (layer "F.Cu") (net 46))
-  (segment (start 32.674314 26.17) (end 24.064314 17.56) (width 0.2) (layer "F.Cu") (net 46))
-  (segment (start 24.23 17.16) (end 12.724315 17.16) (width 0.2) (layer "F.Cu") (net 46))
-  (segment (start 31.564314 29.77) (end 23.924314 22.13) (width 0.2) (layer "F.Cu") (net 134))
-  (segment (start 34.42 29.77) (end 31.564314 29.77) (width 0.2) (layer "F.Cu") (net 134))
-  (segment (start 23.924314 22.13) (end 12.21 22.13) (width 0.2) (layer "F.Cu") (net 134))
-  (segment (start 24.09 21.73) (end 12.241 21.73) (width 0.2) (layer "F.Cu") (net 136))
-  (segment (start 31.73 29.37) (end 24.09 21.73) (width 0.2) (layer "F.Cu") (net 136))
-  (segment (start 34.42 29.37) (end 31.73 29.37) (width 0.2) (layer "F.Cu") (net 136))
-  (segment (start 24.074314 20.62) (end 12.065315 20.62) (width 0.2) (layer "F.Cu") (net 138))
-  (segment (start 34.42 28.57) (end 32.024314 28.57) (width 0.2) (layer "F.Cu") (net 138))
-  (segment (start 32.024314 28.57) (end 24.074314 20.62) (width 0.2) (layer "F.Cu") (net 138))
-  (segment (start 32.19 28.17) (end 24.24 20.22) (width 0.2) (layer "F.Cu") (net 156))
-  (segment (start 34.42 28.17) (end 32.19 28.17) (width 0.2) (layer "F.Cu") (net 156))
-  (segment (start 24.24 20.22) (end 12.231 20.22) (width 0.2) (layer "F.Cu") (net 156))
-  (segment (start 32.66 26.97) (end 24.42 18.73) (width 0.2) (layer "F.Cu") (net 156))
-  (segment (start 32.494314 27.37) (end 24.254314 19.13) (width 0.2) (layer "F.Cu") (net 156))
-  (segment (start 24.254314 19.13) (end 12.221 19.13) (width 0.2) (layer "F.Cu") (net 156))
-  (segment (start 24.42 18.73) (end 12.241 18.73) (width 0.2) (layer "F.Cu") (net 156))
-  (segment (start 34.42 27.37) (end 32.494314 27.37) (width 0.2) (layer "F.Cu") (net 156))
-  (segment (start 34.42 26.97) (end 32.66 26.97) (width 0.2) (layer "F.Cu") (net 156))
+  (segment (start 11.978501 22.5925) (end 10.0285 22.5925) (width 0.15) (layer "F.Cu") (net 134))
+  (segment (start 35.634999 30.8) (end 35.569999 30.735) (width 0.15) (layer "F.Cu") (net 134))
+  (segment (start 35.569999 30.735) (end 30.50408 30.735) (width 0.15) (layer "F.Cu") (net 134))
+  (segment (start 21.99658 22.2275) (end 12.343501 22.2275) (width 0.15) (layer "F.Cu") (net 134))
+  (segment (start 12.343501 22.2275) (end 11.978501 22.5925) (width 0.15) (layer "F.Cu") (net 134))
+  (segment (start 36.16 30.8) (end 35.634999 30.8) (width 0.15) (layer "F.Cu") (net 134))
+  (segment (start 30.50408 30.735) (end 21.99658 22.2275) (width 0.15) (layer "F.Cu") (net 134))
+  (segment (start 11.978501 21.5925) (end 10.0285 21.5925) (width 0.15) (layer "F.Cu") (net 136))
+  (segment (start 22.10842 21.9575) (end 12.343501 21.9575) (width 0.15) (layer "F.Cu") (net 136))
+  (segment (start 30.61592 30.465) (end 22.10842 21.9575) (width 0.15) (layer "F.Cu") (net 136))
+  (segment (start 36.16 30.4) (end 35.634999 30.4) (width 0.15) (layer "F.Cu") (net 136))
+  (segment (start 35.569999 30.465) (end 30.61592 30.465) (width 0.15) (layer "F.Cu") (net 136))
+  (segment (start 35.634999 30.4) (end 35.569999 30.465) (width 0.15) (layer "F.Cu") (net 136))
+  (segment (start 12.343501 21.9575) (end 11.978501 21.5925) (width 0.15) (layer "F.Cu") (net 136))
+  (segment (start 12.343501 20.7275) (end 22.61658 20.7275) (width 0.15) (layer "F.Cu") (net 138))
+  (segment (start 22.61658 20.7275) (end 31.42408 29.535) (width 0.15) (layer "F.Cu") (net 138))
+  (segment (start 31.42408 29.535) (end 35.569999 29.535) (width 0.15) (layer "F.Cu") (net 138))
+  (segment (start 11.978501 21.0925) (end 12.343501 20.7275) (width 0.15) (layer "F.Cu") (net 138))
+  (segment (start 35.634999 29.6) (end 36.16 29.6) (width 0.15) (layer "F.Cu") (net 138))
+  (segment (start 35.569999 29.535) (end 35.634999 29.6) (width 0.15) (layer "F.Cu") (net 138))
+  (segment (start 10.0285 21.0925) (end 11.978501 21.0925) (width 0.15) (layer "F.Cu") (net 138))
+  (segment (start 35.634999 29.2) (end 36.16 29.2) (width 0.15) (layer "F.Cu") (net 140))
+  (segment (start 35.569999 29.265) (end 35.634999 29.2) (width 0.15) (layer "F.Cu") (net 140))
+  (segment (start 31.53592 29.265) (end 35.569999 29.265) (width 0.15) (layer "F.Cu") (net 140))
+  (segment (start 10.0285 20.0925) (end 11.978501 20.0925) (width 0.15) (layer "F.Cu") (net 140))
+  (segment (start 11.978501 20.0925) (end 12.343501 20.4575) (width 0.15) (layer "F.Cu") (net 140))
+  (segment (start 22.72842 20.4575) (end 31.53592 29.265) (width 0.15) (layer "F.Cu") (net 140))
+  (segment (start 12.343501 20.4575) (end 22.72842 20.4575) (width 0.15) (layer "F.Cu") (net 140))
+  (segment (start 36.16 28.4) (end 35.634999 28.4) (width 0.15) (layer "F.Cu") (net 143))
+  (segment (start 32.28408 28.335) (end 23.17658 19.2275) (width 0.15) (layer "F.Cu") (net 143))
+  (segment (start 35.569999 28.335) (end 32.28408 28.335) (width 0.15) (layer "F.Cu") (net 143))
+  (segment (start 23.17658 19.2275) (end 12.343501 19.2275) (width 0.15) (layer "F.Cu") (net 143))
+  (segment (start 11.978501 19.5925) (end 10.0285 19.5925) (width 0.15) (layer "F.Cu") (net 143))
+  (segment (start 12.343501 19.2275) (end 11.978501 19.5925) (width 0.15) (layer "F.Cu") (net 143))
+  (segment (start 35.634999 28.4) (end 35.569999 28.335) (width 0.15) (layer "F.Cu") (net 143))
+  (segment (start 32.39592 28.065) (end 23.28842 18.9575) (width 0.15) (layer "F.Cu") (net 145))
+  (segment (start 35.569999 28.065) (end 32.39592 28.065) (width 0.15) (layer "F.Cu") (net 145))
+  (segment (start 35.634999 28) (end 35.569999 28.065) (width 0.15) (layer "F.Cu") (net 145))
+  (segment (start 12.343501 18.9575) (end 11.978501 18.5925) (width 0.15) (layer "F.Cu") (net 145))
+  (segment (start 11.978501 18.5925) (end 10.0285 18.5925) (width 0.15) (layer "F.Cu") (net 145))
+  (segment (start 36.16 28) (end 35.634999 28) (width 0.15) (layer "F.Cu") (net 145))
+  (segment (start 23.28842 18.9575) (end 12.343501 18.9575) (width 0.15) (layer "F.Cu") (net 145))
+  (segment (start 32.88408 27.135) (end 23.47658 17.7275) (width 0.15) (layer "F.Cu") (net 147))
+  (segment (start 35.634999 27.2) (end 35.569999 27.135) (width 0.15) (layer "F.Cu") (net 147))
+  (segment (start 36.16 27.2) (end 35.634999 27.2) (width 0.15) (layer "F.Cu") (net 147))
+  (segment (start 12.343501 17.7275) (end 11.978501 18.0925) (width 0.15) (layer "F.Cu") (net 147))
+  (segment (start 35.569999 27.135) (end 32.88408 27.135) (width 0.15) (layer "F.Cu") (net 147))
+  (segment (start 23.47658 17.7275) (end 12.343501 17.7275) (width 0.15) (layer "F.Cu") (net 147))
+  (segment (start 11.978501 18.0925) (end 10.0285 18.0925) (width 0.15) (layer "F.Cu") (net 147))
+  (segment (start 23.58842 17.4575) (end 12.343501 17.4575) (width 0.15) (layer "F.Cu") (net 149))
+  (segment (start 36.16 26.8) (end 35.634999 26.8) (width 0.15) (layer "F.Cu") (net 149))
+  (segment (start 32.99592 26.865) (end 23.58842 17.4575) (width 0.15) (layer "F.Cu") (net 149))
+  (segment (start 12.343501 17.4575) (end 11.978501 17.0925) (width 0.15) (layer "F.Cu") (net 149))
+  (segment (start 35.634999 26.8) (end 35.569999 26.865) (width 0.15) (layer "F.Cu") (net 149))
+  (segment (start 11.978501 17.0925) (end 10.0285 17.0925) (width 0.15) (layer "F.Cu") (net 149))
+  (segment (start 35.569999 26.865) (end 32.99592 26.865) (width 0.15) (layer "F.Cu") (net 149))
   (segment (start 14.9 33.67) (end 15.75 34.52) (width 0.127) (layer "F.Cu") (net 165))
   (segment (start 15.75 34.52) (end 16.58 34.52) (width 0.127) (layer "F.Cu") (net 165))

Commit message: high_speed_artwork_done
.
Parts:
- moved R4 56.1 mm to (47.0, -8.30)
- moved Q1 56.1 mm to (41.3, -8.25)
- moved R3 56.1 mm to (44.5, -8.33)
- moved C20 27.4 mm to (71.7, -6.83)
- moved C25 27.4 mm to (66.7, -6.83)
- moved C18 27.4 mm to (61.7, -7.33)
- moved C3 27.4 mm to (57.2, -7.33)
- moved R19 26.0 mm to (80.4, -7.87)
- moved R20 26.0 mm to (77.5, -7.87)
- moved R21 26.0 mm to (77.5, -5.88)
- moved R22 26.0 mm to (80.4, -5.88)
- moved U1 21.7 mm to (28.4, -2.54)
- moved C2 9.00 mm to (24.6, 8.35)
- moved C1 9.00 mm to (24.6, 6.38)
- moved R5 8.61 mm to (41.1, 7.13)
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Connections:
- U7 pad 1: Net-(U7-Pad1) -> /CM4_docker1/CM4_LOW_SPEED/USB2_P
- U7 pad 10: Net-(U7-Pad1) -> /CM4_docker1/CM4_LOW_SPEED/USB2_P
- U7 pad 2: Net-(U7-Pad2) -> /CM4_docker1/CM4_LOW_SPEED/USB2_N
- U7 pad 4: /CM4_docker1/CM4_LOW_SPEED/USBD_N -> /CM4_docker1/CM4_LOW_SPEED/USB2_P
- U7 pad 5: /CM4_docker1/CM4_LOW_SPEED/USBD_P -> /CM4_docker1/CM4_LOW_SPEED/USB2_N
- U7 pad 6: /CM4_docker1/CM4_LOW_SPEED/USBD_P -> /CM4_docker1/CM4_LOW_SPEED/USB2_N
- U7 pad 7: /CM4_docker1/CM4_LOW_SPEED/USBD_N -> /CM4_docker1/CM4_LOW_SPEED/USB2_P
- U7 pad 9: Net-(U7-Pad2) -> /CM4_docker1/CM4_LOW_SPEED/USB2_N
Routing:
- net /CM4_docker1/CM4_LOW_SPEED/USB2_P: track 0.00 -> 58.5 mm
- net /CM4_docker1/CM4_LOW_SPEED/USB2_N: track 0.00 -> 58.5 mm
- net /CM4_docker1/CM4_LOW_SPEED/TRD0_N: track 112.5 -> 56.0 mm
- net /CM4_docker1/CM4_LOW_SPEED/TRD0_P: track 0.00 -> 55.9 mm
- net /CM4_docker1/I2S_LRCK: track 0.00 -> 52.9 mm
- net /CM4_docker1/I2S_ADC: track 0.00 -> 49.7 mm, vias 0 -> 2
- net /CM4_docker1/I2S_BCLK: track 0.00 -> 48.3 mm, vias 0 -> 2
- net /CM4_docker1/CM4_HIGH_SPEED/HDMI0_HOTPLUG: track 0.00 -> 45.1 mm
- net /CM4_docker1/CM4_HIGH_SPEED/HDMI0_CEC: track 0.00 -> 42.1 mm, vias 0 -> 2
- net /CM4_docker1/CM4_HIGH_SPEED/HDMI0_SDA: track 0.00 -> 33.7 mm
- net /CM4_docker1/CM4_HIGH_SPEED/HDMI0_SCL: track 0.00 -> 32.1 mm
- net /CM4_docker1/xHCI-USB3/PD2_N: track 0.00 -> 24.0 mm, vias 0 -> 1
- net /CM4_docker1/xHCI-USB3/PD2_P: track 0.00 -> 24.0 mm, vias 0 -> 1
- net /CM4_docker1/CM4_HIGH_SPEED/PCIE_TX_P: track 0.00 -> 19.2 mm
- net /CM4_docker1/CM4_HIGH_SPEED/PCIE_TX_N: track 0.00 -> 19.2 mm
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Other:
- board text added: "Board thickness : 1.608mm Finished copper weight inners : 1oz Finished copper weight outers : 1/2oz Material type : FR4 Board to : UL94-V0 TG >=130 50R trace width 0.355mm 90R diff pair width 0.170 spacing 0.100mm 100R diff pair width 0.150 spacing 0.120mm"
- board text removed: "Board thickness : 1.56mm Finished copper weight inners : 1oz Finished copper weight outers : 1oz Board finish : OSP Material type : FR4 Colour of solder resists : Green Colour of silk screens : White Only on the top side Board to : UL94-V0 TG >=130 50R trace width 0.13mm@ 3GHz 90R diff pair width 0.147 spacing 0.253mm @ 2.5GHz 100R diff pair width 0.127 spacing 0.253mm @ 2GHz"

Commit message: .
.
Parts:
- moved R11 56.7 mm to (-10.3, 57.4)
- moved C39 56.7 mm to (-8.40, 57.4)
- moved R10 56.7 mm to (-12.3, 57.3)
- moved R9 33.0 mm to (-8.64, 44.6)
- moved R8 33.0 mm to (-5.59, 44.5)
- moved R13 19.0 mm to (3.61, -16.2)
- moved R12 19.0 mm to (0.58, -14.4)
- moved R14 19.0 mm to (3.49, -14.4)
- moved R15 19.0 mm to (0.58, -16.4)
- moved R16 19.0 mm to (0.41, -11.8)
- moved R17 19.0 mm to (3.20, -9.89)
- moved R18 19.0 mm to (3.37, -11.9)
- moved C2 17.8 mm to (24.1, -9.46)
- moved U4 17.8 mm to (24.9, -14.8)
- moved C1 17.8 mm to (24.1, -11.4)
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Connections:
- net Net-(C11-Pad1) renamed /CM4_docker1/xHCI-USB3/clock1
- net Net-(C12-Pad1) renamed /CM4_docker1/xHCI-USB3/SW_OUT
- net Net-(C12-Pad2) renamed /CM4_docker1/xHCI-USB3/FB
- net Net-(C16-Pad1) renamed /CM4_docker1/xHCI-USB3/clock2
- net Net-(L2-Pad1) renamed /CM4_docker1/xHCI-USB3/LX
- net Net-(R1-Pad2) renamed /CM4_docker1/xHCI-USB3/EN
- J10 pad 10: /CM4_docker1/SD_CLK -> /CM4_docker1/SD_DAT0
- J10 pad 5: /CM4_docker1/SD_DAT3 -> /CM4_docker1/SD_CMD
- J10 pad 6: /CM4_docker1/SD_DAT2 -> /CM4_docker1/SD_CLK
- J10 pad 7: /CM4_docker1/SD_DAT1 -> /CM4_docker1/SD_DAT3
- J10 pad 8: /CM4_docker1/SD_DAT0 -> /CM4_docker1/SD_DAT2
- J10 pad 9: /CM4_docker1/SD_CMD -> /CM4_docker1/SD_DAT1
- U8 pad 5: unconnected-(U8-Pad5) -> /CM4_docker1/xHCI-USB3/PG
Routing:
- net /CM4_docker1/I2C1_SDA: track 0.00 -> 45.4 mm, vias 0 -> 2
- net /CM4_docker1/I2C1_SCL: track 0.00 -> 43.7 mm, vias 0 -> 2
- net /CM4_docker1/SD_CMD: track 0.00 -> 41.3 mm, vias 0 -> 2
- net /CM4_docker1/SD_DAT1: track 0.00 -> 40.3 mm, vias 0 -> 2
- net /CM4_docker1/SD_DAT2: track 0.00 -> 39.4 mm, vias 0 -> 2
- net /CM4_docker1/SD_CLK: track 0.00 -> 38.7 mm
- net /CM4_docker1/SD_DAT3: track 0.00 -> 38.7 mm
- net /CM4_docker1/SD_DAT0: track 0.00 -> 36.4 mm
- net /CM4_docker1/xHCI-USB3/clock1: track 0.00 -> 7.69 mm
- net /CM4_docker1/xHCI-USB3/clock2: track 0.00 -> 5.41 mm
- net /CM4_docker1/xHCI-USB3/FB: track 0.00 -> 5.31 mm
- net /CM4_docker1/xHCI-USB3/EN: track 0.00 -> 4.93 mm
- net /CM4_docker1/xHCI-USB3/SW_OUT: track 0.00 -> 4.34 mm
- net /CM4_docker1/CM4_HIGH_SPEED/PCIE_CLK_N: track 18.3 -> 18.8 mm
- net /CM4_docker1/CM4_HIGH_SPEED/PCIE_CLK_P: track 18.2 -> 18.8 mm
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- added copper zone on F.Cu, net /CM4_docker1/+5V
- added copper zone on F.Cu, net /CM4_docker1/xHCI-USB3/LX
- added copper zone on F.Cu, net /CM4_docker1/xHCI-USB3/SW_OUT
