File: audio/audio.kicad_pcb (KiCad board)
At the start: 4 copper layers, 175 x 75 mm, 158 parts, among them J1 HDMI, J10 Conn_01x10, J11 MIC1, J12 MIC2, J13 MIC3, J14 MIC4, J2 JK00177, J3 USB3_A, J4 1054500101, J5 1054500101, J6 Conn_01x10, J7 Conn_01x10, J8 Conn_01x10, J9 Conn_01x10, Q1 DMG1012T, U1 RT9742SNGV, U10 ac108, U11 TCR3RM33, U12 TCR3RM33, U2 ISO1540, U3 VL805, U4 AP22653W6, U5 TPD4EUSB30, U6 TPD4EUSB30, U7 TPD4EUSB30, U8 AP3402, U9 SI8663BB-B-IS1, Y1 25MHz

Commit message: .
.
Parts:
- moved C4 63.9 mm to (13.3, 26.1), turned to -90 degrees
- moved C13 62.8 mm to (22.5, 25.4), turned to -90 degrees
- moved L1 62.5 mm to (15.9, 25.2), turned to 0 degrees
- moved C15 62.4 mm to (23.6, 25.4), turned to -90 degrees
- moved C19 60.1 mm to (23.6, 27.5)
- moved C8 59.4 mm to (18.6, 26.2), turned to -90 degrees
- moved C9 58.8 mm to (20.3, 25.4), turned to -90 degrees
- moved C27 58.3 mm to (20.3, 27.5)
- moved C23 58.3 mm to (21.4, 27.5)
- moved C22 58.2 mm to (22.5, 27.5)
- moved C10 58.0 mm to (21.4, 25.4), turned to -90 degrees
- moved C31 52.2 mm to (28.2, 34.1)
- moved C29 49.9 mm to (18.2, 36.9)
- moved C28 48.7 mm to (23.7, 34.6), turned to 0 degrees
- moved C34 44.8 mm to (18.3, 40.0), turned to 180 degrees
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Routing:
- net /CM4_docker1/xHCI-USB3/FB: track 5.31 -> 7.46 mm
- net /CM4_docker1/xHCI-USB3/EN: track 4.93 -> 6.01 mm
- net /CM4_docker1/xHCI-USB3/SW_OUT: track 4.34 -> 5.38 mm
- added copper zone on F.Cu, net /CM4_docker1/3.3V
- added copper zone on F.Cu, net /CM4_docker1/xHCI-USB3/A3.3v

Commit message: .
.
Parts:
- moved R17 118.9 mm to (117.8, 22.0)
- moved R10 47.0 mm to (34.2, 64.3)
- moved R11 43.9 mm to (33.0, 64.3), turned to -90 degrees
- moved C39 42.4 mm to (33.0, 66.6), turned to -90 degrees
- moved C20 37.8 mm to (36.8, 7.50), turned to 90 degrees
- moved C25 35.3 mm to (34.5, 7.50), turned to 90 degrees
- moved C3 32.8 mm to (25.8, 2.10), turned to 0 degrees
- moved R4 32.2 mm to (20.8, 10.2)
- moved R3 31.2 mm to (19.5, 10.2)
- moved C18 27.1 mm to (39.1, 7.50), turned to 90 degrees
- moved Q1 26.4 mm to (22.5, 10.2), turned to 90 degrees
- moved C1 26.2 mm to (6.00, 7.50), turned to -90 degrees
- moved C10 23.3 mm to (25.8, 48.3)
- moved C9 22.9 mm to (22.2, 48.3)
- moved U1 21.8 mm to (8.50, 6.50), turned to 90 degrees
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Connections:
- net Net-(C39-Pad1) renamed /CM4_docker1/CM4_LOW_SPEED/MXCT
- net Net-(J2-Pad14) renamed /CM4_docker1/CM4_LOW_SPEED/LED_GREEN
- net Net-(J2-Pad15) renamed /CM4_docker1/CM4_LOW_SPEED/LED_YELLOW
- net Net-(R5-Pad1) renamed /CM4_docker1/xHCI-USB3/ILIM
- J5 pad A1: /CM4_docker1/+5V -> GND
- J5 pad A12: /CM4_docker1/+5V -> GND
- J5 pad A4: GND -> /CM4_docker1/+5V
- J5 pad A9: GND -> /CM4_docker1/+5V
- J5 pad B1: /CM4_docker1/+5V -> GND
- J5 pad B12: /CM4_docker1/+5V -> GND
- J5 pad B4: GND -> /CM4_docker1/+5V
- J5 pad B9: GND -> /CM4_docker1/+5V
- J5 pad S1: /CM4_docker1/+5V -> GND
- J5 pad S2: /CM4_docker1/+5V -> GND
- J5 pad S3: /CM4_docker1/+5V -> GND
- J5 pad S4: /CM4_docker1/+5V -> GND
- R19 pad 1: GND -> /CM4_docker1/+5V
- R20 pad 2: /CM4_docker1/+5V -> GND
- R21 pad 1: GND -> /CM4_docker1/+5V
- R22 pad 2: /CM4_docker1/+5V -> GND
Routing:
- net /CM4_docker1/CM4_LOW_SPEED/MXCT: track 0.00 -> 24.0 mm
- net /CM4_docker1/xHCI-USB3/A1.05v: track 0.00 -> 9.64 mm
- net /CM4_docker1/xHCI-USB3/A3.3v: track 0.03 -> 7.19 mm, vias 0 -> 2
- net /CM4_docker1/CM4_HIGH_SPEED/PCIE_CLK_P: track 18.8 -> 12.0 mm
- net /CM4_docker1/CM4_HIGH_SPEED/PCIE_TX_P: track 19.2 -> 12.8 mm
- net /CM4_docker1/CM4_HIGH_SPEED/PCIE_TX_N: track 19.2 -> 12.8 mm
- net /CM4_docker1/CM4_HIGH_SPEED/PCIE_CLK_N: track 18.8 -> 12.8 mm
- net /CM4_docker1/xHCI-USB3/PD1_P: track 7.99 -> 13.0 mm, vias 2 -> 1
- net /CM4_docker1/xHCI-USB3/PD1_N: track 8.43 -> 13.1 mm, vias 2 -> 1
- net /CM4_docker1/xHCI-USB3/C2_N: track 3.26 -> 7.84 mm
- net /CM4_docker1/CM4_HIGH_SPEED/PCIE_RX_N: track 8.81 -> 4.40 mm
- net /CM4_docker1/xHCI-USB3/C2_P: track 4.05 -> 8.28 mm
- net /CM4_docker1/CM4_HIGH_SPEED/PCIE_RX_P: track 8.81 -> 4.85 mm
- net /CM4_docker1/xHCI-USB3/PEXTX_P: track 8.14 -> 4.60 mm
- net /CM4_docker1/xHCI-USB3/SSRX1_N: track 7.15 -> 10.3 mm
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- added copper zone on F.Cu, net /CM4_docker1/xHCI-USB3/A1.05v

Commit message: .
.
Parts:
- added C72: 100n, Capacitor_SMD:C_0402_1005Metric, F.Cu at (27.2, 44.9)
- moved C7 29.3 mm to (36.8, 69.8), turned to 90 degrees
- moved R1 25.5 mm to (33.6, 73.8)
- moved R2 23.2 mm to (33.6, 72.6), turned to 180 degrees
- moved U8 22.4 mm to (33.3, 70.0), turned to 0 degrees
- moved R11 18.8 mm to (32.8, 45.5), turned to 0 degrees
- moved R10 17.7 mm to (32.8, 46.7), turned to 0 degrees
- moved C24 16.9 mm to (13.2, 70.7), turned to 90 degrees
- moved C12 15.5 mm to (29.3, 69.2), turned to 90 degrees
- moved R6 12.8 mm to (27.7, 68.8), turned to 0 degrees
- moved L2 12.4 mm to (27.8, 71.7), turned to 180 degrees
- moved C26 12.4 mm to (15.5, 70.7), turned to 90 degrees
- moved R7 11.6 mm to (26.2, 69.2), turned to -90 degrees
- moved L3 7.05 mm to (18.2, 71.5), turned to 180 degrees
- moved C3 6.11 mm to (30.5, 6.00)
- moved R5 6.10 mm to (23.8, 6.00), turned to -90 degrees
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Connections:
- CM4_MODULE1 pad 103: /CM4_docker1/CM4_LOW_SPEED/USB2_N -> /CM4_docker1/USB_DEBUG_N
- CM4_MODULE1 pad 105: /CM4_docker1/CM4_LOW_SPEED/USB2_P -> /CM4_docker1/USB_DEBUG_P
- J10 pad 2: GND -> /CM4_docker1/+5V
- J10 pad 3: /CM4_docker1/3.3V -> GND
- J2 pad 13: /CM4_docker1/CM4_LOW_SPEED/+3.3v -> /CM4_docker1/3.3V
- J2 pad 16: /CM4_docker1/CM4_LOW_SPEED/+3.3v -> /CM4_docker1/3.3V
- J4 pad A6: /CM4_docker1/CM4_LOW_SPEED/USB2_P -> /CM4_docker1/USB_DEBUG_P
- J4 pad A7: /CM4_docker1/CM4_LOW_SPEED/USB2_N -> /CM4_docker1/USB_DEBUG_N
- J4 pad B6: /CM4_docker1/CM4_LOW_SPEED/USB2_P -> /CM4_docker1/USB_DEBUG_P
- J4 pad B7: /CM4_docker1/CM4_LOW_SPEED/USB2_N -> /CM4_docker1/USB_DEBUG_N
- J6 pad 1: /CM4_docker1/+5V -> /CM4_docker1/USB_DEBUG_N
- J6 pad 2: /CM4_docker1/+5V -> /CM4_docker1/USB_DEBUG_P
- J6 pad 3: /CM4_docker1/3.3V -> GND
- J7 pad 1: GND -> /CM4_docker1/+5V
- J7 pad 10: GND -> /CM4_docker1/3.3V
- J7 pad 2: GND -> /CM4_docker1/+5V
- J7 pad 3: GND -> /CM4_docker1/+5V
- J7 pad 4: GND -> /CM4_docker1/+5V
- U7 pad 1: /CM4_docker1/CM4_LOW_SPEED/USB2_P -> /CM4_docker1/USB_DEBUG_P
- U7 pad 10: /CM4_docker1/CM4_LOW_SPEED/USB2_P -> /CM4_docker1/USB_DEBUG_P
- U7 pad 2: /CM4_docker1/CM4_LOW_SPEED/USB2_N -> /CM4_docker1/USB_DEBUG_N
- U7 pad 4: /CM4_docker1/CM4_LOW_SPEED/USB2_P -> /CM4_docker1/USB_DEBUG_P
- U7 pad 5: /CM4_docker1/CM4_LOW_SPEED/USB2_N -> /CM4_docker1/USB_DEBUG_N
- U7 pad 6: /CM4_docker1/CM4_LOW_SPEED/USB2_N -> /CM4_docker1/USB_DEBUG_N
- U7 pad 7: /CM4_docker1/CM4_LOW_SPEED/USB2_P -> /CM4_docker1/USB_DEBUG_P
- U7 pad 9: /CM4_docker1/CM4_LOW_SPEED/USB2_N -> /CM4_docker1/USB_DEBUG_N
Routing:
- net /CM4_docker1/3.3V: track 0.07 -> 144.3 mm, vias 0 -> 16
- net /CM4_docker1/USB_DEBUG_P: track 0.00 -> 84.4 mm, vias 0 -> 2
- net /CM4_docker1/USB_DEBUG_N: track 0.00 -> 82.3 mm, vias 0 -> 2
- net /CM4_docker1/+5V: track 0.00 -> 65.0 mm, vias 0 -> 54
- net /CM4_docker1/CM4_LOW_SPEED/USB2_P: track 59.2 -> 0.00 mm
- net /CM4_docker1/CM4_LOW_SPEED/USB2_N: track 59.2 -> 0.00 mm
- net /CM4_docker1/CM4_LOW_SPEED/LED_GREEN: track 0.00 -> 43.7 mm, vias 0 -> 1
- net /CM4_docker1/CM4_LOW_SPEED/ETH_LEDG: track 0.00 -> 42.9 mm, vias 0 -> 2
- net /CM4_docker1/CM4_LOW_SPEED/ETH_LEDY: track 0.00 -> 42.3 mm, vias 0 -> 2
- net /CM4_docker1/xHCI-USB3/A1.05v: track 9.64 -> 50.3 mm, vias 0 -> 20
- net GND: track 2.34 -> 21.0 mm, vias 0 -> 62
- net /CM4_docker1/POWER/CC2: track 0.00 -> 16.2 mm
- net /CM4_docker1/CM4_LOW_SPEED/LED_YELLOW: track 0.00 -> 11.8 mm, vias 0 -> 1
- net /CM4_docker1/POWER/CC1: track 0.00 -> 9.73 mm
- net /CM4_docker1/xHCI-USB3/A3.3v: track 7.19 -> 15.5 mm, vias 2 -> 9
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- added copper zone on B.Cu, net /CM4_docker1/+5V
- added copper zone on In1.Cu, net /CM4_docker1/+5V
- added copper zone on In2.Cu, net /CM4_docker1/xHCI-USB3/A1.05v
- added copper zone on B.Cu, net /CM4_docker1/xHCI-USB3/A3.3v
- added copper zone on B.Cu, net GND
- added copper zone on F.Cu, net GND
- added copper zone on In1.Cu, net GND
- added copper zone on In2.Cu, net GND
Other:
- outline, holes or cut-outs redrawn
