File: audio/audio.kicad_pcb (KiCad board)
At the start: 4 copper layers, 251 x 75 mm, 121 parts, among them J1 HDMI, J11 MIC1, J12 MIC2, J13 MIC3, J14 MIC4, J2 JK00177, J4 1054500101, J5 1054500101, J6 Conn_01x10, J7 Conn_01x10, J8 Conn_01x10, J9 Conn_01x10, U1 RT9742SNGV, U10 ac108, U11 TCR3RM33, U12 TCR3RM33, U13 TCR3RM33, U14 TCR3RM33, U2 ISO1540, U5 TPD4EUSB30, U6 TPD4EUSB30, U7 TPD4EUSB30, U9 SI8663BB-B-IS1, X1 ASE-24.000MHz

Commit message: .
.
Parts:
- removed C14: 100uF, Capacitor_Tantalum_SMD:CP_EIA-3528-21_Kemet-B
- removed C18, C20, C25, C3: 10u, Capacitor_SMD:C_0805_2012Metric
- removed R5: 15K 1%, Resistor_SMD:R_0402_1005Metric
- added R1: NC, Resistor_SMD:R_0402_1005Metric, F.Cu at (32.0, 41.8)
- added R2: NC, Resistor_SMD:R_0402_1005Metric, F.Cu at (32.0, 42.8)
- added R3: 2.2K 1%, Resistor_SMD:R_0402_1005Metric, F.Cu at (32.0, 43.8)
- added R4: 2.2K 1%, Resistor_SMD:R_0402_1005Metric, F.Cu at (32.0, 44.8)
- added U3: TPD4EUSB30, Package_SON:USON-10_2.5x1.0mm_P0.5mm, F.Cu at (9.75, 38.2)
- R10, R11: value 470R -> 2k
- moved J5 67.5 mm to (3.60, 37.5), turned to -90 degrees
- moved R19 62.5 mm to (13.2, 34.0)
- moved R20 62.5 mm to (13.2, 32.8)
- moved R21 62.5 mm to (15.2, 34.0)
- moved R22 62.5 mm to (15.2, 32.8)
- moved C73 52.8 mm to (14.9, 42.9), turned to 90 degrees
- moved R11 0.84 mm to (32.0, 45.8)
- moved R10 0.80 mm to (32.0, 46.7)
Connections:
- net /CM4_docker1/CM4_HIGH_SPEED/USB_OTG_ID renamed /CM4_docker1/USB_OTG
- J2 pad 13: /CM4_docker1/3.3V -> /CM4_docker1/CM4_LOW_SPEED/5V
- J2 pad 16: /CM4_docker1/3.3V -> /CM4_docker1/CM4_LOW_SPEED/5V
- J5 pad A6: unconnected-(J5-PadA6) -> /CM4_docker1/POWER/D+
- J5 pad A7: unconnected-(J5-PadA7) -> /CM4_docker1/POWER/D-
Routing:
- net /CM4_docker1/3.3V: track 118.8 -> 2.69 mm, vias 15 -> 0
- net /CM4_docker1/xHCI-USB3/VBUS: track 51.2 -> 0.00 mm, vias 4 -> 0
- net /CM4_docker1/CM4_LOW_SPEED/5V: track 0.00 -> 40.1 mm, vias 0 -> 2
- net /CM4_docker1/+5V: track 81.1 -> 54.2 mm, vias 84 -> 47
- net /CM4_docker1/POWER/D-: track 0.00 -> 26.4 mm
- net /CM4_docker1/POWER/D+: track 0.00 -> 26.4 mm
- net /CM4_docker1/USB_DEBUG_N: track 62.0 -> 71.7 mm
- net /CM4_docker1/USB_DEBUG_P: track 63.3 -> 73.0 mm
- net /CM4_docker1/USB_OTG: track 73.7 -> 82.7 mm
- net /CM4_docker1/POWER/CC1: track 9.73 -> 7.65 mm
- net /CM4_docker1/nRPIBOOT: track 47.0 -> 45.0 mm
- net GND: track 30.8 -> 29.1 mm, vias 175 -> 155
- net /CM4_docker1/xHCI-USB3/ILIM: track 1.53 -> 0.00 mm
- net /CM4_docker1/CM4_LOW_SPEED/LED_GREEN: track 43.7 -> 42.8 mm
- net /CM4_docker1/POWER/CC2: track 16.1 -> 15.2 mm, vias 0 -> 2
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- removed copper zone on In1.Cu, net /CM4_docker1/+5V
- removed copper zone on B.Cu, net /CM4_docker1/3.3V
- removed copper zone on F.Cu, net /CM4_docker1/3.3V
- removed copper zone on F.Cu, net /CM4_docker1/xHCI-USB3/VBUS
- removed copper zone on In2.Cu, net GND

Commit message: .
.
Parts:
- added U4: SPU0414HR5H-SB, CM4IO:SPU0414HR5H-SB, B.Cu at (100.0, 0.00)
- added U8: MIC_MODULE_4PIN, CM4IO:MIC_MODULE_4PIN, F.Cu at (101.0, 5.25)
Other:
- board size 251 x 75 mm -> 251 x 78.2 mm
Changed lines of the file:
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@@
   (net 267 "/CM4_docker1/POWER/D+")
   (net 268 "/CM4_docker1/USB_OTG")
+  (net 269 "unconnected-(U4-Pad1)")
+  (net 270 "unconnected-(U4-Pad2)")
+  (net 271 "unconnected-(U4-Pad3)")
+  (net 272 "unconnected-(U4-Pad4)")
+  (net 273 "unconnected-(U8-Pad1)")
+  (net 274 "unconnected-(U8-Pad2)")
+  (net 275 "unconnected-(U8-Pad3)")
+  (net 276 "unconnected-(U8-Pad4)")
   (footprint "Resistor_SMD:R_0603_1608Metric" (layer "F.Cu")
     (at 191.9 19.5 90)
@@
     )
   )
+  (footprint "CM4IO:MIC_MODULE_4PIN" (layer "F.Cu")
+    (at 101 5.25 180)
+    (property "Sheetfile" "mic_moudle.kicad_sch")
+    (property "Sheetname" "mic_moudle")
+    (attr smd)
+    (fp_text reference "U8" (at 1 4.25 180 unlocked) (layer "F.SilkS") hide
+      (effects (font (size 1 1) (thickness 0.15)))
+    )
+    (fp_text value "MIC_MODULE_4PIN" (at 1 -5 180 unlocked) (layer "F.Fab")
+      (effects (font (size 1 1) (thickness 0.15)))
+    )
+    (fp_text user "${REFERENCE}" (at 1 -3 180 unlocked) (layer "F.Fab")
+      (effects (font (size 1 1) (thickness 0.15)))
+    )
+    (fp_line (start -1 -1) (end 3 -1) (layer "F.SilkS") (width 0.12))
+    (fp_line (start 3 -1) (end 3 3) (layer "F.SilkS") (width 0.12))
+    (fp_line (start 3 3) (end -1 3) (layer "F.SilkS") (width 0.12))
+    (fp_line (start -1 3) (end -1 -1) (layer "F.SilkS") (width 0.12))
+    (pad "1" thru_hole circle (at 0 0 180) (size 1.5 1.5) (drill 0.8) (layers *.Cu *.Mask)
+      (net 273 "unconnected-(U8-Pad1)") (pinfunction "VCC") (pintype "input"))
+    (pad "2" thru_hole circle (at 0 2 180) (size 1.5 1.5) (drill 0.8) (layers *.Cu *.Mask)
+      (net 274 "unconnected-(U8-Pad2)") (pinfunction "GND") (pintype "input"))
+    (pad "3" thru_hole circle (at 2 2 180) (size 1.5 1.5) (drill 0.8) (layers *.Cu *.Mask)
+      (net 275 "unconnected-(U8-Pad3)") (pinfunction "MIC+") (pintype "input"))
+    (pad "4" thru_hole circle (at 2 0 180) (size 1.5 1.5) (drill 0.8) (layers *.Cu *.Mask)
+      (net 276 "unconnected-(U8-Pad4)") (pinfunction "MIC-") (pintype "input"))
+    (model "${KIPRJMOD}/CM4IO.3dshapes/2pin_header.stp"
+      (offset (xyz -0.25 -2 2.9))
+      (scale (xyz 1 1 1))
+      (rotate (xyz 0 -90 0))
+    )
+  )
   (footprint "Resistor_SMD:R_0603_1608Metric" (layer "F.Cu")
     (at 228 26.8)
@@
     )
   )
+  (footprint "CM4IO:SPU0414HR5H-SB" (layer "B.Cu")
+    (at 100 0 -90)
+    (property "Sheetfile" "mic_moudle.kicad_sch")
+    (property "Sheetname" "mic_moudle")
+    (property "automotive" "No")
+    (property "category" "IC")
+    (property "current" "155uA")
+    (property "device class L1" "Electromechanical")
+    (property "device class L2" "Audio Products")
+    (property "device class L3" "Microphones")
+    (property "digikey description" "MICROPHONE MEMS ANALOG OMNI")
+    (property "digikey part number" "423-1134-1-ND")
+    (property "direction" "Omidirectional")
+    (property "height" "1.2mm")
+    (property "lead free" "Yes")
+    (property "library id" "f86fcaa495503a79")
+    (property "manufacturer" "Knowles Acoustics")
+    (property "max supply voltage" "3.6V")
+    (property "min supply voltage" "1.5V")
+    (property "mouser description" "Knowles Acoustics Spu0414hr5h-Sb / Mic Sisonic Ultramini Top Max Rf")
+    (property "mouser part number" "721-SPU0414HR5H-SB")
+    (property "operating supply voltage" "1.5-3.6V")
+    (property "package" "SMT_3MM76_2MM95")
+    (property "resistance" "400Ω")
+    (property "rohs" "Yes")
+    (property "temperature range high" "+100°C")
+    (property "temperature range low" "-40°C")
+    (attr through_hole)
+    (fp_text reference "U4" (at -1.93 2.325 90) (layer "B.SilkS") hide
+      (effects (font (size 1 1) (thickness 0.15)) (justify left mirror))
+    )
+    (fp_text value "SPU0414HR5H-SB" (at 0 3 90) (layer "B.SilkS") hide
+      (effects (font (size 1.27 1.27) (thickness 0.15)) (justify mirror))
+    )
+    (fp_line (start -1.93 -0.075) (end -1.93 0.075) (layer "B.SilkS") (width 0.15))
+    (fp_line (start 1.93 -0.075) (end 1.93 0.075) (layer "B.SilkS") (width 0.15))
+    (fp_line (start -0.455 1.525) (end 0.455 1.525) (layer "B.SilkS") (width 0.15))
+    (fp_line (start -0.455 -1.525) (end 0.455 -1.525) (layer "B.SilkS") (width 0.15))
+    (fp_circle (center 2.33 -0.85) (end 2.455 -0.85) (layer "B.SilkS") (width 0.25) (fill none))
+    (fp_line (start -1.955 1.55) (end -1.955 -1.55) (layer "B.CrtYd") (width 0.15))
+    (fp_line (start -1.955 -1.55) (end 1.955 -1.55) (layer "B.CrtYd") (width 0.15))
+    (fp_line (start 1.955 -1.55) (end 1.955 1.55) (layer "B.CrtYd") (width 0.15))
+    (fp_line (start 1.955 1.55) (end 1.955 1.55) (layer "B.CrtYd") (width 0.15))
+    (fp_line (start 1.955 1.55) (end -1.955 1.55) (layer "B.CrtYd") (width 0.15))
+    (fp_line (start -1.93 -1.525) (end -1.93 1.525) (layer "B.Fab") (width 0.15))
+    (fp_line (start 1.93 1.525) (end 1.93 -1.525) (layer "B.Fab") (width 0.15))
+    (fp_line (start -1.93 1.525) (end 1.93 1.525) (layer "B.Fab") (width 0.15))
+    (fp_line (start 1.93 -1.525) (end -1.93 -1.525) (layer "B.Fab") (width 0.15))
+    (pad "1" smd circle (at 1.23 -0.85 270) (size 0.8 0.8) (layers "B.Cu" "B.Paste" "B.Mask")
+      (net 269 "unconnected-(U4-Pad1)") (pinfunction "VDD") (pintype "power_in"))
+    (pad "2" smd circle (at -1.23 -0.85 270) (size 0.8 0.8) (layers "B.Cu" "B.Paste" "B.Mask")
+      (net 270 "unconnected-(U4-Pad2)") (pinfunction "GROUND") (pintype "power_in"))
+    (pad "3" smd circle (at -1.23 0.85 270) (size 0.8 0.8) (layers "B.Cu" "B.Paste" "B.Mask")
+      (net 271 "unconnected-(U4-Pad3)") (pinfunction "GAIN") (pintype "passive"))
+    (pad "4" smd circle (at 1.23 0.85 270) (size 0.8 0.8) (layers "B.Cu" "B.Paste" "B.Mask")
+      (net 272 "unconnected-(U4-Pad4)") (pinfunction "OUTPUT") (pintype "passive"))
+    (model "${KIPRJMOD}/CM4IO.3dshapes/SPU0414HR5H-SB.step"
+      (offset (xyz 0 0 0))
+      (scale (xyz 1 1 1))
+      (rotate (xyz 0 0 0))
+    )
+  )
   (footprint "Connector_PinSocket_2.54mm:PinSocket_1x10_P2.54mm_Vertical" (layer "B.Cu")
     (at 207 3 -90)
@@
   (gr_line (start 194 46) (end 209.5 46) (layer "Edge.Cuts") (width 0.15))
   (gr_line (start 0 75) (end 0 0) (layer "Edge.Cuts") (width 0.15))
+  (gr_rect (start 98 -3.21) (end 102 7.75) (layer "Edge.Cuts") (width 0.1) (fill none))
   (gr_arc (start 192.5 28) (mid 193.56066 28.43934) (end 194 29.5) (layer "Edge.Cuts") (width 0.15))
   (gr_line (start 251 0) (end 251 75) (layer "Edge.Cuts") (width 0.15))

Commit message: .
.
Parts:
- added C3: 0.1uF, Capacitor_SMD:C_0402_1005Metric, F.Cu at (78.5, 2.40)
- added C4: 0.1uF, Capacitor_SMD:C_0402_1005Metric, F.Cu at (80.9, 2.71)
- added C5: 10nF, Capacitor_SMD:C_0402_1005Metric, F.Cu at (78.5, 4.41)
- added R5: 0, Resistor_SMD:R_0402_1005Metric, F.Cu at (78.5, 1.41)
- added R6: 0, Resistor_SMD:R_0402_1005Metric, F.Cu at (78.5, 3.40)
- moved U4 20.7 mm to (79.5, 2.71)
- moved U8 20.7 mm to (80.5, 7.96)
Connections:
- U4 pad 1: unconnected-(U4-Pad1) -> /mic_moudle/VDD
- U4 pad 2: unconnected-(U4-Pad2) -> /mic_moudle/GND
- U4 pad 3: unconnected-(U4-Pad3) -> /mic_moudle/GAIN
- U4 pad 4: unconnected-(U4-Pad4) -> /mic_moudle/OUT
- U8 pad 1: unconnected-(U8-Pad1) -> /mic_moudle/VDD
- U8 pad 2: unconnected-(U8-Pad2) -> /mic_moudle/GND
- U8 pad 3: unconnected-(U8-Pad3) -> /mic_moudle/MIC+
Routing:
- net /mic_moudle/VDD: track 0.00 -> 3.09 mm, vias 0 -> 2
- net /mic_moudle/OUT: track 0.00 -> 1.96 mm, vias 0 -> 1
- net /mic_moudle/GAIN: track 0.00 -> 1.94 mm, vias 0 -> 1
- net /mic_moudle/MIC+: track 0.00 -> 1.75 mm
- net Net-(C5-Pad1): track 0.00 -> 1.05 mm
- net Net-(C3-Pad2): track 0.00 -> 1.01 mm
- net /mic_moudle/GND: track 0.00 -> 0.02 mm, vias 0 -> 1
- added copper zone on B.Cu, net /mic_moudle/GND
- added copper zone on F.Cu, net /mic_moudle/GND
- added copper zone on In1.Cu, net /mic_moudle/GND
- added copper zone on In2.Cu, net /mic_moudle/VDD
Other:
- board size 251 x 78.2 mm -> 251 x 75 mm

Commit message: .
.
Parts:
- added ?: , , F.Cu at (179.5, 71.5)
- added J2: JK00177, Connector_RJ:RJ45_Pulse_JK00177NL_Horizontal, F.Cu at (201.6, 63.2)
- added U15: MIC_4PIN_SMD, CM4IO:MIC_4PIN_SMD, F.Cu at (173.0, -1.54)
Connections:
- U8 pad 4: unconnected-(U8-Pad4) -> /mic_moudle/NC
Other:
- board size 251 x 75 mm -> 273.8 x 120.4 mm
