File: audio/audio.kicad_sch (KiCad schematic)
At the start: 0 parts

Commit message: .
.
Other:
- sheet 4ch_mic ports: added ISO_SCK, ISO_SDA, VDD_3.3V; removed none
- sheet isolation_module ports: added AVCC_5V, AVCC_GND, ISO_SCL, ISO_SDA, VDD_3.3V, VDD_5V, VDD_GND; removed none
Changed lines of the file:
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@@
 (kicad_sch (version 20211123) (generator eeschema)
   (paper "A4")
+  (wire (pts (xy 105.41 60.96) (xy 123.19 60.96))
+    (stroke (width 0) (type default) (color 0 0 0 0))
+  )
+  (wire (pts (xy 105.41 33.02) (xy 123.19 33.02))
+    (stroke (width 0) (type default) (color 0 0 0 0))
+  )
+  (wire (pts (xy 105.41 63.5) (xy 123.19 63.5))
+    (stroke (width 0) (type default) (color 0 0 0 0))
+  )
+  (wire (pts (xy 105.41 44.45) (xy 123.19 44.45))
+    (stroke (width 0) (type default) (color 0 0 0 0))
+  )
+  (wire (pts (xy 105.41 46.99) (xy 123.19 46.99))
+    (stroke (width 0) (type default) (color 0 0 0 0))
+  )
+  (wire (pts (xy 105.41 57.15) (xy 123.19 57.15))
+    (stroke (width 0) (type default) (color 0 0 0 0))
+  )
+  (wire (pts (xy 105.41 35.56) (xy 123.19 35.56))
+    (stroke (width 0) (type default) (color 0 0 0 0))
+  )
   (sheet (at 78.74 26.67) (size 26.67 43.18) (fields_autoplaced)
     (stroke (width 0.1524) (type solid) (color 0 0 0 0))
@@
       (effects (font (size 1.27 1.27)) (justify left))
     )
+    (pin "VDD_5V" output (at 105.41 33.02 0)
+      (effects (font (size 1.27 1.27)) (justify right))
+    )
+    (pin "VDD_GND" output (at 105.41 35.56 0)
+      (effects (font (size 1.27 1.27)) (justify right))
+    )
+    (pin "AVCC_GND" output (at 105.41 63.5 0)
+      (effects (font (size 1.27 1.27)) (justify right))
+    )
+    (pin "AVCC_5V" output (at 105.41 60.96 0)
+      (effects (font (size 1.27 1.27)) (justify right))
+    )
+    (pin "VDD_3.3V" input (at 105.41 57.15 0)
+      (effects (font (size 1.27 1.27)) (justify right))
+    )
+    (pin "ISO_SDA" bidirectional (at 105.41 44.45 0)
+      (effects (font (size 1.27 1.27)) (justify right))
+    )
+    (pin "ISO_SCL" bidirectional (at 105.41 46.99 0)
+      (effects (font (size 1.27 1.27)) (justify right))
+    )
   )
   (sheet (at 123.19 26.67) (size 31.75 43.18) (fields_autoplaced)
@@
     )
     (pin "VDD_GND" input (at 123.19 35.56 180)
+      (effects (font (size 1.27 1.27)) (justify left))
+    )
+    (pin "VDD_3.3V" output (at 123.19 57.15 180)
+      (effects (font (size 1.27 1.27)) (justify left))
+    )
+    (pin "ISO_SDA" bidirectional (at 123.19 44.45 180)
+      (effects (font (size 1.27 1.27)) (justify left))
+    )
+    (pin "ISO_SCK" bidirectional (at 123.19 46.99 180)
       (effects (font (size 1.27 1.27)) (justify left))
     )
@@
       (reference "C57") (unit 1) (value "1uF") (footprint "Capacitor_SMD:C_0402_1005Metric")
     )
+    (path "/039620fc-845c-4f42-b371-a9cdeb447748/1bb55229-ee61-4734-afb9-e122552e5efc"
+      (reference "C?") (unit 1) (value "10uF") (footprint "Capacitor_SMD:C_0402_1005Metric")
+    )
+    (path "/039620fc-845c-4f42-b371-a9cdeb447748/35a714f4-35b2-4606-a330-f54351eb8b8f"
+      (reference "C?") (unit 1) (value "10uF") (footprint "Capacitor_SMD:C_0402_1005Metric")
+    )
+    (path "/039620fc-845c-4f42-b371-a9cdeb447748/42fd9cc3-a1c7-48e6-a1b5-dfa90ff36a9b"
+      (reference "C?") (unit 1) (value "10uF") (footprint "Capacitor_SMD:C_0402_1005Metric")
+    )
+    (path "/039620fc-845c-4f42-b371-a9cdeb447748/62e4a09c-e079-40c9-88c9-84fb093328d9"
+      (reference "C?") (unit 1) (value "0.1uF") (footprint "Capacitor_SMD:C_0402_1005Metric")
+    )
+    (path "/039620fc-845c-4f42-b371-a9cdeb447748/8a543b7f-afd8-458e-91cc-5b7626ce57d9"
+      (reference "C?") (unit 1) (value "0.1uF") (footprint "Capacitor_SMD:C_0402_1005Metric")
+    )
+    (path "/039620fc-845c-4f42-b371-a9cdeb447748/9fc4e6e4-f57f-4832-98ce-0a1682dc2ac4"
+      (reference "C?") (unit 1) (value "10uF") (footprint "Capacitor_SMD:C_0402_1005Metric")
+    )
+    (path "/039620fc-845c-4f42-b371-a9cdeb447748/b19d8232-7a79-4e8f-b138-c3f1514264e3"
+      (reference "C?") (unit 1) (value "0.1uF") (footprint "Capacitor_SMD:C_0402_1005Metric")
+    )
+    (path "/039620fc-845c-4f42-b371-a9cdeb447748/b857485a-1914-49df-939c-3768a8e1153f"
+      (reference "C?") (unit 1) (value "0.1uF") (footprint "Capacitor_SMD:C_0402_1005Metric")
+    )
     (path "/90bebbb0-1fdd-4048-9d12-a8c8747778ea/323b8967-7dfd-44f3-9141-90ee1155f22c/42f6fe2f-8af7-44f7-8fc7-5a6761485dc5"
       (reference "CM4_MODULE1") (unit 1) (value "ComputeModule4-CM4") (footprint "CM4IO:Raspberry-Pi-4-Compute-Module")
@@
       (reference "PS1") (unit 1) (value "R05CTE05S-R") (footprint "CM4IO:SOIC127P1030X265-16N")
     )
-    (path "/039620fc-845c-4f42-b371-a9cdeb447748/980c7cbb-f3ea-4894-a81f-d7b4f5ba2b0d"
-      (reference "PS2") (unit 1) (value "R05CTE05S-R") (footprint "CM4IO:SOIC127P1030X265-16N")
+    (path "/039620fc-845c-4f42-b371-a9cdeb447748/4c6bb1da-9734-45ea-bd03-ec3fa27347d8"
+      (reference "PS?") (unit 1) (value "R05CTE05S-R") (footprint "CM4IO:SOIC127P1030X265-16N")
     )
     (path "/90bebbb0-1fdd-4048-9d12-a8c8747778ea/2d9b1a0f-1381-458a-afc7-6a2863de9fe8/55100669-b608-4057-b206-1b2655b8bece"
@@
       (reference "R41") (unit 1) (value "0") (footprint "Resistor_SMD:R_0603_1608Metric")
     )
+    (path "/039620fc-845c-4f42-b371-a9cdeb447748/7de2a3b2-fa46-4fd6-b370-1525aa40da25"
+      (reference "R?") (unit 1) (value "1k") (footprint "Resistor_SMD:R_0603_1608Metric")
+    )
+    (path "/039620fc-845c-4f42-b371-a9cdeb447748/bc525e79-f897-46c9-90af-41caba500e8f"
+      (reference "R?") (unit 1) (value "1k") (footprint "Resistor_SMD:R_0603_1608Metric")
+    )
     (path "/90bebbb0-1fdd-4048-9d12-a8c8747778ea/6ec665d8-c64e-4e17-9c29-206f5c3ea2cd/bcffc3e4-1087-40df-8d6c-be5df8e256f5"

Commit message: .
.
Other:
- sheet 4ch_mic ports: added ISO_ADC, ISO_BCLK, ISO_LRCK; removed none
- sheet isolation_module ports: added ISO_ADC, ISO_BCLK, ISO_LRCK; removed none

Commit message: .
.
Other:
- sheet CM4_docker1 ports: added 3.3V_I2C, GND_I2C, nRPIBOOT; removed none
- sheet isolation_module ports: added 3.3V_I2C, GND_I2C, nRPIBOOT; removed none
Changed lines of the file:
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@@
+    (stroke (width 0) (type default) (color 0 0 0 0))
+  )
+  (polyline (pts (xy 55.88 52.07) (xy 78.74 52.07))
     (stroke (width 0) (type default) (color 0 0 0 0))
   )
@@
     (stroke (width 0) (type default) (color 0 0 0 0))
   )
+  (polyline (pts (xy 55.88 59.69) (xy 78.74 59.69))
+    (stroke (width 0) (type default) (color 0 0 0 0))
+  )
   (polyline (pts (xy 55.88 46.99) (xy 78.74 46.99))
+    (stroke (width 0) (type default) (color 0 0 0 0))
+  )
+  (polyline (pts (xy 55.88 54.61) (xy 78.74 54.61))
     (stroke (width 0) (type default) (color 0 0 0 0))
   )
@@
       (effects (font (size 1.27 1.27)) (justify right))
     )
+    (pin "3.3V_I2C" input (at 78.74 52.07 180)
+      (effects (font (size 1.27 1.27)) (justify left))
+    )
+    (pin "GND_I2C" input (at 78.74 54.61 180)
+      (effects (font (size 1.27 1.27)) (justify left))
+    )
+    (pin "nRPIBOOT" output (at 78.74 59.69 180)
+      (effects (font (size 1.27 1.27)) (justify left))
+    )
   )
   (sheet (at 113.03 26.67) (size 30.48 59.69) (fields_autoplaced)
@@
     )
     (pin "3.3V" output (at 55.88 35.56 0)
+      (effects (font (size 1.27 1.27)) (justify right))
+    )
+    (pin "nRPIBOOT" input (at 55.88 59.69 0)
+      (effects (font (size 1.27 1.27)) (justify right))
+    )
+    (pin "3.3V_I2C" output (at 55.88 52.07 0)
+      (effects (font (size 1.27 1.27)) (justify right))
+    )
+    (pin "GND_I2C" output (at 55.88 54.61 0)
       (effects (font (size 1.27 1.27)) (justify right))
     )
@@
       (reference "R34") (unit 1) (value "0") (footprint "Resistor_SMD:R_0402_1005Metric")
     )
+    (path "/039620fc-845c-4f42-b371-a9cdeb447748/ca8d7f23-dc48-45e9-856b-6a49ad1068d0"
+      (reference "R35") (unit 1) (value "15K 1%") (footprint "Resistor_SMD:R_0402_1005Metric")
+    )
+    (path "/90bebbb0-1fdd-4048-9d12-a8c8747778ea/323b8967-7dfd-44f3-9141-90ee1155f22c/53c58d75-ab0d-495b-a51b-18ab3fbf9d4a"
+      (reference "R36") (unit 1) (value "30K 1%") (footprint "Resistor_SMD:R_0402_1005Metric")
+    )
     (path "/039620fc-845c-4f42-b371-a9cdeb447748/3099ad66-db62-4727-9240-9c7aa19db569"
