File: audio/audio.kicad_sch (KiCad schematic)
At the start: 0 parts

Commit message: .
.
Other:
- added sheet mic_moudle (mic_moudle.kicad_sch)
Changed lines of the file:
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@@
+    )
+  )
+  (sheet (at 154.94 26.67) (size 27.94 58.42) (fields_autoplaced)
+    (stroke (width 0.1524) (type solid) (color 0 0 0 0))
+    (fill (color 0 0 0 0.0000))
+    (property "Sheet name" "mic_moudle" (id 0) (at 154.94 25.9584 0)
+      (effects (font (size 1.27 1.27)) (justify left bottom))
+    )
+    (property "Sheet file" "mic_moudle.kicad_sch" (id 1) (at 154.94 85.6746 0)
+      (effects (font (size 1.27 1.27)) (justify left top))
     )
   )
@@
     (path "/90bebbb0-1fdd-4048-9d12-a8c8747778ea/323b8967-7dfd-44f3-9141-90ee1155f22c" (page "6"))
     (path "/90bebbb0-1fdd-4048-9d12-a8c8747778ea/3d5c4cf7-13f4-49bb-b4ff-0f2ab6b41503" (page "8"))
+    (path "/daa996b3-8cca-4e80-978a-b45cd225225a" (page "8"))
   )
   (symbol_instances
@@
       (reference "U3") (unit 1) (value "TPD4EUSB30") (footprint "Package_SON:USON-10_2.5x1.0mm_P0.5mm")
     )
+    (path "/daa996b3-8cca-4e80-978a-b45cd225225a/02ec9700-875a-4205-8a71-8de7e45fd48f"
+      (reference "U4") (unit 1) (value "SPU0414HR5H-SB") (footprint "CM4IO:SPU0414HR5H-SB")
+    )
     (path "/90bebbb0-1fdd-4048-9d12-a8c8747778ea/323b8967-7dfd-44f3-9141-90ee1155f22c/5c4d2ec8-6904-46e1-9ee8-610590ef91b6"
       (reference "U5") (unit 1) (value "TPD4EUSB30") (footprint "Package_SON:USON-10_2.5x1.0mm_P0.5mm")
@@
       (reference "U7") (unit 1) (value "TPD4EUSB30") (footprint "Package_SON:USON-10_2.5x1.0mm_P0.5mm")
     )
+    (path "/daa996b3-8cca-4e80-978a-b45cd225225a/a033fd0f-e292-408f-ae2b-f7c5975e789f"
+      (reference "U8") (unit 1) (value "MIC_MODULE_4PIN") (footprint "CM4IO:MIC_MODULE_4PIN")
+    )
     (path "/039620fc-845c-4f42-b371-a9cdeb447748/0c56e234-7ade-4a53-955a-94963a078856"

Commit message: .
.
Changed lines of the file:
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@@
     )
   )
-  (sheet (at 154.94 26.67) (size 27.94 58.42) (fields_autoplaced)
+  (sheet (at 176.53 26.67) (size 27.94 58.42) (fields_autoplaced)
     (stroke (width 0.1524) (type solid) (color 0 0 0 0))
     (fill (color 0 0 0 0.0000))
-    (property "Sheet name" "mic_moudle" (id 0) (at 154.94 25.9584 0)
+    (property "Sheet name" "mic_moudle" (id 0) (at 176.53 25.9584 0)
       (effects (font (size 1.27 1.27)) (justify left bottom))
     )
-    (property "Sheet file" "mic_moudle.kicad_sch" (id 1) (at 154.94 85.6746 0)
+    (property "Sheet file" "mic_moudle.kicad_sch" (id 1) (at 176.53 85.6746 0)
       (effects (font (size 1.27 1.27)) (justify left top))
     )
@@
       (reference "U14") (unit 1) (value "TCR3RM33") (footprint "CM4IO:TCR3RM33")
     )
+    (path "/37bdbadf-9ce7-4cff-96aa-5222c88e6059/62312893-d00b-4ab7-8850-40f6021f4305"
+      (reference "U15") (unit 1) (value "MIC_4PIN_SMD") (footprint "CM4IO:MIC_4PIN_SMD")
+    )
     (path "/37bdbadf-9ce7-4cff-96aa-5222c88e6059/92925ad6-0127-4058-9a64-eaafaf821f0a"
