File: audio/CM4_LOW_SPEED.kicad_sch (KiCad schematic)
At the start: 8 parts, among them J4 THD-02-R, U5 TPD4EUSB30, U6 TPD4EUSB30, U7 MagJack-A70-112-331N126

Commit message: .
.
Parts:
- removed J4: THD-02-R, Connector_PinHeader_2.54mm:PinHeader_2x02_P2.54mm_Vertical, symbol Connector_Generic:Conn_02x02_Odd_Even
- removed U7: MagJack-A70-112-331N126, CM4IO:TRJG0926HENL, symbol CM4IO:MagJack-A70-112-331N126
- added J2: JK00177, Connector_RJ:RJ45_Pulse_JK00177NL_Horizontal, symbol Connector:JK00177
Connections:
- net +3.3v: now also J2.13 (LED2+), J2.16 (LED1+)
- net ETH_LEDG: now also R11.2; no longer R10.2
- net ETH_LEDY: now also R10.2; no longer R11.2
- net GND: now also J2.SH
- net TRD0_N: now also J2.10 (MX1-)
- net TRD0_P: now also J2.11 (MX1+)
- net TRD1_N: now also J2.5 (MX2-)
- net TRD1_P: now also J2.4 (MX2+)
- net TRD2_N: now also J2.2 (MX3-)
- net TRD2_P: now also J2.3 (MX3+)
- net TRD3_N: now also J2.9 (MX4-)
- net TRD3_P: now also J2.8 (MX4+)
- net at R10.1: now also J2.15 (LED1-)
- net at R11.1: now also J2.14 (LED2-)
- net at C39.1: now also J2.1 (MXCT3), J2.12 (MXCT1), J2.6 (MXCT2), J2.7 (MXCT4)
Other:
- note removed: "POE Header"
- moved on the sheet: U5, U6

Commit message: .
.
Parts:
- added J4: 1054500101, CM4IO:MOLEX_105450-0101, symbol CM4IO:1054500101
- added R12, R13, R14, R15: 5.1K 5%, Resistor_SMD:R_0402_1005Metric, symbol Device:R
- added U7: TPD4EUSB30, Package_SON:USON-10_2.5x1.0mm_P0.5mm, symbol CM4IO:TPD4EUSB30
Connections:
- net GND: now also J4.A1 (GND_A), J4.A12 (GND_A), J4.B1 (GND_B), J4.B12 (GND_B), J4.S1 (SHIELD), J4.S2 (SHIELD), J4.S3 (SHIELD), J4.S4 (SHIELD), R13.2, R15.2, U7.3 (GND), U7.8 (GND)
- new net: U7.1 (D1+), U7.10
- new net: U7.2 (D1-), U7.9
- new net 5V: J4.A4 (VBUS_A), J4.A9 (VBUS_A), J4.B4 (VBUS_B), J4.B9 (VBUS_B), R12.1, R14.1
- new net CC1: J4.A5 (CC1), R12.2, R13.1
- new net CC2: J4.B5 (CC2), R14.2, R15.1
- new net USB2_N: J4.A7 (D1-), J4.B7 (D2-)
- new net USB2_P: J4.A6 (D1+), J4.B6 (D2+)
- new net USBD_N: U7.4 (D2+), U7.7
- new net USBD_P: U7.5 (D2-), U7.6
Other:
- note added: "Micro USB ESD protection"
- note added: "USB 2.0"
- moved on the sheet: C39, CM4_MODULE1A, J2, R10, R11, U5, U6

Commit message: .
.
Parts:
- added R16, R17, R18: 2.2K 1%, Resistor_SMD:R_0402_1005Metric, symbol Device:R
Connections:
- net 5V: no longer J4.A4 (VBUS_A), J4.A9 (VBUS_A), J4.B4 (VBUS_B), J4.B9 (VBUS_B)
- net GND: now also R16.1, R17.2
- new net USBOTG: R16.2, R17.1, R18.2
- new net VBUS: J4.A4 (VBUS_A), J4.A9 (VBUS_A), J4.B4 (VBUS_B), J4.B9 (VBUS_B), R18.1

Commit message: .
.
Changed lines of the file:
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@@
+    (stroke (width 0) (type solid) (color 0 0 0 0))
+  )
+  (wire (pts (xy 95.25 90.17) (xy 108.204 90.17))
     (stroke (width 0) (type solid) (color 0 0 0 0))
   )

Commit message: .
.
Connections:
- net GND: now also CM4_MODULE1.98 (GND)
- net USBOTG: no longer R16.2, R18.2
- net I2S_LRCK: now reaches CM4_MODULE1.26 (GPIO19)
- net I2S_ADC: now reaches CM4_MODULE1.27 (GPIO20)
- net I2S_BCLK: now reaches CM4_MODULE1.49 (GPIO18)
- net I2C1_SCL: now reaches CM4_MODULE1.56 (GPIO3)
- net I2C1_SDA: now reaches CM4_MODULE1.58 (GPIO2)
- net 3.3V: now reaches CM4_MODULE1.84 (+3.3v_(Output))
- net 3.3V: now also CM4_MODULE1.86 (+3.3v_(Output))
- new net: R16.2, R18.2
Other:
- moved on the sheet: CM4_MODULE1A, R16, R17, R18

Commit message: .
.
Parts:
- removed R17: 2.2K 1%, Resistor_SMD:R_0402_1005Metric, symbol Device:R
Connections:
- net USBOTG: now also R16.2, R18.2
- net SD_CLK: now reaches CM4_MODULE1.57 (SD_CLK)
- net SD_DAT3: now reaches CM4_MODULE1.61 (SD_DAT3)
- net SD_CMD: now reaches CM4_MODULE1.62 (SD_CMD)
- net SD_DAT0: now reaches CM4_MODULE1.63 (SD_DAT0)
- net SD_DAT1: now reaches CM4_MODULE1.67 (SD_DAT1)
- net SD_DAT2: now reaches CM4_MODULE1.69 (SD_DAT2)
Changed lines of the file:
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@@
   (junction (at 262.89 128.27) (diameter 0) (color 0 0 0 0)
   )
+  (junction (at 135.89 109.22) (diameter 0) (color 0 0 0 0)
+  )
   (junction (at 233.68 52.07) (diameter 0) (color 0 0 0 0)
   )
@@
     (stroke (width 0) (type solid) (color 0 0 0 0))
   )
+  (wire (pts (xy 110.49 101.6) (xy 96.52 101.6))
+    (stroke (width 0) (type solid) (color 0 0 0 0))
+  )
+  (wire (pts (xy 143.51 101.6) (xy 143.51 92.71))
+    (stroke (width 0) (type default) (color 0 0 0 0))
+  )
   (wire (pts (xy 217.17 43.18) (xy 217.17 41.91))
     (stroke (width 0) (type solid) (color 0 0 0 0))
   )
-  (wire (pts (xy 143.51 92.71) (xy 143.51 101.6))
-    (stroke (width 0) (type default) (color 0 0 0 0))
-  )
   (wire (pts (xy 229.87 69.85) (xy 237.49 69.85))
     (stroke (width 0) (type solid) (color 0 0 0 0))
   )
+  (wire (pts (xy 110.49 106.68) (xy 96.52 106.68))
+    (stroke (width 0) (type solid) (color 0 0 0 0))
+  )
   (wire (pts (xy 208.28 24.13) (xy 219.71 24.13))
     (stroke (width 0) (type solid) (color 0 0 0 0))
@@
     (stroke (width 0) (type solid) (color 0 0 0 0))
   )
+  (wire (pts (xy 21.59 106.68) (xy 35.56 106.68))
+    (stroke (width 0) (type solid) (color 0 0 0 0))
+  )
+  (wire (pts (xy 110.49 114.3) (xy 96.52 114.3))
+    (stroke (width 0) (type solid) (color 0 0 0 0))
+  )
   (wire (pts (xy 130.81 96.52) (xy 138.43 96.52))
     (stroke (width 0) (type default) (color 0 0 0 0))
@@
     (stroke (width 0) (type default) (color 0 0 0 0))
   )
+  (wire (pts (xy 135.89 109.22) (xy 143.51 109.22))
+    (stroke (width 0) (type default) (color 0 0 0 0))
+  )
   (wire (pts (xy 153.67 99.06) (xy 168.91 99.06))
     (stroke (width 0) (type default) (color 0 0 0 0))
   )
-  (wire (pts (xy 144.78 151.13) (xy 144.78 144.78))
-    (stroke (width 0) (type default) (color 0 0 0 0))
-  )
   (polyline (pts (xy 279.4 12.7) (xy 279.4 86.36))
     (stroke (width 0) (type solid) (color 0 0 0 0))
   )
+  (wire (pts (xy 135.89 109.22) (xy 135.89 119.38))
+    (stroke (width 0) (type default) (color 0 0 0 0))
+  )
   (wire (pts (xy 21.59 152.4) (xy 35.56 152.4))
     (stroke (width 0) (type default) (color 0 0 0 0))
@@
     (stroke (width 0) (type default) (color 0 0 0 0))
   )
-  (wire (pts (xy 130.81 109.22) (xy 143.51 109.22))
+  (wire (pts (xy 130.81 109.22) (xy 135.89 109.22))
     (stroke (width 0) (type default) (color 0 0 0 0))
   )
@@
     (stroke (width 0) (type solid) (color 0 0 0 0))
   )
-  (wire (pts (xy 144.78 127) (xy 144.78 137.16))
-    (stroke (width 0) (type solid) (color 0 0 0 0))
-  )
   (wire (pts (xy 20.32 33.02) (xy 35.56 33.02))
     (stroke (width 0) (type solid) (color 0 0 0 0))
@@
     (stroke (width 0) (type default) (color 0 0 0 0))
   )
+  (wire (pts (xy 96.52 116.84) (xy 110.49 116.84))
+    (stroke (width 0) (type solid) (color 0 0 0 0))
+  )
   (wire (pts (xy 248.92 142.24) (xy 248.92 144.78))
     (stroke (width 0) (type default) (color 0 0 0 0))
   )
+  (wire (pts (xy 96.52 109.22) (xy 110.49 109.22))
+    (stroke (width 0) (type solid) (color 0 0 0 0))
+  )
   (wire (pts (xy 96.52 63.5) (xy 109.474 63.5))
     (stroke (width 0) (type solid) (color 0 0 0 0))
@@
     (stroke (width 0) (type default) (color 0 0 0 0))
   )
-  (wire (pts (xy 139.065 127) (xy 144.78 127))
-    (stroke (width 0) (type solid) (color 0 0 0 0))
-  )
-  (wire (pts (xy 135.89 92.71) (xy 143.51 92.71))
-    (stroke (width 0) (type default) (color 0 0 0 0))
-  )
   (wire (pts (xy 193.04 57.15) (xy 201.93 57.15))
     (stroke (width 0) (type solid) (color 0 0 0 0))
@@
   )
   (wire (pts (xy 233.68 52.07) (xy 237.49 52.07))
+    (stroke (width 0) (type default) (color 0 0 0 0))
+  )
+  (wire (pts (xy 143.51 92.71) (xy 152.4 92.71))
     (stroke (width 0) (type default) (color 0 0 0 0))
   )
@@
     (effects (font (size 1.27 1.27)) (justify right bottom))
   )
+  (label "SD_DAT3" (at 107.95 106.68 180)
+    (effects (font (size 1.27 1.27)) (justify right bottom))
+  )
+  (label "SD_CLK" (at 106.68 101.6 180)
+    (effects (font (size 1.27 1.27)) (justify right bottom))
+  )
   (label "+3.3v" (at 236.22 21.59 180)
     (effects (font (size 1.27 1.27)) (justify right bottom))
@@
     (effects (font (size 1.27 1.27)) (justify left bottom))
   )
+  (label "SD_CMD" (at 31.75 106.68 180)
+    (effects (font (size 1.27 1.27)) (justify right bottom))
+  )
   (label "GND" (at 219.71 130.81 0)
     (effects (font (size 1.27 1.27)) (justify left bottom))
@@
     (effects (font (size 1.27 1.27)) (justify left bottom))
   )
+  (label "SD_DAT2" (at 107.95 116.84 180)
+    (effects (font (size 1.27 1.27)) (justify right bottom))
+  )
   (label "TRD1_N" (at 166.37 62.23 180)
     (effects (font (size 1.27 1.27)) (justify right bottom))
@@
     (effects (font (size 1.27 1.27)) (justify left bottom))
   )
-  (label "VBUS" (at 137.16 92.71 0)
+  (label "VBUS" (at 146.05 92.71 0)
     (effects (font (size 1.27 1.27)) (justify left bottom))
   )
@@
     (effects (font (size 1.27 1.27)) (justify left bottom))
   )
+  (label "SD_DAT1" (at 107.95 114.3 180)
+    (effects (font (size 1.27 1.27)) (justify right bottom))
+  )
   (label "+3.3v" (at 236.22 69.85 180)
     (effects (font (size 1.27 1.27)) (justify right bottom))
@@
     (effects (font (size 1.27 1.27)) (justify left bottom))
   )
+  (label "SD_DAT0" (at 107.95 109.22 180)
+    (effects (font (size 1.27 1.27)) (justify right bottom))
+  )
   (label "I2S_BCLK" (at 99.06 91.44 0)
     (effects (font (size 1.27 1.27)) (justify left bottom))
@@
     (effects (font (size 1.27 1.27)) (justify left bottom))
   )
-  (hierarchical_label "USBOTG" (shape output) (at 139.065 127 180)
+  (hierarchical_label "USBOTG" (shape output) (at 135.89 119.38 270)
     (effects (font (size 1.27 1.27)) (justify right))
   )
@@
     (effects (font (size 1.27 1.27)) (justify right))
   )
+  (hierarchical_label "SD_DAT3" (shape input) (at 110.49 106.68 0)
+    (effects (font (size 1.27 1.27)) (justify left))
+  )
   (hierarchical_label "I2C1_SCL" (shape output) (at 22.606 99.06 180)
     (effects (font (size 1.27 1.27)) (justify right))
@@
     (effects (font (size 1.27 1.27)) (justify left))
   )
+  (hierarchical_label "SD_DAT0" (shape input) (at 110.49 109.22 0)
+    (effects (font (size 1.27 1.27)) (justify left))
+  )
   (hierarchical_label "USB2_N" (shape input) (at 224.79 115.57 0)
     (effects (font (size 1.27 1.27)) (justify left))
   )
+  (hierarchical_label "SD_CMD" (shape input) (at 21.59 106.68 180)
+    (effects (font (size 1.27 1.27)) (justify right))
+  )
   (hierarchical_label "I2S_ADC" (shape input) (at 109.474 63.5 0)
     (effects (font (size 1.27 1.27)) (justify left))
   )
+  (hierarchical_label "SD_CLK" (shape input) (at 110.49 101.6 0)
+    (effects (font (size 1.27 1.27)) (justify left))
+  )
   (hierarchical_label "GND" (shape output) (at 21.59 152.4 180)
     (effects (font (size 1.27 1.27)) (justify right))
@@
     (effects (font (size 1.27 1.27)) (justify right))
   )
+  (hierarchical_label "SD_DAT2" (shape input) (at 110.49 116.84 0)
+    (effects (font (size 1.27 1.27)) (justify left))
+  )
+  (hierarchical_label "SD_DAT1" (shape input) (at 110.49 114.3 0)
+    (effects (font (size 1.27 1.27)) (justify left))
+  )
   (hierarchical_label "I2S_BCLK" (shape bidirectional) (at 109.474 91.44 0)
     (effects (font (size 1.27 1.27)) (justify left))
-  )
-  (symbol (lib_id "power:GND") (at 144.78 151.13 0) (unit 1)
-    (in_bom yes) (on_board yes)
-    (property "Reference" "#PWR0131" (id 0) (at 144.78 157.48 0)
-      (effects (font (size 1.27 1.27)) hide)
-    )
-    (property "Value" "GND" (id 1) (at 144.907 155.5242 0))
-    (property "Footprint" "" (id 2) (at 144.78 151.13 0)
-      (effects (font (size 1.27 1.27)) hide)
-    )
-    (property "Datasheet" "" (id 3) (at 144.78 151.13 0)
-      (effects (font (size 1.27 1.27)) hide)
-    )
-    (pin "1")
   )
   (symbol (lib_id "power:GND") (at 180.34 72.39 0) (unit 1)
@@
     (pin "200")
   )
-  (symbol (lib_id "Device:R") (at 144.78 140.97 0) (unit 1)
-    (in_bom yes) (on_board yes)
-    (property "Reference" "R17" (id 0) (at 139.065 139.7 0)
-      (effects (font (size 1.27 1.27)) (justify left))
-    )
-    (property "Value" "2.2K 1%" (id 1) (at 135.255 142.24 0)
-      (effects (font (size 1.27 1.27)) (justify left))
-    )
-    (property "Footprint" "Resistor_SMD:R_0402_1005Metric" (id 2) (at 143.002 140.97 90)
-      (effects (font (size 1.27 1.27)) hide)
-    )
-    (property "Datasheet" "https://fscdn.rohm.com/en/products/databook/datasheet/passive/resistor/chip_resistor/mcr-e.pdf" (id 3) (at 144.78 140.97 0)
-      (effects (font (size 1.27 1.27)) hide)
-    )
-    (property "Field4" "Farnell" (id 4) (at 144.78 140.97 0)
-      (effects (font (size 1.27 1.27)) hide)
-    )
-    (property "Field5" "9239278" (id 5) (at 144.78 140.97 0)
-      (effects (font (size 1.27 1.27)) hide)
-    )
-    (property "Field7" "KOA EUROPE GMBH" (id 6) (at 144.78 140.97 0)
-      (effects (font (size 1.27 1.27)) hide)
-    )
-    (property "Field6" "RK73G1ETQTP2201D         " (id 7) (at 144.78 140.97 0)
-      (effects (font (size 1.27 1.27)) hide)
-    )
-    (property "Part Description" "Resistor 2.2K M1005 1% 63mW" (id 8) (at 144.78 140.97 0)
-      (effects (font (size 1.27 1.27)) hide)
-    )
-    (property "Field8" "120889581" (id 9) (at 144.78 140.97 0)
-      (effects (font (size 1.27 1.27)) hide)
-    )
-    (pin "1")
-    (pin "2")
-  )
   (symbol (lib_id "CM4IO:1054500101") (at 173.99 90.17 0) (unit 1)

Commit message: high_speed_artwork_done
.
Connections:
- net USBD_N is gone; now on net USB2_P: U7.4 (D2+), U7.7
- net USBD_P is gone; now on net USB2_N: U7.5 (D2-), U7.6
- net USB2_N: now also U7.2 (D1-), U7.9
- net USB2_P: now also U7.1 (D1+), U7.10
Changed lines of the file:
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@@
+    (stroke (width 0) (type solid) (color 0 0 0 0))
+  )
+  (wire (pts (xy 217.17 105.41) (xy 233.68 105.41))
     (stroke (width 0) (type solid) (color 0 0 0 0))
   )
@@
   (wire (pts (xy 262.89 142.24) (xy 262.89 144.78))
     (stroke (width 0) (type default) (color 0 0 0 0))
+  )
+  (wire (pts (xy 217.17 110.49) (xy 233.68 110.49))
+    (stroke (width 0) (type solid) (color 0 0 0 0))
   )
   (wire (pts (xy 228.6 49.53) (xy 237.49 49.53))
@@
     (effects (font (size 1.27 1.27)) (justify left bottom))
   )
-  (label "USBD_P" (at 262.89 110.49 0)
-    (effects (font (size 1.27 1.27)) (justify left bottom))
-  )
   (label "TRD0_N" (at 200.66 57.15 180)
     (effects (font (size 1.27 1.27)) (justify right bottom))
@@
     (effects (font (size 1.27 1.27)) (justify left bottom))
   )
+  (label "USB2_P" (at 262.89 105.41 0)
+    (effects (font (size 1.27 1.27)) (justify left bottom))
+  )
   (label "SD_DAT2" (at 107.95 116.84 180)
     (effects (font (size 1.27 1.27)) (justify right bottom))
@@
     (effects (font (size 1.27 1.27)) (justify left bottom))
   )
+  (label "USB2_P" (at 223.52 105.41 0)
+    (effects (font (size 1.27 1.27)) (justify left bottom))
+  )
   (label "USB2_P" (at 157.48 115.57 0)
     (effects (font (size 1.27 1.27)) (justify left bottom))
@@
     (effects (font (size 1.27 1.27)) (justify right bottom))
   )
-  (label "USBD_N" (at 262.89 105.41 0)
+  (label "USB2_N" (at 223.52 110.49 0)
     (effects (font (size 1.27 1.27)) (justify left bottom))
   )
@@
     (effects (font (size 1.27 1.27)) (justify left bottom))
   )
+  (label "USB2_N" (at 262.89 110.49 0)
+    (effects (font (size 1.27 1.27)) (justify left bottom))
+  )

Commit message: .
.
Connections:
- net MXCT: now reaches C39.1, J2.1 (MXCT3), J2.12 (MXCT1), J2.6 (MXCT2), J2.7 (MXCT4)
- net LED_GREEN: now reaches J2.14 (LED2-), R11.1
- net LED_YELLOW: now reaches J2.15 (LED1-), R10.1
Changed lines of the file:
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@@
+    (effects (font (size 1.27 1.27)) (justify left bottom))
+  )
+  (label "MXCT" (at 220.98 41.91 0)
     (effects (font (size 1.27 1.27)) (justify left bottom))
   )
@@
     (effects (font (size 1.27 1.27)) (justify left bottom))
   )
+  (label "LED_YELLOW" (at 228.6 24.13 0)
+    (effects (font (size 1.27 1.27)) (justify left bottom))
+  )
+  (label "LED_GREEN" (at 228.2336 72.39 0)
+    (effects (font (size 1.27 1.27)) (justify left bottom))
+  )
