File: audio/CM4_LOW_SPEED.kicad_sch (KiCad schematic)
At the start: 15 parts, among them J2 JK00177, J4 1054500101, U5 TPD4EUSB30, U6 TPD4EUSB30, U7 TPD4EUSB30

Commit message: .
.
Connections:
- net +3.3v is gone; now on net 3.3V: J2.13 (LED2+), J2.16 (LED1+)
Changed lines of the file:
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@@
     (effects (font (size 1.27 1.27)) (justify right bottom))
   )
-  (label "+3.3v" (at 236.22 21.59 180)
+  (label "3.3V" (at 236.22 21.59 180)
     (effects (font (size 1.27 1.27)) (justify right bottom))
   )
@@
     (effects (font (size 1.27 1.27)) (justify right bottom))
   )
-  (label "+3.3v" (at 236.22 69.85 180)
+  (label "3.3V" (at 236.22 69.85 180)
     (effects (font (size 1.27 1.27)) (justify right bottom))
   )

Commit message: .
.
Connections:
- net 5V is gone; now on net VBUS: R12.1, R14.1
- net USB2_N: no longer U7.2 (D1-), U7.9
- net USB2_P: no longer U7.1 (D1+), U7.10
- new net: U7.1 (D1+), U7.10
- new net: U7.2 (D1-), U7.9
Changed lines of the file:
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@@
+    (effects (font (size 1.27 1.27)) (justify left bottom))
+  )
+  (label "VBUS" (at 266.4996 128.27 0)
     (effects (font (size 1.27 1.27)) (justify left bottom))
   )
@@
   )
   (label "TRD2_P" (at 99.314 43.18 0)
-    (effects (font (size 1.27 1.27)) (justify left bottom))
-  )
-  (label "5V" (at 267.97 128.27 0)
     (effects (font (size 1.27 1.27)) (justify left bottom))
   )
@@
     (effects (font (size 1.27 1.27)) (justify left bottom))
   )
-  (label "USB2_P" (at 223.52 105.41 0)
-    (effects (font (size 1.27 1.27)) (justify left bottom))
-  )
   (label "USB2_P" (at 157.48 115.57 0)
     (effects (font (size 1.27 1.27)) (justify left bottom))
@@
     (effects (font (size 1.27 1.27)) (justify right bottom))
   )
-  (label "USB2_N" (at 223.52 110.49 0)
-    (effects (font (size 1.27 1.27)) (justify left bottom))
-  )
   (label "GND" (at 132.08 96.52 0)

Commit message: .
.
Parts:
- added R36: 30K 1%, Resistor_SMD:R_0402_1005Metric, symbol Device:R
Connections:
- net 3.3V: now also CM4_MODULE1.78 (GPIO_VREF(1.8v/3.3v_Input))
- net GND: now also CM4_MODULE1.1 (GND), CM4_MODULE1.13 (GND), CM4_MODULE1.14 (GND), CM4_MODULE1.2 (GND), CM4_MODULE1.22 (GND), CM4_MODULE1.23 (GND), CM4_MODULE1.32 (GND), CM4_MODULE1.33 (GND), CM4_MODULE1.42 (GND), CM4_MODULE1.43 (GND), CM4_MODULE1.52 (GND), CM4_MODULE1.53 (GND), CM4_MODULE1.60 (GND), CM4_MODULE1.66 (GND), CM4_MODULE1.7 (GND), CM4_MODULE1.71 (GND), CM4_MODULE1.74 (GND), CM4_MODULE1.8 (GND), R36.2
- net +5V: now reaches CM4_MODULE1.77 (+5v_(Input))
- net +5V: now also CM4_MODULE1.79 (+5v_(Input)), CM4_MODULE1.81 (+5v_(Input)), CM4_MODULE1.83 (+5v_(Input)), CM4_MODULE1.85 (+5v_(Input)), CM4_MODULE1.87 (+5v_(Input))
- net nRPIBOOT: now reaches CM4_MODULE1.93 (nRPIBOOT)
- net nRPIBOOT: now also R36.1

Commit message: .
.
Connections:
- net nEXTRST: now reaches CM4_MODULE1.100 (nEXTRST)
- net GLOBAL_EN: now reaches CM4_MODULE1.99 (Global_EN)
Changed lines of the file:
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@@
     (stroke (width 0) (type solid) (color 0 0 0 0))
+  )
+  (wire (pts (xy 20.32 154.94) (xy 35.56 154.94))
+    (stroke (width 0) (type default) (color 0 0 0 0))
   )
   (wire (pts (xy 96.52 48.26) (xy 109.474 48.26))
@@
   (wire (pts (xy 35.56 134.62) (xy 35.56 137.16))
     (stroke (width 0) (type default) (color 0 0 0 0))
+  )
+  (wire (pts (xy 96.52 154.94) (xy 113.03 154.94))
+    (stroke (width 0) (type solid) (color 0 0 0 0))
   )
   (wire (pts (xy 153.67 118.11) (xy 168.91 118.11))
@@
     (effects (font (size 1.27 1.27)) (justify left bottom))
   )
+  (label "GLOBAL_EN" (at 110.49 154.94 180)
+    (effects (font (size 1.27 1.27)) (justify right bottom))
+  )
   (label "I2C1_SCL" (at 25.4 99.06 0)
     (effects (font (size 1.27 1.27)) (justify left bottom))
@@
   (label "TRD0_P" (at 236.22 29.21 180)
     (effects (font (size 1.27 1.27)) (justify right bottom))
+  )
+  (label "nEXTRST" (at 24.13 154.94 0)
+    (effects (font (size 1.27 1.27)) (justify left bottom))
   )
   (label "nRPIBOOT" (at 101.6 147.32 0)
@@
     (effects (font (size 1.27 1.27)) (justify right))
   )
+  (hierarchical_label "nEXTRST" (shape output) (at 20.32 154.94 180)
+    (effects (font (size 1.27 1.27)) (justify right))
+  )
+  (hierarchical_label "GLOBAL_EN" (shape input) (at 113.03 154.94 0)
+    (effects (font (size 1.27 1.27)) (justify left))
+  )
   (hierarchical_label "I2S_LRCK" (shape bidirectional) (at 22.606 60.96 180)

Commit message: .
.
Parts:
- R10, R11: value 470R -> 2k
Connections:
- net 3.3V: no longer J2.13 (LED2+), J2.16 (LED1+)
- new net 5V: J2.13 (LED2+), J2.16 (LED1+)
Changed lines of the file:
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@@
     (effects (font (size 1.27 1.27)) (justify left bottom))
   )
-  (label "3.3V" (at 236.22 21.59 180)
+  (label "5V" (at 236.22 21.59 180)
     (effects (font (size 1.27 1.27)) (justify right bottom))
   )
@@
     (effects (font (size 1.27 1.27)) (justify right bottom))
   )
-  (label "3.3V" (at 236.22 69.85 180)
+  (label "5V" (at 236.22 69.85 180)
     (effects (font (size 1.27 1.27)) (justify right bottom))
   )
@@
     (in_bom yes) (on_board yes)
     (property "Reference" "R11" (id 0) (at 223.52 67.1322 90))
-    (property "Value" "470R" (id 1) (at 223.52 69.4436 90))
+    (property "Value" "2k" (id 1) (at 223.52 69.4436 90))
     (property "Footprint" "Resistor_SMD:R_0402_1005Metric" (id 2) (at 223.52 70.612 90)
       (effects (font (size 1.27 1.27)) hide)
@@
     (in_bom yes) (on_board yes)
     (property "Reference" "R10" (id 0) (at 223.52 29.21 90))
-    (property "Value" "470R" (id 1) (at 223.52 26.67 90))
+    (property "Value" "2k" (id 1) (at 223.52 26.67 90))
     (property "Footprint" "Resistor_SMD:R_0402_1005Metric" (id 2) (at 223.52 22.352 90)
       (effects (font (size 1.27 1.27)) hide)
