File: audio/CM4_LOW_SPEED.kicad_sch (KiCad schematic)
At the start: 16 parts, among them J2 JK00177, J4 1054500101, U5 TPD4EUSB30, U6 TPD4EUSB30, U7 TPD4EUSB30

Commit message: .
.
Parts:
- R12, R13, R14, R15: value 5.1K 5% -> NC
Changed lines of the file:
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@@
       (effects (font (size 1.27 1.27)) (justify left))
     )
-    (property "Value" "5.1K 5%" (at 264.668 149.733 0)
+    (property "Value" "NC" (at 264.668 149.733 0)
       (effects (font (size 1.27 1.27)) (justify left))
     )
@@
       (effects (font (size 1.27 1.27)) (justify left))
     )
-    (property "Value" "5.1K 5%" (at 250.698 138.303 0)
+    (property "Value" "NC" (at 250.698 138.303 0)
       (effects (font (size 1.27 1.27)) (justify left))
     )
@@
       (effects (font (size 1.27 1.27)) (justify left))
     )
-    (property "Value" "5.1K 5%" (at 264.668 138.303 0)
+    (property "Value" "NC" (at 264.668 138.303 0)
       (effects (font (size 1.27 1.27)) (justify left))
     )
@@
       (effects (font (size 1.27 1.27)) (justify left))
     )
-    (property "Value" "5.1K 5%" (at 250.698 149.733 0)
-      (effects (font (size 1.27 1.27)) (justify left))
-    )
+    (property "Value" "NC" (at 250.698 149.733 0)
+      (effects (font (size 1.27 1.27)) (justify left))
+    )

Commit message: .
.
Parts:
- R10, R11: value 2k -> 2.2K 1%
Changed lines of the file:
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@@
       (effects (font (size 1.27 1.27)))
     )
-    (property "Value" "2k" (at 223.52 69.4436 90)
+    (property "Value" "2.2K 1%" (at 223.52 69.4436 90)
       (effects (font (size 1.27 1.27)))
     )
@@
       (effects (font (size 1.27 1.27)))
     )
-    (property "Value" "2k" (at 223.52 26.67 90)
+    (property "Value" "2.2K 1%" (at 223.52 26.67 90)
       (effects (font (size 1.27 1.27)))
     )

Commit message: ,
,
Parts:
- R36: value 30K 1% -> 15K 1%
Changed lines of the file:
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@@
       (effects (font (size 1.27 1.27)) (justify left))
     )
-    (property "Value" "30K 1%" (at 113.538 162.433 0)
+    (property "Value" "15K 1%" (at 113.538 162.433 0)
       (effects (font (size 1.27 1.27)) (justify left))
     )

Commit message: USB_OK
.
Parts:
- R13, R15: value NC -> 5.1k
- R16, R18: value 2.2K 1% -> NC
Changed lines of the file:
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@@
       (effects (font (size 1.27 1.27)) (justify left))
     )
-    (property "Value" "NC" (at 264.668 149.733 0)
+    (property "Value" "5.1k" (at 264.668 149.733 0)
       (effects (font (size 1.27 1.27)) (justify left))
     )
@@
       (effects (font (size 1.27 1.27)) (justify left))
     )
-    (property "Value" "2.2K 1%" (at 145.288 106.553 0)
+    (property "Value" "NC" (at 145.288 106.553 0)
       (effects (font (size 1.27 1.27)) (justify left))
     )
@@
       (effects (font (size 1.27 1.27)) (justify left))
     )
-    (property "Value" "2.2K 1%" (at 132.588 106.553 0)
+    (property "Value" "NC" (at 132.588 106.553 0)
       (effects (font (size 1.27 1.27)) (justify left))
     )
@@
       (effects (font (size 1.27 1.27)) (justify left))
     )
-    (property "Value" "NC" (at 250.698 149.733 0)
-      (effects (font (size 1.27 1.27)) (justify left))
-    )
+    (property "Value" "5.1k" (at 250.698 149.733 0)
+      (effects (font (size 1.27 1.27)) (justify left))
+    )
