File: audio/isolation_module.kicad_sch (KiCad schematic)
At the start: 0 parts

Commit message: .
.
Parts:
- added J8, J9: Conn_01x10, Connector_PinSocket_2.54mm:PinSocket_1x10_P2.54mm_Vertical, symbol Connector_Generic:Conn_01x10
- added PS1: R05CTE05S-R, CM4IO:SOIC127P1030X265-16N, symbol CM4IO:R05CTE05S-R
Connections:
- new net +5V: J8.1 (Pin_1), J8.2 (Pin_2)
- new net 3.3V: J8.3 (Pin_3)
- new net GND: J8.10 (Pin_10), J8.4 (Pin_4), J8.6 (Pin_6), J8.8 (Pin_8), J9.1 (Pin_1), J9.10 (Pin_10), J9.2 (Pin_2), J9.3 (Pin_3), J9.4 (Pin_4), J9.5 (Pin_5), J9.6 (Pin_6), J9.8 (Pin_8)
- new net I2C1_SCL: J9.9 (Pin_9)
- new net I2C1_SDA: J9.7 (Pin_7)
- new net I2S_ADC: J8.7 (Pin_7)
- new net I2S_BCLK: J8.9 (Pin_9)
- new net I2S_LRCK: J8.5 (Pin_5)
Changed lines of the file:
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@@
 (kicad_sch (version 20211123) (generator eeschema)
   (paper "A4")
+  (wire (pts (xy 50.8 120.65) (xy 66.04 120.65))
+    (stroke (width 0) (type default) (color 0 0 0 0))
+  )
+  (wire (pts (xy 50.8 72.39) (xy 66.04 72.39))
+    (stroke (width 0) (type default) (color 0 0 0 0))
+  )
+  (wire (pts (xy 50.8 77.47) (xy 66.04 77.47))
+    (stroke (width 0) (type default) (color 0 0 0 0))
+  )
+  (wire (pts (xy 50.8 100.33) (xy 66.04 100.33))
+    (stroke (width 0) (type default) (color 0 0 0 0))
+  )
+  (wire (pts (xy 50.8 82.55) (xy 66.04 82.55))
+    (stroke (width 0) (type default) (color 0 0 0 0))
+  )
+  (wire (pts (xy 50.8 80.01) (xy 66.04 80.01))
+    (stroke (width 0) (type default) (color 0 0 0 0))
+  )
+  (wire (pts (xy 50.8 118.11) (xy 66.04 118.11))
+    (stroke (width 0) (type default) (color 0 0 0 0))
+  )
+  (wire (pts (xy 50.8 59.69) (xy 66.04 59.69))
+    (stroke (width 0) (type default) (color 0 0 0 0))
+  )
+  (wire (pts (xy 50.8 105.41) (xy 66.04 105.41))
+    (stroke (width 0) (type default) (color 0 0 0 0))
+  )
+  (wire (pts (xy 50.8 110.49) (xy 66.04 110.49))
+    (stroke (width 0) (type default) (color 0 0 0 0))
+  )
+  (wire (pts (xy 50.8 69.85) (xy 66.04 69.85))
+    (stroke (width 0) (type default) (color 0 0 0 0))
+  )
+  (wire (pts (xy 50.8 64.77) (xy 66.04 64.77))
+    (stroke (width 0) (type default) (color 0 0 0 0))
+  )
+  (wire (pts (xy 50.8 97.79) (xy 66.04 97.79))
+    (stroke (width 0) (type default) (color 0 0 0 0))
+  )
+  (wire (pts (xy 50.8 74.93) (xy 66.04 74.93))
+    (stroke (width 0) (type default) (color 0 0 0 0))
+  )
+  (wire (pts (xy 50.8 102.87) (xy 66.04 102.87))
+    (stroke (width 0) (type default) (color 0 0 0 0))
+  )
+  (wire (pts (xy 50.8 115.57) (xy 66.04 115.57))
+    (stroke (width 0) (type default) (color 0 0 0 0))
+  )
+  (wire (pts (xy 50.8 62.23) (xy 66.04 62.23))
+    (stroke (width 0) (type default) (color 0 0 0 0))
+  )
+  (wire (pts (xy 50.8 67.31) (xy 66.04 67.31))
+    (stroke (width 0) (type default) (color 0 0 0 0))
+  )
+  (wire (pts (xy 50.8 113.03) (xy 66.04 113.03))
+    (stroke (width 0) (type default) (color 0 0 0 0))
+  )
+  (wire (pts (xy 50.8 107.95) (xy 66.04 107.95))
+    (stroke (width 0) (type default) (color 0 0 0 0))
+  )
+  (label "I2S_LRCK" (at 54.61 72.39 0)
+    (effects (font (size 1.27 1.27)) (justify left bottom))
+  )
+  (label "GND" (at 54.61 64.77 0)
+    (effects (font (size 1.27 1.27)) (justify left bottom))
+  )
+  (label "+5V" (at 54.61 80.01 0)
+    (effects (font (size 1.27 1.27)) (justify left bottom))
+  )
+  (label "3.3V" (at 54.61 77.47 0)
+    (effects (font (size 1.27 1.27)) (justify left bottom))
+  )
+  (label "GND" (at 54.61 113.03 0)
+    (effects (font (size 1.27 1.27)) (justify left bottom))
+  )
+  (label "I2S_ADC" (at 54.61 67.31 0)
+    (effects (font (size 1.27 1.27)) (justify left bottom))
+  )
+  (label "I2C1_SDA" (at 54.61 105.41 0)
+    (effects (font (size 1.27 1.27)) (justify left bottom))
+  )
+  (label "GND" (at 54.61 97.79 0)
+    (effects (font (size 1.27 1.27)) (justify left bottom))
+  )
+  (label "I2C1_SCL" (at 54.61 100.33 0)
+    (effects (font (size 1.27 1.27)) (justify left bottom))
+  )
+  (label "GND" (at 54.61 107.95 0)
+    (effects (font (size 1.27 1.27)) (justify left bottom))
+  )
+  (label "GND" (at 54.61 69.85 0)
+    (effects (font (size 1.27 1.27)) (justify left bottom))
+  )
+  (label "GND" (at 54.61 110.49 0)
+    (effects (font (size 1.27 1.27)) (justify left bottom))
+  )
+  (label "GND" (at 54.61 120.65 0)
+    (effects (font (size 1.27 1.27)) (justify left bottom))
+  )
+  (label "+5V" (at 54.61 82.55 0)
+    (effects (font (size 1.27 1.27)) (justify left bottom))
+  )
+  (label "I2S_BCLK" (at 54.61 62.23 0)
+    (effects (font (size 1.27 1.27)) (justify left bottom))
+  )
+  (label "GND" (at 54.61 102.87 0)
+    (effects (font (size 1.27 1.27)) (justify left bottom))
+  )
+  (label "GND" (at 54.61 115.57 0)
+    (effects (font (size 1.27 1.27)) (justify left bottom))
+  )
+  (label "GND" (at 54.61 59.69 0)
+    (effects (font (size 1.27 1.27)) (justify left bottom))
+  )
+  (label "GND" (at 54.61 118.11 0)
+    (effects (font (size 1.27 1.27)) (justify left bottom))
+  )
+  (label "GND" (at 54.61 74.93 0)
+    (effects (font (size 1.27 1.27)) (justify left bottom))
+  )
+  (symbol (lib_id "Connector_Generic:Conn_01x10") (at 45.72 72.39 180) (unit 1)
+    (in_bom yes) (on_board yes) (fields_autoplaced)
+    (property "Reference" "J8" (id 0) (at 45.72 53.34 0))
+    (property "Value" "Conn_01x10" (id 1) (at 45.72 55.88 0))
+    (property "Footprint" "Connector_PinSocket_2.54mm:PinSocket_1x10_P2.54mm_Vertical" (id 2) (at 45.72 72.39 0)
+      (effects (font (size 1.27 1.27)) hide)
+    )
+    (property "Datasheet" "~" (id 3) (at 45.72 72.39 0)
+      (effects (font (size 1.27 1.27)) hide)
+    )
+    (pin "1")
+    (pin "10")
+    (pin "2")
+    (pin "3")
+    (pin "4")
+    (pin "5")
+    (pin "6")
+    (pin "7")
+    (pin "8")
+    (pin "9")
+  )
+  (symbol (lib_id "CM4IO:R05CTE05S-R") (at 82.55 59.69 0) (unit 1)
+    (in_bom yes) (on_board yes) (fields_autoplaced)
+    (property "Reference" "PS1" (id 0) (at 102.87 52.07 0))
+    (property "Value" "R05CTE05S-R" (id 1) (at 102.87 54.61 0))
+    (property "Footprint" "CM4IO:SOIC127P1030X265-16N" (id 2) (at 147.32 58.42 0)
+      (effects (font (size 1.27 1.27)) (justify left) hide)
+    )
+    (property "Datasheet" "https://recom-power.com/pdf/Econoline/RxxCTExxS.pdf" (id 3) (at 147.32 60.96 0)
+      (effects (font (size 1.27 1.27)) (justify left) hide)
+    )
+    (property "Description" "1 Watt 16-Pin SOIC Single Output, 5VDC, Tape & Reel" (id 4) (at 147.32 63.5 0)
+      (effects (font (size 1.27 1.27)) (justify left) hide)
+    )
+    (property "Height" "2.65" (id 5) (at 119.38 64.77 0)
+      (effects (font (size 1.27 1.27)) (justify left) hide)
+    )
+    (property "Manufacturer_Name" "RECOM Power" (id 6) (at 147.32 68.58 0)
+      (effects (font (size 1.27 1.27)) (justify left) hide)
+    )
+    (property "Manufacturer_Part_Number" "R05CTE05S-R" (id 7) (at 147.32 71.12 0)
+      (effects (font (size 1.27 1.27)) (justify left) hide)
+    )
+    (property "Mouser Part Number" "919-R05CTE05S-R" (id 8) (at 147.32 73.66 0)
+      (effects (font (size 1.27 1.27)) (justify left) hide)
+    )
+    (property "Mouser Price/Stock" "https://www.mouser.co.uk/ProductDetail/RECOM-Power/R05CTE05S-R?qs=7D1LtPJG0i0SUCKLd%252BnSSQ%3D%3D" (id 9) (at 147.32 76.2 0)
+      (effects (font (size 1.27 1.27)) (justify left) hide)
+    )
+    (property "Arrow Part Number" "" (id 10) (at 119.38 77.47 0)
+      (effects (font (size 1.27 1.27)) (justify left) hide)
+    )
+    (property "Arrow Price/Stock" "" (id 11) (at 119.38 80.01 0)
+      (effects (font (size 1.27 1.27)) (justify left) hide)
+    )
+    (property "Mouser Testing Part Number" "" (id 12) (at 119.38 82.55 0)
+      (effects (font (size 1.27 1.27)) (justify left) hide)
+    )
+    (property "Mouser Testing Price/Stock" "" (id 13) (at 119.38 85.09 0)
+      (effects (font (size 1.27 1.27)) (justify left) hide)
+    )
+    (pin "1")
+    (pin "10")
+    (pin "11")
+    (pin "12")
+    (pin "13")
+    (pin "14")
+    (pin "15")
+    (pin "16")
+    (pin "2")
+    (pin "3")
+    (pin "4")
+    (pin "5")
+    (pin "6")
+    (pin "7")
+    (pin "8")
+    (pin "9")
+  )
+  (symbol (lib_id "Connector_Generic:Conn_01x10") (at 45.72 110.49 180) (unit 1)
+    (in_bom yes) (on_board yes) (fields_autoplaced)
+    (property "Reference" "J9" (id 0) (at 45.72 91.44 0))
+    (property "Value" "Conn_01x10" (id 1) (at 45.72 93.98 0))
+    (property "Footprint" "Connector_PinSocket_2.54mm:PinSocket_1x10_P2.54mm_Vertical" (id 2) (at 45.72 110.49 0)
+      (effects (font (size 1.27 1.27)) hide)
+    )
+    (property "Datasheet" "~" (id 3) (at 45.72 110.49 0)
+      (effects (font (size 1.27 1.27)) hide)
+    )
+    (pin "1")
+    (pin "10")
+    (pin "2")
+    (pin "3")
+    (pin "4")
+    (pin "5")
+    (pin "6")
+    (pin "7")
+    (pin "8")
+    (pin "9")
+  )
 )

Commit message: .
.
Parts:
- added PS2: R05CTE05S-R, CM4IO:SOIC127P1030X265-16N, symbol CM4IO:R05CTE05S-R
- added U10: ac108, CM4IO:AC108, symbol CM4IO:ac108
- added U2: ISO1540, Package_SO:SOIC-8_3.9x4.9mm_P1.27mm, symbol Isolator:ISO1540
- added U9: SI8663BB-B-IS1, CM4IO:SI8663BB-B-IS1, symbol CM4IO:SI8663BB-B-IS1
Changed lines of the file:
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@@
     (effects (font (size 1.27 1.27)) (justify left bottom))
+  )
+  (symbol (lib_id "CM4IO:SI8663BB-B-IS1") (at 80.01 123.19 0) (unit 1)
+    (in_bom yes) (on_board yes) (fields_autoplaced)
+    (property "Reference" "U9" (id 0) (at 100.33 111.76 0)
+      (effects (font (size 1.524 1.524)))
+    )
+    (property "Value" "SI8663BB-B-IS1" (id 1) (at 100.33 115.57 0)
+      (effects (font (size 1.524 1.524)))
+    )
+    (property "Footprint" "CM4IO:SI8663BB-B-IS1" (id 2) (at 100.33 117.094 0)
+      (effects (font (size 1.524 1.524)) hide)
+    )
+    (property "Datasheet" "" (id 3) (at 80.01 123.19 0)
+      (effects (font (size 1.524 1.524)))
+    )
+    (pin "1")
+    (pin "10")
+    (pin "11")
+    (pin "12")
+    (pin "13")
+    (pin "14")
+    (pin "15")
+    (pin "16")
+    (pin "2")
+    (pin "3")
+    (pin "4")
+    (pin "5")
+    (pin "6")
+    (pin "7")
+    (pin "8")
+    (pin "9")
   )
   (symbol (lib_id "Connector_Generic:Conn_01x10") (at 45.72 72.39 180) (unit 1)
@@
     (pin "9")
   )
+  (symbol (lib_id "CM4IO:R05CTE05S-R") (at 140.97 59.69 0) (unit 1)
+    (in_bom yes) (on_board yes) (fields_autoplaced)
+    (property "Reference" "PS2" (id 0) (at 161.29 52.07 0))
+    (property "Value" "R05CTE05S-R" (id 1) (at 161.29 54.61 0))
+    (property "Footprint" "CM4IO:SOIC127P1030X265-16N" (id 2) (at 205.74 58.42 0)
+      (effects (font (size 1.27 1.27)) (justify left) hide)
+    )
+    (property "Datasheet" "https://recom-power.com/pdf/Econoline/RxxCTExxS.pdf" (id 3) (at 205.74 60.96 0)
+      (effects (font (size 1.27 1.27)) (justify left) hide)
+    )
+    (property "Description" "1 Watt 16-Pin SOIC Single Output, 5VDC, Tape & Reel" (id 4) (at 205.74 63.5 0)
+      (effects (font (size 1.27 1.27)) (justify left) hide)
+    )
+    (property "Height" "2.65" (id 5) (at 177.8 64.77 0)
+      (effects (font (size 1.27 1.27)) (justify left) hide)
+    )
+    (property "Manufacturer_Name" "RECOM Power" (id 6) (at 205.74 68.58 0)
+      (effects (font (size 1.27 1.27)) (justify left) hide)
+    )
+    (property "Manufacturer_Part_Number" "R05CTE05S-R" (id 7) (at 205.74 71.12 0)
+      (effects (font (size 1.27 1.27)) (justify left) hide)
+    )
+    (property "Mouser Part Number" "919-R05CTE05S-R" (id 8) (at 205.74 73.66 0)
+      (effects (font (size 1.27 1.27)) (justify left) hide)
+    )
+    (property "Mouser Price/Stock" "https://www.mouser.co.uk/ProductDetail/RECOM-Power/R05CTE05S-R?qs=7D1LtPJG0i0SUCKLd%252BnSSQ%3D%3D" (id 9) (at 205.74 76.2 0)
+      (effects (font (size 1.27 1.27)) (justify left) hide)
+    )
+    (property "Arrow Part Number" "" (id 10) (at 177.8 77.47 0)
+      (effects (font (size 1.27 1.27)) (justify left) hide)
+    )
+    (property "Arrow Price/Stock" "" (id 11) (at 177.8 80.01 0)
+      (effects (font (size 1.27 1.27)) (justify left) hide)
+    )
+    (property "Mouser Testing Part Number" "" (id 12) (at 177.8 82.55 0)
+      (effects (font (size 1.27 1.27)) (justify left) hide)
+    )
+    (property "Mouser Testing Price/Stock" "" (id 13) (at 177.8 85.09 0)
+      (effects (font (size 1.27 1.27)) (justify left) hide)
+    )
+    (pin "1")
+    (pin "10")
+    (pin "11")
+    (pin "12")
+    (pin "13")
+    (pin "14")
+    (pin "15")
+    (pin "16")
+    (pin "2")
+    (pin "3")
+    (pin "4")
+    (pin "5")
+    (pin "6")
+    (pin "7")
+    (pin "8")
+    (pin "9")
+  )
   (symbol (lib_id "CM4IO:R05CTE05S-R") (at 82.55 59.69 0) (unit 1)
     (in_bom yes) (on_board yes) (fields_autoplaced)
@@
     (pin "9")
   )
+  (symbol (lib_id "Isolator:ISO1540") (at 95.25 100.33 0) (unit 1)
+    (in_bom yes) (on_board yes) (fields_autoplaced)
+    (property "Reference" "U2" (id 0) (at 95.25 90.17 0))
+    (property "Value" "ISO1540" (id 1) (at 95.25 92.71 0))
+    (property "Footprint" "Package_SO:SOIC-8_3.9x4.9mm_P1.27mm" (id 2) (at 95.25 109.22 0)
+      (effects (font (size 1.27 1.27)) hide)
+    )
+    (property "Datasheet" "http://www.ti.com/lit/ds/symlink/iso1541.pdf" (id 3) (at 95.25 99.06 0)
+      (effects (font (size 1.27 1.27)) hide)
+    )
+    (pin "1")
+    (pin "2")
+    (pin "3")
+    (pin "4")
+    (pin "5")
+    (pin "6")
+    (pin "7")
+    (pin "8")
+  )
   (symbol (lib_id "Connector_Generic:Conn_01x10") (at 45.72 110.49 180) (unit 1)
     (in_bom yes) (on_board yes) (fields_autoplaced)
@@
     (pin "9")
   )
+  (symbol (lib_id "CM4IO:ac108") (at 196.85 44.45 0) (unit 1)
+    (in_bom yes) (on_board yes) (fields_autoplaced)
+    (property "Reference" "U10" (id 0) (at 237.49 41.91 0))
+    (property "Value" "ac108" (id 1) (at 237.49 44.45 0))
+    (property "Footprint" "CM4IO:AC108" (id 2) (at 196.85 44.45 0)
+      (effects (font (size 1.27 1.27)) hide)
+    )
+    (property "Datasheet" "" (id 3) (at 196.85 44.45 0)
+      (effects (font (size 1.27 1.27)) hide)
+    )
+    (pin "1")
+    (pin "10")
+    (pin "11")
+    (pin "12")
+    (pin "13")
+    (pin "14")
+    (pin "15")
+    (pin "16")
+    (pin "17")
+    (pin "18")
+    (pin "19")
+    (pin "2")
+    (pin "20")
+    (pin "21")
+    (pin "22")
+    (pin "23")
+    (pin "24")
+    (pin "25")
+    (pin "26")
+    (pin "27")
+    (pin "28")
+    (pin "29")
+    (pin "3")
+    (pin "30")
+    (pin "31")
+    (pin "32")
+    (pin "33")
+    (pin "34")
+    (pin "35")
+    (pin "36")
+    (pin "37")
+    (pin "38")
+    (pin "39")
+    (pin "4")
+    (pin "40")
+    (pin "41")
+    (pin "42")
+    (pin "43")
+    (pin "44")
+    (pin "45")
+    (pin "46")
+    (pin "47")
+    (pin "48")
+    (pin "5")
+    (pin "6")
+    (pin "7")
+    (pin "8")
+    (pin "9")
+    (pin "PAD")
+  )
 )

Commit message: .
.
Parts:
- removed U10: ac108, CM4IO:AC108, symbol CM4IO:ac108
Changed lines of the file:
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@@
     (pin "9")
   )
-  (symbol (lib_id "CM4IO:ac108") (at 196.85 44.45 0) (unit 1)
-    (in_bom yes) (on_board yes) (fields_autoplaced)
-    (property "Reference" "U10" (id 0) (at 237.49 41.91 0))
-    (property "Value" "ac108" (id 1) (at 237.49 44.45 0))
-    (property "Footprint" "CM4IO:AC108" (id 2) (at 196.85 44.45 0)
-      (effects (font (size 1.27 1.27)) hide)
-    )
-    (property "Datasheet" "" (id 3) (at 196.85 44.45 0)
-      (effects (font (size 1.27 1.27)) hide)
-    )
-    (pin "1")
-    (pin "10")
-    (pin "11")
-    (pin "12")
-    (pin "13")
-    (pin "14")
-    (pin "15")
-    (pin "16")
-    (pin "17")
-    (pin "18")
-    (pin "19")
-    (pin "2")
-    (pin "20")
-    (pin "21")
-    (pin "22")
-    (pin "23")
-    (pin "24")
-    (pin "25")
-    (pin "26")
-    (pin "27")
-    (pin "28")
-    (pin "29")
-    (pin "3")
-    (pin "30")
-    (pin "31")
-    (pin "32")
-    (pin "33")
-    (pin "34")
-    (pin "35")
-    (pin "36")
-    (pin "37")
-    (pin "38")
-    (pin "39")
-    (pin "4")
-    (pin "40")
-    (pin "41")
-    (pin "42")
-    (pin "43")
-    (pin "44")
-    (pin "45")
-    (pin "46")
-    (pin "47")
-    (pin "48")
-    (pin "5")
-    (pin "6")
-    (pin "7")
-    (pin "8")
-    (pin "9")
-    (pin "PAD")
-  )
 )

Commit message: .
.
Other:
- moved on the sheet: PS1, PS2, U2, U9

Commit message: .
.
Parts:
- removed PS2: R05CTE05S-R, CM4IO:SOIC127P1030X265-16N, symbol CM4IO:R05CTE05S-R
- added C? (x4): 10uF, Capacitor_SMD:C_0402_1005Metric, symbol Device:C_Small
- added C? (x4): 0.1uF, Capacitor_SMD:C_0402_1005Metric, symbol Device:C_Small
- added PS?: R05CTE05S-R, CM4IO:SOIC127P1030X265-16N, symbol CM4IO:R05CTE05S-R
- added R? (x2): 1k, Resistor_SMD:R_0603_1608Metric, symbol Device:R_Small_US
Connections:
- net +5V: now also PS1.3 (+VIN_1), PS1.4 (+VIN_2), C?.1, C?.1
- net 3.3V: now also U2.1 (VCC1), R?.1, R?.1
- net GND: now also PS1.1 (-VIN_1), PS1.2 (-VIN_2), PS1.5 (SGNDIN_1), PS1.6 (SGNDIN_2), PS1.7 (SGNDIN_3), PS1.8 (SGNDIN_4), U2.4 (GND1), C?.2, C?.2
- net I2C1_SCL: now also U2.3 (SCL1), R?.2
- net I2C1_SDA: now also U2.2 (SDA1), R?.2
- net VDD_GND: now reaches PS1.11 (SGNDOUT_2)
- net VDD_GND: now also PS1.12 (SGNDOUT_3), PS1.15 (-VOUT_1), PS1.16 (-VOUT_2), PS1.9 (SGNDOUT_1), U2.5 (GND2), C?.2, C?.2, C?.2, C?.2, PS?.1 (-VIN_1), PS?.2 (-VIN_2), PS?.5 (SGNDIN_1), PS?.6 (SGNDIN_2), PS?.7 (SGNDIN_3), PS?.8 (SGNDIN_4)
- net VDD_5V: now reaches PS1.13 (+VOUT_1)
- net VDD_5V: now also PS1.14 (+VOUT_2), C?.1, C?.1, C?.1, C?.1, PS?.3 (+VIN_1), PS?.4 (+VIN_2)
- net ISO_SCL: now reaches U2.6 (SCL2)
- net ISO_SDA: now reaches U2.7 (SDA2)
- net VDD_3.3V: now reaches U2.8 (VCC2)
- new net AVCC_5V: C?.1, C?.1, PS?.13 (+VOUT_1), PS?.14 (+VOUT_2)
- new net AVCC_GND: C?.2, C?.2, PS?.11 (SGNDOUT_2), PS?.12 (SGNDOUT_3), PS?.15 (-VOUT_1), PS?.16 (-VOUT_2), PS?.9 (SGNDOUT_1)
Other:
- moved on the sheet: PS1, U2, U9

Commit message: .
.
Parts:
- added C58, C67: 1uF, Capacitor_SMD:C_0402_1005Metric, symbol Device:C_Small
- added C59, C62, C65, C66: 0.1uF, Capacitor_SMD:C_0402_1005Metric, symbol Device:C_Small
- added R42, R43, R44, R45, R50, R51, R52, R53: 0, Resistor_SMD:R_0603_1608Metric, symbol Device:R_Small_US
- added R48, R49: 1k, Resistor_SMD:R_0603_1608Metric, symbol Device:R_Small_US
- gave numbers to parts that had none: 11
Connections:
- net 3.3V: now also U9.1 (VDD1), C58.1, C59.2, C62.1
- net GND: now also U9.8 (GND1), C58.2, C59.1, C62.2
- net I2S_ADC: now also U9.7 (A6)
- net I2S_BCLK: now also R42.1, R43.1
- net I2S_LRCK: now also R44.1, R45.1
- net ISO_SCL: now also R49.2
- net ISO_SDA: now also R48.2
- net VDD_3.3V: now also U9.16 (VDD2), C65.2, C66.1, C67.2, R48.1, R49.1
- net VDD_GND: now also U9.9 (GND2), C65.1, C66.2, C67.1
- net ISO_ADC: now reaches U9.10 (B6)
- net ISO_LRCK_TX: now reaches U9.11 (B5)
- net ISO_LRCK_TX: now also R53.2
- net ISO_BCLK_TX: now reaches U9.12 (B4)
- net ISO_BCLK_TX: now also R51.2
- net ISO_LRCK_RX: now reaches U9.13 (B3)
- net ISO_LRCK_RX: now also R52.2
- net ISO_BCLK_RX: now reaches U9.14 (B2)
- net ISO_BCLK_RX: now also R50.2
- net I2S_BCLK_TX: now reaches U9.3 (A2)
- net I2S_BCLK_TX: now also R42.2
- net I2S_LRCK_TX: now reaches U9.4 (A3)
- net I2S_LRCK_TX: now also R44.2
- net I2S_BCLK_RX: now reaches U9.5 (A4)
- net I2S_BCLK_RX: now also R43.2
- net I2S_LRCK_RX: now reaches U9.6 (A5)
- net I2S_LRCK_RX: now also R45.2
- new net ISO_BCLK: R50.1, R51.1
- new net ISO_LRCK: R52.1, R53.1
Other:
- moved on the sheet: C60, C61, C63, C64, C68, C69, C70, C71, J8, J9, PS1, PS2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
