File: audio/isolation_module.kicad_sch (KiCad schematic)
At the start: 32 parts, among them J8 Conn_01x10, J9 Conn_01x10, U2 ISO1540, U9 SI8663BB-B-IS1

Commit message: .
.
Connections:
- net +5V: now also J8.3 (Pin_3), J9.10 (Pin_10), J9.2 (Pin_2), J9.3 (Pin_3), J9.4 (Pin_4); no longer J8.1 (Pin_1), J8.2 (Pin_2)
- net 3.3V: now also J8.4 (Pin_4), J9.1 (Pin_1); no longer J8.3 (Pin_3)
- net GND: no longer J8.4 (Pin_4), J9.1 (Pin_1), J9.10 (Pin_10), J9.2 (Pin_2), J9.3 (Pin_3), J9.4 (Pin_4)
- net I2C1_SCL: now also J9.7 (Pin_7); no longer J9.9 (Pin_9)
- net I2C1_SDA: now also J9.9 (Pin_9); no longer J9.7 (Pin_7)
- new net USB_DEBUG_N: J8.1 (Pin_1)
- new net USB_DEBUG_P: J8.2 (Pin_2)
Changed lines of the file:
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@@
+    (effects (font (size 1.27 1.27)) (justify left bottom))
+  )
+  (label "+5V" (at 41.91 123.19 0)
     (effects (font (size 1.27 1.27)) (justify left bottom))
   )
@@
     (effects (font (size 1.27 1.27)) (justify left bottom))
   )
-  (label "+5V" (at 41.91 83.82 0)
-    (effects (font (size 1.27 1.27)) (justify left bottom))
-  )
   (label "I2C1_SCL" (at 134.62 121.92 0)
     (effects (font (size 1.27 1.27)) (justify left bottom))
@@
     (effects (font (size 1.27 1.27)) (justify left bottom))
   )
+  (label "+5V" (at 41.91 81.28 0)
+    (effects (font (size 1.27 1.27)) (justify left bottom))
+  )
   (label "3.3V" (at 121.92 152.4 0)
     (effects (font (size 1.27 1.27)) (justify left bottom))
@@
     (effects (font (size 1.27 1.27)) (justify left bottom))
   )
-  (label "3.3V" (at 41.91 81.28 0)
-    (effects (font (size 1.27 1.27)) (justify left bottom))
-  )
   (label "VDD_5V" (at 271.78 67.31 0)
     (effects (font (size 1.27 1.27)) (justify left bottom))
   )
+  (label "USB_DEBUG_N" (at 41.91 86.36 0)
+    (effects (font (size 1.27 1.27)) (justify left bottom))
+  )
   (label "I2S_LRCK_RX" (at 121.92 165.1 0)
     (effects (font (size 1.27 1.27)) (justify left bottom))
@@
     (effects (font (size 1.27 1.27)) (justify left bottom))
   )
+  (label "USB_DEBUG_P" (at 41.91 83.82 0)
+    (effects (font (size 1.27 1.27)) (justify left bottom))
+  )
   (label "AVCC_GND" (at 322.58 72.39 0)
     (effects (font (size 1.27 1.27)) (justify left bottom))
   )
-  (label "GND" (at 41.91 118.11 0)
+  (label "+5V" (at 41.91 120.65 0)
     (effects (font (size 1.27 1.27)) (justify left bottom))
   )
@@
     (effects (font (size 1.27 1.27)) (justify left bottom))
   )
-  (label "I2C1_SDA" (at 41.91 110.49 0)
-    (effects (font (size 1.27 1.27)) (justify left bottom))
-  )
-  (label "GND" (at 41.91 102.87 0)
+  (label "I2C1_SDA" (at 41.91 105.41 0)
     (effects (font (size 1.27 1.27)) (justify left bottom))
   )
@@
     (effects (font (size 1.27 1.27)) (justify left bottom))
   )
-  (label "I2C1_SCL" (at 41.91 105.41 0)
+  (label "I2C1_SCL" (at 41.91 110.49 0)
     (effects (font (size 1.27 1.27)) (justify left bottom))
   )
@@
     (effects (font (size 1.27 1.27)) (justify left bottom))
   )
+  (label "3.3V" (at 41.91 125.73 0)
+    (effects (font (size 1.27 1.27)) (justify left bottom))
+  )
   (label "+5V" (at 128.27 67.31 0)
     (effects (font (size 1.27 1.27)) (justify left bottom))
@@
     (effects (font (size 1.27 1.27)) (justify left bottom))
   )
+  (label "+5V" (at 41.91 102.87 0)
+    (effects (font (size 1.27 1.27)) (justify left bottom))
+  )
   (label "GND" (at 134.62 124.46 0)
     (effects (font (size 1.27 1.27)) (justify left bottom))
@@
     (effects (font (size 1.27 1.27)) (justify left bottom))
   )
-  (label "GND" (at 41.91 125.73 0)
-    (effects (font (size 1.27 1.27)) (justify left bottom))
-  )
-  (label "+5V" (at 41.91 86.36 0)
-    (effects (font (size 1.27 1.27)) (justify left bottom))
-  )
   (label "ISO_LRCK_RX" (at 199.39 182.88 0)
     (effects (font (size 1.27 1.27)) (justify left bottom))
   )
+  (label "+5V" (at 41.91 118.11 0)
+    (effects (font (size 1.27 1.27)) (justify left bottom))
+  )
   (label "ISO_SCL" (at 170.18 121.92 0)
     (effects (font (size 1.27 1.27)) (justify left bottom))
@@
     (effects (font (size 1.27 1.27)) (justify left bottom))
   )
-  (label "GND" (at 41.91 120.65 0)
-    (effects (font (size 1.27 1.27)) (justify left bottom))
-  )
   (label "GND" (at 41.91 63.5 0)
     (effects (font (size 1.27 1.27)) (justify left bottom))
@@
     (effects (font (size 1.27 1.27)) (justify left bottom))
   )
+  (label "3.3V" (at 41.91 78.74 0)
+    (effects (font (size 1.27 1.27)) (justify left bottom))
+  )
   (label "VDD_GND" (at 199.39 62.23 0)
     (effects (font (size 1.27 1.27)) (justify left bottom))
   )
-  (label "GND" (at 41.91 123.19 0)
-    (effects (font (size 1.27 1.27)) (justify left bottom))
-  )
   (label "GND" (at 116.84 116.84 0)
     (effects (font (size 1.27 1.27)) (justify left bottom))
   )
-  (label "GND" (at 41.91 78.74 0)
-    (effects (font (size 1.27 1.27)) (justify left bottom))
-  )
   (label "I2S_BCLK" (at 76.2 165.1 0)
     (effects (font (size 1.27 1.27)) (justify left bottom))
@@
     (effects (font (size 1.27 1.27)) (justify left bottom))
   )
+  (hierarchical_label "I2C1_SDA" (shape input) (at 53.34 105.41 0)
+    (effects (font (size 1.27 1.27)) (justify left))
+  )
+  (hierarchical_label "3.3V" (shape input) (at 53.34 78.74 0)
+    (effects (font (size 1.27 1.27)) (justify left))
+  )
   (hierarchical_label "I2S_BCLK" (shape input) (at 53.34 66.04 0)
     (effects (font (size 1.27 1.27)) (justify left))
@@
     (effects (font (size 1.27 1.27)) (justify left))
   )
-  (hierarchical_label "I2C1_SDA" (shape input) (at 53.34 110.49 0)
+  (hierarchical_label "+5V" (shape input) (at 53.34 120.65 0)
     (effects (font (size 1.27 1.27)) (justify left))
   )
@@
     (effects (font (size 1.27 1.27)) (justify left))
   )
-  (hierarchical_label "3.3V" (shape input) (at 53.34 81.28 0)
-    (effects (font (size 1.27 1.27)) (justify left))
-  )
   (hierarchical_label "AVCC_GND" (shape output) (at 353.06 62.23 0)
     (effects (font (size 1.27 1.27)) (justify left))
   )
+  (hierarchical_label "I2C1_SCL" (shape input) (at 53.34 110.49 0)
+    (effects (font (size 1.27 1.27)) (justify left))
+  )
   (hierarchical_label "GND" (shape input) (at 53.34 63.5 0)
     (effects (font (size 1.27 1.27)) (justify left))
   )
+  (hierarchical_label "+5V" (shape input) (at 53.34 118.11 0)
+    (effects (font (size 1.27 1.27)) (justify left))
+  )
   (hierarchical_label "ISO_BCLK" (shape bidirectional) (at 233.68 171.45 0)
     (effects (font (size 1.27 1.27)) (justify left))
   )
+  (hierarchical_label "+5V" (shape input) (at 53.34 81.28 0)
+    (effects (font (size 1.27 1.27)) (justify left))
+  )
   (hierarchical_label "ISO_ADC" (shape input) (at 233.68 201.93 0)
     (effects (font (size 1.27 1.27)) (justify left))
   )
+  (hierarchical_label "3.3V" (shape input) (at 53.34 125.73 0)
+    (effects (font (size 1.27 1.27)) (justify left))
+  )
+  (hierarchical_label "+5V" (shape input) (at 53.34 123.19 0)
+    (effects (font (size 1.27 1.27)) (justify left))
+  )
   (hierarchical_label "VDD_5V" (shape output) (at 209.55 67.31 0)
     (effects (font (size 1.27 1.27)) (justify left))
@@
     (effects (font (size 1.27 1.27)) (justify left))
   )
-  (hierarchical_label "+5V" (shape input) (at 53.34 83.82 0)
-    (effects (font (size 1.27 1.27)) (justify left))
-  )
-  (hierarchical_label "I2C1_SCL" (shape input) (at 53.34 105.41 0)
-    (effects (font (size 1.27 1.27)) (justify left))
-  )
   (hierarchical_label "VDD_GND" (shape output) (at 209.55 62.23 0)
     (effects (font (size 1.27 1.27)) (justify left))
   )
+  (hierarchical_label "+5V" (shape input) (at 53.34 102.87 0)
+    (effects (font (size 1.27 1.27)) (justify left))
+  )

Commit message: .
.
Connections:
- net +5V: now also J8.4 (Pin_4); no longer J9.10 (Pin_10), J9.2 (Pin_2), J9.3 (Pin_3), J9.4 (Pin_4)
- net 3.3V: now also J8.10 (Pin_10); no longer C62.1, J8.4 (Pin_4), J9.1 (Pin_1), R46.1, R47.1, U2.1 (VCC1)
- net GND: no longer C62.2, J8.10 (Pin_10), J9.5 (Pin_5), J9.6 (Pin_6), J9.8 (Pin_8), U2.4 (GND1)
- new net 3.3V_I2C: C62.1, J9.1 (Pin_1), R46.1, R47.1, U2.1 (VCC1)
- new net GND_I2C: C62.2, J9.10 (Pin_10), J9.2 (Pin_2), J9.3 (Pin_3), J9.4 (Pin_4), J9.5 (Pin_5), J9.6 (Pin_6), J9.8 (Pin_8), U2.4 (GND1)
Changed lines of the file:
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@@
     (stroke (width 0) (type default) (color 0 0 0 0))
   )
-  (wire (pts (xy 88.9 128.27) (xy 99.06 128.27))
+  (wire (pts (xy 80.01 128.27) (xy 99.06 128.27))
     (stroke (width 0) (type default) (color 0 0 0 0))
   )
@@
     (stroke (width 0) (type default) (color 0 0 0 0))
   )
-  (wire (pts (xy 88.9 121.92) (xy 99.06 121.92))
+  (wire (pts (xy 80.01 121.92) (xy 99.06 121.92))
     (stroke (width 0) (type default) (color 0 0 0 0))
   )
@@
     (effects (font (size 1.27 1.27)) (justify left bottom))
   )
+  (label "GND_I2C" (at 41.91 107.95 0)
+    (effects (font (size 1.27 1.27)) (justify left bottom))
+  )
   (label "I2C1_SCL" (at 107.95 128.27 0)
     (effects (font (size 1.27 1.27)) (justify left bottom))
@@
     (effects (font (size 1.27 1.27)) (justify left bottom))
   )
-  (label "+5V" (at 41.91 123.19 0)
-    (effects (font (size 1.27 1.27)) (justify left bottom))
-  )
   (label "ISO_BCLK_RX" (at 177.8 157.48 0)
     (effects (font (size 1.27 1.27)) (justify left bottom))
@@
     (effects (font (size 1.27 1.27)) (justify left bottom))
   )
+  (label "GND_I2C" (at 41.91 123.19 0)
+    (effects (font (size 1.27 1.27)) (justify left bottom))
+  )
   (label "ISO_LRCK_TX" (at 199.39 189.23 0)
     (effects (font (size 1.27 1.27)) (justify left bottom))
@@
     (effects (font (size 1.27 1.27)) (justify left bottom))
   )
+  (label "GND_I2C" (at 41.91 120.65 0)
+    (effects (font (size 1.27 1.27)) (justify left bottom))
+  )
+  (label "GND_I2C" (at 41.8567 118.11 0)
+    (effects (font (size 1.27 1.27)) (justify left bottom))
+  )
   (label "+5V" (at 41.91 81.28 0)
     (effects (font (size 1.27 1.27)) (justify left bottom))
@@
     (effects (font (size 1.27 1.27)) (justify left bottom))
   )
+  (label "+5V" (at 41.91 78.74 0)
+    (effects (font (size 1.27 1.27)) (justify left bottom))
+  )
   (label "USB_DEBUG_P" (at 41.91 83.82 0)
     (effects (font (size 1.27 1.27)) (justify left bottom))
@@
     (effects (font (size 1.27 1.27)) (justify left bottom))
   )
-  (label "+5V" (at 41.91 120.65 0)
-    (effects (font (size 1.27 1.27)) (justify left bottom))
-  )
   (label "I2S_ADC" (at 41.91 71.12 0)
     (effects (font (size 1.27 1.27)) (justify left bottom))
   )
+  (label "GND_I2C" (at 41.8567 115.57 0)
+    (effects (font (size 1.27 1.27)) (justify left bottom))
+  )
   (label "I2C1_SDA" (at 41.91 105.41 0)
     (effects (font (size 1.27 1.27)) (justify left bottom))
@@
     (effects (font (size 1.27 1.27)) (justify left bottom))
   )
+  (label "3.3V" (at 41.91 63.5 0)
+    (effects (font (size 1.27 1.27)) (justify left bottom))
+  )
   (label "I2S_LRCK" (at 76.2 182.88 0)
     (effects (font (size 1.27 1.27)) (justify left bottom))
@@
     (effects (font (size 1.27 1.27)) (justify left bottom))
   )
-  (label "3.3V" (at 135.89 116.84 0)
+  (label "3.3V_I2C" (at 83.0384 121.92 0)
     (effects (font (size 1.27 1.27)) (justify left bottom))
   )
@@
     (effects (font (size 1.27 1.27)) (justify left bottom))
   )
-  (label "GND" (at 41.91 113.03 0)
-    (effects (font (size 1.27 1.27)) (justify left bottom))
-  )
-  (label "3.3V" (at 41.91 125.73 0)
+  (label "3.3V_I2C" (at 41.91 125.73 0)
     (effects (font (size 1.27 1.27)) (justify left bottom))
   )
@@
     (effects (font (size 1.27 1.27)) (justify left bottom))
   )
-  (label "3.3V" (at 92.71 121.92 0)
-    (effects (font (size 1.27 1.27)) (justify left bottom))
-  )
-  (label "+5V" (at 41.91 102.87 0)
-    (effects (font (size 1.27 1.27)) (justify left bottom))
-  )
-  (label "GND" (at 134.62 124.46 0)
+  (label "3.3V_I2C" (at 134.6448 116.84 0)
+    (effects (font (size 1.27 1.27)) (justify left bottom))
+  )
+  (label "GND_I2C" (at 41.8567 113.03 0)
     (effects (font (size 1.27 1.27)) (justify left bottom))
   )
@@
     (effects (font (size 1.27 1.27)) (justify left bottom))
   )
-  (label "GND" (at 41.91 115.57 0)
+  (label "GND_I2C" (at 134.62 124.46 0)
     (effects (font (size 1.27 1.27)) (justify left bottom))
   )
@@
     (effects (font (size 1.27 1.27)) (justify left bottom))
   )
+  (label "GND_I2C" (at 41.91 102.87 0)
+    (effects (font (size 1.27 1.27)) (justify left bottom))
+  )
   (label "ISO_LRCK_RX" (at 199.39 182.88 0)
     (effects (font (size 1.27 1.27)) (justify left bottom))
   )
-  (label "+5V" (at 41.91 118.11 0)
-    (effects (font (size 1.27 1.27)) (justify left bottom))
-  )
   (label "ISO_SCL" (at 170.18 121.92 0)
     (effects (font (size 1.27 1.27)) (justify left bottom))
@@
     (effects (font (size 1.27 1.27)) (justify left bottom))
   )
-  (label "GND" (at 41.91 107.95 0)
-    (effects (font (size 1.27 1.27)) (justify left bottom))
-  )
   (label "I2C1_SDA" (at 107.95 121.92 0)
     (effects (font (size 1.27 1.27)) (justify left bottom))
@@
     (effects (font (size 1.27 1.27)) (justify left bottom))
   )
+  (label "GND_I2C" (at 115.05 116.84 0)
+    (effects (font (size 1.27 1.27)) (justify left bottom))
+  )
   (label "GND" (at 128.27 72.39 0)
     (effects (font (size 1.27 1.27)) (justify left bottom))
@@
     (effects (font (size 1.27 1.27)) (justify left bottom))
   )
-  (label "GND" (at 41.91 63.5 0)
+  (label "3.3V_I2C" (at 82.55 128.27 0)
     (effects (font (size 1.27 1.27)) (justify left bottom))
   )
@@
     (effects (font (size 1.27 1.27)) (justify left bottom))
   )
-  (label "3.3V" (at 92.71 128.27 0)
-    (effects (font (size 1.27 1.27)) (justify left bottom))
-  )
-  (label "3.3V" (at 41.91 78.74 0)
-    (effects (font (size 1.27 1.27)) (justify left bottom))
-  )
   (label "VDD_GND" (at 199.39 62.23 0)
     (effects (font (size 1.27 1.27)) (justify left bottom))
   )
-  (label "GND" (at 116.84 116.84 0)
-    (effects (font (size 1.27 1.27)) (justify left bottom))
-  )
   (label "I2S_BCLK" (at 76.2 165.1 0)
     (effects (font (size 1.27 1.27)) (justify left bottom))
@@
     (effects (font (size 1.27 1.27)) (justify left))
   )
-  (hierarchical_label "3.3V" (shape input) (at 53.34 78.74 0)
-    (effects (font (size 1.27 1.27)) (justify left))
-  )
   (hierarchical_label "I2S_BCLK" (shape input) (at 53.34 66.04 0)
     (effects (font (size 1.27 1.27)) (justify left))
@@
     (effects (font (size 1.27 1.27)) (justify left))
   )
-  (hierarchical_label "+5V" (shape input) (at 53.34 120.65 0)
-    (effects (font (size 1.27 1.27)) (justify left))
-  )
   (hierarchical_label "ISO_SCL" (shape bidirectional) (at 181.61 121.92 0)
     (effects (font (size 1.27 1.27)) (justify left))
@@
     (effects (font (size 1.27 1.27)) (justify left))
   )
+  (hierarchical_label "GND_I2C" (shape input) (at 53.34 102.87 0)
+    (effects (font (size 1.27 1.27)) (justify left))
+  )
   (hierarchical_label "AVCC_GND" (shape output) (at 353.06 62.23 0)
     (effects (font (size 1.27 1.27)) (justify left))
@@
     (effects (font (size 1.27 1.27)) (justify left))
   )
-  (hierarchical_label "GND" (shape input) (at 53.34 63.5 0)
-    (effects (font (size 1.27 1.27)) (justify left))
-  )
-  (hierarchical_label "+5V" (shape input) (at 53.34 118.11 0)
-    (effects (font (size 1.27 1.27)) (justify left))
-  )
   (hierarchical_label "ISO_BCLK" (shape bidirectional) (at 233.68 171.45 0)
     (effects (font (size 1.27 1.27)) (justify left))
@@
     (effects (font (size 1.27 1.27)) (justify left))
   )
+  (hierarchical_label "3.3V_I2C" (shape input) (at 53.34 125.73 0)
+    (effects (font (size 1.27 1.27)) (justify left))
+  )
   (hierarchical_label "ISO_ADC" (shape input) (at 233.68 201.93 0)
     (effects (font (size 1.27 1.27)) (justify left))
   )
-  (hierarchical_label "3.3V" (shape input) (at 53.34 125.73 0)
-    (effects (font (size 1.27 1.27)) (justify left))
-  )
-  (hierarchical_label "+5V" (shape input) (at 53.34 123.19 0)
+  (hierarchical_label "3.3V" (shape input) (at 53.34 63.5 0)
+    (effects (font (size 1.27 1.27)) (justify left))
+  )
+  (hierarchical_label "+5V" (shape input) (at 53.34 78.74 0)
     (effects (font (size 1.27 1.27)) (justify left))
   )
@@
     (effects (font (size 1.27 1.27)) (justify left))
   )
-  (hierarchical_label "+5V" (shape input) (at 53.34 102.87 0)
-    (effects (font (size 1.27 1.27)) (justify left))
-  )
