File: audio/isolation_module.kicad_sch (KiCad schematic)
At the start: 32 parts, among them J8 Conn_01x10, J9 Conn_01x10, U2 ISO1540, U9 SI8663BB-B-IS1

Commit message: .
.
Parts:
- added R35: 15K 1%, Resistor_SMD:R_0402_1005Metric, symbol Device:R
Connections:
- net +5V: now also R35.1
- net 3.3V_I2C: now also J9.10 (Pin_10); no longer J9.1 (Pin_1)
- net GND: no longer J8.8 (Pin_8)
- net GND_I2C: now also J9.1 (Pin_1); no longer J9.10 (Pin_10)
- new net nRPIBOOT: J8.8 (Pin_8), R35.2

Commit message: .
.
Parts:
- added C75, C76, C77, C78: 1uF, Capacitor_SMD:C_0402_1005Metric, symbol Device:C_Small
- added U13, U14: TCR3RM33, CM4IO:TCR3RM33, symbol CM4IO:TCR3RM33
Connections:
- net +5V: now also C75.1, U13.3 (CONTROL), U13.4 (VIN); no longer J8.4 (Pin_4)
- net 3.3V: now also C76.1, U13.1 (VOUT); no longer J8.10 (Pin_10)
- net 3.3V_I2C: now also C78.1, U14.1 (VOUT); no longer J9.10 (Pin_10)
- net GND: now also J8.10 (Pin_10), J8.4 (Pin_4), C75.2, C76.2, U13.2 (GND_1), U13.5 (GND_2); no longer J8.6 (Pin_6)
- net GND_I2C: now also J9.10 (Pin_10), C77.2, C78.2, U14.2 (GND_1), U14.5 (GND_2); no longer J9.1 (Pin_1), J9.2 (Pin_2), J9.3 (Pin_3), J9.4 (Pin_4)
- new net +5V_I2C: C77.1, J9.1 (Pin_1), J9.2 (Pin_2), J9.3 (Pin_3), J9.4 (Pin_4), U14.3 (CONTROL), U14.4 (VIN)
- new net GLOBAL_EN: J8.6 (Pin_6)

Commit message: .
.
Parts:
- R42, R44, R50, R52: value 0 -> NC
Changed lines of the file:
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@@
     (in_bom yes) (on_board yes)
     (property "Reference" "R44" (id 0) (at 91.44 180.34 90))
-    (property "Value" "0" (id 1) (at 95.25 180.34 90))
+    (property "Value" "NC" (id 1) (at 95.25 180.34 90))
     (property "Footprint" "Resistor_SMD:R_0603_1608Metric" (id 2) (at 92.71 182.88 0)
       (effects (font (size 1.27 1.27)) hide)
@@
     (in_bom yes) (on_board yes)
     (property "Reference" "R42" (id 0) (at 91.44 162.56 90))
-    (property "Value" "0" (id 1) (at 95.25 162.56 90))
+    (property "Value" "NC" (id 1) (at 95.25 162.56 90))
     (property "Footprint" "Resistor_SMD:R_0603_1608Metric" (id 2) (at 92.71 165.1 0)
       (effects (font (size 1.27 1.27)) hide)
@@
     (in_bom yes) (on_board yes)
     (property "Reference" "R50" (id 0) (at 215.9 167.64 90))
-    (property "Value" "0" (id 1) (at 212.09 167.64 90))
+    (property "Value" "NC" (id 1) (at 212.09 167.64 90))
     (property "Footprint" "Resistor_SMD:R_0603_1608Metric" (id 2) (at 214.63 165.1 0)
       (effects (font (size 1.27 1.27)) hide)
@@
     (in_bom yes) (on_board yes)
     (property "Reference" "R52" (id 0) (at 215.9 185.42 90))
-    (property "Value" "0" (id 1) (at 212.09 185.42 90))
+    (property "Value" "NC" (id 1) (at 212.09 185.42 90))
     (property "Footprint" "Resistor_SMD:R_0603_1608Metric" (id 2) (at 214.63 182.88 0)
       (effects (font (size 1.27 1.27)) hide)
