File: audio/isolation_module.kicad_sch (KiCad schematic)
At the start: 39 parts, among them J8 Conn_01x10, J9 Conn_01x10, U13 TCR3RM33, U14 TCR3RM33, U2 ISO1540, U9 SI8663BB-B-IS1

Commit message: .
.
Parts:
- removed R42, R44, R50, R52: NC, Resistor_SMD:R_0603_1608Metric, symbol Device:R_Small_US
Changed lines of the file:
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@@
   (junction (at 269.24 62.23) (diameter 0) (color 0 0 0 0)
   )
-  (junction (at 220.98 189.23) (diameter 0) (color 0 0 0 0)
-  )
   (junction (at 176.53 74.93) (diameter 0) (color 0 0 0 0)
   )
@@
   (junction (at 198.12 152.4) (diameter 0) (color 0 0 0 0)
   )
-  (junction (at 86.36 165.1) (diameter 0) (color 0 0 0 0)
-  )
   (junction (at 135.89 72.39) (diameter 0) (color 0 0 0 0)
   )
-  (junction (at 220.98 171.45) (diameter 0) (color 0 0 0 0)
-  )
   (junction (at 279.4 62.23) (diameter 0) (color 0 0 0 0)
   )
@@
   (junction (at 97.79 152.4) (diameter 0) (color 0 0 0 0)
   )
-  (junction (at 86.36 182.88) (diameter 0) (color 0 0 0 0)
-  )
   (junction (at 195.58 67.31) (diameter 0) (color 0 0 0 0)
   )
@@
     (stroke (width 0) (type default))
   )
-  (wire (pts (xy 217.17 182.88) (xy 220.98 182.88))
-    (stroke (width 0) (type default))
-  )
-  (wire (pts (xy 95.25 182.88) (xy 110.49 182.88))
-    (stroke (width 0) (type default))
-  )
   (wire (pts (xy 328.93 67.31) (xy 339.09 67.31))
     (stroke (width 0) (type default))
@@
     (stroke (width 0) (type default))
   )
-  (wire (pts (xy 86.36 182.88) (xy 90.17 182.88))
-    (stroke (width 0) (type default))
-  )
   (wire (pts (xy 199.39 120.65) (xy 209.55 120.65))
     (stroke (width 0) (type default))
@@
     (stroke (width 0) (type default))
   )
-  (wire (pts (xy 86.36 165.1) (xy 90.17 165.1))
-    (stroke (width 0) (type default))
-  )
   (wire (pts (xy 120.65 160.02) (xy 135.89 160.02))
     (stroke (width 0) (type default))
@@
     (stroke (width 0) (type default))
   )
-  (wire (pts (xy 212.09 165.1) (xy 196.85 165.1))
-    (stroke (width 0) (type default))
-  )
   (wire (pts (xy 176.53 62.23) (xy 185.42 62.23))
     (stroke (width 0) (type default))
@@
     (stroke (width 0) (type default))
   )
-  (wire (pts (xy 95.25 165.1) (xy 110.49 165.1))
-    (stroke (width 0) (type default))
-  )
   (wire (pts (xy 195.58 67.31) (xy 209.55 67.31))
     (stroke (width 0) (type default))
@@
     (stroke (width 0) (type default))
   )
-  (wire (pts (xy 217.17 165.1) (xy 220.98 165.1))
-    (stroke (width 0) (type default))
-  )
   (wire (pts (xy 38.1 107.95) (xy 53.34 107.95))
     (stroke (width 0) (type default))
@@
     (stroke (width 0) (type default))
   )
-  (wire (pts (xy 220.98 182.88) (xy 220.98 189.23))
-    (stroke (width 0) (type default))
-  )
   (wire (pts (xy 185.42 62.23) (xy 195.58 62.23))
     (stroke (width 0) (type default))
@@
     (stroke (width 0) (type default))
   )
-  (wire (pts (xy 233.68 171.45) (xy 220.98 171.45))
+  (wire (pts (xy 217.17 171.45) (xy 233.68 171.45))
     (stroke (width 0) (type default))
   )
@@
     (stroke (width 0) (type default))
   )
-  (wire (pts (xy 212.09 182.88) (xy 196.85 182.88))
-    (stroke (width 0) (type default))
-  )
   (wire (pts (xy 260.35 62.23) (xy 269.24 62.23))
     (stroke (width 0) (type default))
@@
     (stroke (width 0) (type default))
   )
-  (wire (pts (xy 233.68 189.23) (xy 220.98 189.23))
+  (wire (pts (xy 217.17 189.23) (xy 233.68 189.23))
     (stroke (width 0) (type default))
   )
@@
     (stroke (width 0) (type default))
   )
-  (wire (pts (xy 220.98 165.1) (xy 220.98 171.45))
-    (stroke (width 0) (type default))
-  )
   (wire (pts (xy 252.73 62.23) (xy 260.35 62.23))
     (stroke (width 0) (type default))
@@
     (stroke (width 0) (type default))
   )
-  (wire (pts (xy 220.98 171.45) (xy 217.17 171.45))
-    (stroke (width 0) (type default))
-  )
-  (wire (pts (xy 220.98 189.23) (xy 217.17 189.23))
-    (stroke (width 0) (type default))
-  )
   (wire (pts (xy 320.04 72.39) (xy 320.04 74.93))
     (stroke (width 0) (type default))
@@
     (effects (font (size 1.27 1.27)) (justify left bottom))
   )
-  (label "ISO_BCLK_RX" (at 199.1827 165.1 0) (fields_autoplaced)
-    (effects (font (size 1.27 1.27)) (justify left bottom))
-  )
   (label "3.3V_I2C" (at 83.0384 121.92 0) (fields_autoplaced)
     (effects (font (size 1.27 1.27)) (justify left bottom))
@@
     (effects (font (size 1.27 1.27)) (justify left bottom))
   )
-  (label "I2S_LRCK_TX" (at 96.52 182.88 0) (fields_autoplaced)
-    (effects (font (size 1.27 1.27)) (justify left bottom))
-  )
   (label "VDD_3.3V" (at 200.6146 127 0) (fields_autoplaced)
     (effects (font (size 1.27 1.27)) (justify left bottom))
@@
     (effects (font (size 1.27 1.27)) (justify left bottom))
   )
-  (label "ISO_LRCK_RX" (at 199.39 182.88 0) (fields_autoplaced)
-    (effects (font (size 1.27 1.27)) (justify left bottom))
-  )
   (label "ISO_SCL" (at 170.18 121.92 0) (fields_autoplaced)
     (effects (font (size 1.27 1.27)) (justify left bottom))
@@
   )
   (label "I2S_ADC" (at 127 167.64 0) (fields_autoplaced)
-    (effects (font (size 1.27 1.27)) (justify left bottom))
-  )
-  (label "I2S_BCLK_TX" (at 96.52 165.1 0) (fields_autoplaced)
     (effects (font (size 1.27 1.27)) (justify left bottom))
   )
@@
     )
   )
-  (symbol (lib_id "Device:R_Small_US") (at 92.71 182.88 90) (unit 1)
-    (in_bom yes) (on_board yes) (dnp no)
-    (property "Reference" "R44" (at 91.44 180.34 90)
-      (effects (font (size 1.27 1.27)))
-    )
-    (property "Value" "NC" (at 95.25 180.34 90)
-      (effects (font (size 1.27 1.27)))
-    )
-    (property "Footprint" "Resistor_SMD:R_0603_1608Metric" (at 92.71 182.88 0)
-      (effects (font (size 1.27 1.27)) hide)
-    )
-    (property "Datasheet" "~" (at 92.71 182.88 0)
-      (effects (font (size 1.27 1.27)) hide)
-    )
-    (pin "1")
-    (pin "2")
-    (instances
-      (project "audio"
-        (path "/2e4f7337-6386-43b5-93e9-f72e36e0825c/039620fc-845c-4f42-b371-a9cdeb447748"
-          (reference "R44") (unit 1)
-        )
-      )
-    )
-  )
   (symbol (lib_id "Device:C_Small") (at 328.93 64.77 180) (unit 1)
     (in_bom yes) (on_board yes) (dnp no)
@@
         (path "/2e4f7337-6386-43b5-93e9-f72e36e0825c/039620fc-845c-4f42-b371-a9cdeb447748"
           (reference "C59") (unit 1)
-        )
-      )
-    )
-  )
-  (symbol (lib_id "Device:R_Small_US") (at 92.71 165.1 90) (unit 1)
-    (in_bom yes) (on_board yes) (dnp no)
-    (property "Reference" "R42" (at 91.44 162.56 90)
-      (effects (font (size 1.27 1.27)))
-    )
-    (property "Value" "NC" (at 95.25 162.56 90)
-      (effects (font (size 1.27 1.27)))
-    )
-    (property "Footprint" "Resistor_SMD:R_0603_1608Metric" (at 92.71 165.1 0)
-      (effects (font (size 1.27 1.27)) hide)
-    )
-    (property "Datasheet" "~" (at 92.71 165.1 0)
-      (effects (font (size 1.27 1.27)) hide)
-    )
-    (pin "1")
-    (pin "2")
-    (instances
-      (project "audio"
-        (path "/2e4f7337-6386-43b5-93e9-f72e36e0825c/039620fc-845c-4f42-b371-a9cdeb447748"
-          (reference "R42") (unit 1)
         )
       )
@@
     )
   )
-  (symbol (lib_id "Device:R_Small_US") (at 214.63 165.1 270) (unit 1)
-    (in_bom yes) (on_board yes) (dnp no)
-    (property "Reference" "R50" (at 215.9 167.64 90)
-      (effects (font (size 1.27 1.27)))
-    )
-    (property "Value" "NC" (at 212.09 167.64 90)
-      (effects (font (size 1.27 1.27)))
-    )
-    (property "Footprint" "Resistor_SMD:R_0603_1608Metric" (at 214.63 165.1 0)
-      (effects (font (size 1.27 1.27)) hide)
-    )
-    (property "Datasheet" "~" (at 214.63 165.1 0)
-      (effects (font (size 1.27 1.27)) hide)
-    )
-    (pin "1")
-    (pin "2")
-    (instances
-      (project "audio"
-        (path "/2e4f7337-6386-43b5-93e9-f72e36e0825c/039620fc-845c-4f42-b371-a9cdeb447748"
-          (reference "R50") (unit 1)
-        )
-      )
-    )
-  )
   (symbol (lib_id "Device:C_Small") (at 260.35 64.77 180) (unit 1)
     (in_bom yes) (on_board yes) (dnp no)
@@
         )
       )
-    )
-  )
-  (symbol (lib_id "Device:R_Small_US") (at 214.63 182.88 270) (unit 1)
-    (in_bom yes) (on_board yes) (dnp no)
-    (property "Reference" "R52" (at 215.9 185.42 90)
-      (effects (font (size 1.27 1.27)))
-    )
-    (property "Value" "NC" (at 212.09 185.42 90)
-      (effects (font (size 1.27 1.27)))
-    )
-    (property "Footprint" "Resistor_SMD:R_0603_1608Metric" (at 214.63 182.88 0)
-      (effects (font (size 1.27 1.27)) hide)
-    )
-    (property "Datasheet" "~" (at 214.63 182.88 0)
-      (effects (font (size 1.27 1.27)) hide)
-    )
-    (pin "1")
-    (pin "2")
-    (instances
-      (project "audio"
-        (path "/2e4f7337-6386-43b5-93e9-f72e36e0825c/039620fc-845c-4f42-b371-a9cdeb447748"
-          (reference "R52") (unit 1)
-        )
-      )
