File: audio/4ch_mic.kicad_sch (KiCad schematic)
At the start: 0 parts

Commit message: .
.
Parts:
- added C? (x16): 1uF, Capacitor_SMD:C_0402_1005Metric, symbol Device:C_Small
- added C?: 10uF, Capacitor_SMD:C_0402_1005Metric, symbol Device:C_Small
- added R? (x11): 0, Capacitor_SMD:C_0603_1608Metric, symbol Device:R_Small_US
- added R? (x4): 10, Capacitor_SMD:C_0603_1608Metric, symbol Device:R_Small_US
- added R? (x2): 10k, Capacitor_SMD:C_0603_1608Metric, symbol Device:R_Small_US
- added R? (x3): 0, symbol Device:R_Small_US
- added U10: ac108, CM4IO:AC108, symbol CM4IO:ac108
- added U11, U?: TCR3RM33, CM4IO:TCR3RM33, symbol CM4IO:TCR3RM33
Connections:
- new net: R?.1, R?.2, R?.2
- new net: R?.1, R?.1, R?.1, R?.1, R?.2, R?.2
- new net ALDOIN: C?.1, R?.2, U10.27 (ALDOIN)
- new net ALDOOUT: C?.1, R?.1, R?.2, U10.28 (ALDOOUT)
- new net AVCC_3.3V: C?.1, R?.1, R?.2, U11.1 (VOUT)
- new net AVCC_5V: C?.1, R?.1, R?.1, R?.2, U11.3 (CONTROL), U11.4 (VIN)
- new net AVCC_ANA1: C?.1, R?.2, U10.20 (AVCC_ANA1)
- new net AVCC_ANA2: C?.1, R?.2, U10.40 (AVCC_ANA2)
- new net AVCC_GND: C?.2, C?.2, C?.2, C?.2, C?.2, C?.2, C?.2, C?.2, C?.2, R?.2, U10.33 (AGND), U11.2 (GND_1), U11.5 (GND_2)
- new net BCLK: R?.2, U10.15 (BCLK)
- new net CP_EN: R?.2, U10.44 (CP_EN)
- new net CP_VPN: C?.2, U10.42 (CP_VPN)
- new net CP_VPP: C?.1, U10.43 (CP_VPP)
- new net DEV_ID0: U10.4 (DEV_ID0)
- new net DLDOIN: C?.1, R?.2, U10.45 (DLDOIN)
- new net DLDOOUT: C?.1, U10.46 (DLDOOUT)
- new net GND: U10.32 (VRN)
- new net ISO_BCLK: R?.1
- new net ISO_LRCK: R?.1
- new net ISO_MCLK: R?.1
- new net ISO_SDOUT: R?.1
- new net LRCK: R?.2, U10.18 (LRCK)
- new net MCLK: R?.2, U10.8 (MCLK)
- new net RSTn: R?.2, U10.19 (RSTn)
- new net RVCC: C?.1, R?.2, U10.29 (RVCC)
- new net SCK: U10.9 (SCK)
- new net SDA: U10.10 (SDA)
- new net SDOUT1: R?.2, U10.16 (SDOUT1)
- new net TEST: U10.5 (TEST)
- new net VCC_DIO: C?.1, C?.1, R?.2, U10.11 (VCC_I2S), U10.7 (VCC_DIO)
- new net VDD_3.3V: C?.1, R?.1, R?.1, R?.1, U?.1 (VOUT)
- new net VDD_5V: C?.1, R?.1, R?.1, R?.1, U?.3 (CONTROL), U?.4 (VIN)
- new net VDD_CORE: C?.1, U10.41 (VDD_CPOUT), U10.6 (VDD_CORE)
- new net VDD_GND: C?.2, C?.2, C?.2, C?.2, C?.2, C?.2, C?.2, R?.1, U10.PAD (GND), U?.2 (GND_1), U?.5 (GND_2)
- new net VREF: C?.1, U10.30 (VREF)
- new net VRP: C?.1, U10.31 (VRP)
Other:
- note added: "ANALOG POWER"
- note added: "DIGITAL_INTERFACE"
- note added: "DIGITAL_POWER"
- note added: "POWER_INPUT"

Commit message: .
.
Parts:
- added J11: MIC1, CM4IO:GROVE_4PIN, symbol CM4IO:GROVE_4PIN
- added J12: MIC2, CM4IO:GROVE_4PIN, symbol CM4IO:GROVE_4PIN
- added J13: MIC3, CM4IO:GROVE_4PIN, symbol CM4IO:GROVE_4PIN
- added J14: MIC4, CM4IO:GROVE_4PIN, symbol CM4IO:GROVE_4PIN
- gave numbers to parts that had none: 38
Connections:
- net AVCC_3.3V: now also J11.2, J12.2, J13.2, J14.2
- net AVCC_GND: now also J11.1, J11.MP1, J11.MP2, J12.1, J12.MP1, J12.MP2, J13.1, J13.MP1, J13.MP2, J14.1, J14.MP1, J14.MP2
- net MIC1P: now reaches U10.22 (MIC1P)
- net MIC1P: now also J11.4
- net MIC1N: now reaches U10.23 (MIC1N)
- net MIC1N: now also J11.3
- net MIC2P: now reaches U10.25 (MIC2P)
- net MIC2P: now also J12.4
- net MIC2N: now reaches U10.26 (MIC2N)
- net MIC2N: now also J12.3
- net MIC3P: now reaches U10.35 (MIC3P)
- net MIC3P: now also J13.4
- net MIC3N: now reaches U10.36 (MIC3N)
- net MIC3N: now also J13.3
- net MIC4P: now reaches U10.38 (MIC4P)
- net MIC4P: now also J14.4
- net MIC4N: now reaches U10.39 (MIC4N)
- net MIC4N: now also J14.3
Other:
- note added: "EXTERNEL MIC"

Commit message: .
.
Parts:
- R17, R23, R24, R25, R26, R27, R28, R29, R30, R31, R35, R36, R37, R38, R39, R40, R41: footprint Capacitor_SMD:C_0603_1608Metric -> Resistor_SMD:R_0603_1608Metric
- R32, R33, R34: footprint (none) -> Resistor_SMD:R_0603_1608Metric
Changed lines of the file:
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@@
     (property "Reference" "R37" (id 0) (at 289.56 71.12 90))
     (property "Value" "0" (id 1) (at 293.37 71.12 90))
-    (property "Footprint" "Capacitor_SMD:C_0603_1608Metric" (id 2) (at 290.83 73.66 0)
+    (property "Footprint" "Resistor_SMD:R_0603_1608Metric" (id 2) (at 290.83 73.66 0)
       (effects (font (size 1.27 1.27)) hide)
     )
@@
     (property "Reference" "R27" (id 0) (at 63.5 187.96 90))
     (property "Value" "10" (id 1) (at 67.31 187.96 90))
-    (property "Footprint" "Capacitor_SMD:C_0603_1608Metric" (id 2) (at 64.77 190.5 0)
+    (property "Footprint" "Resistor_SMD:R_0603_1608Metric" (id 2) (at 64.77 190.5 0)
       (effects (font (size 1.27 1.27)) hide)
     )
@@
     (property "Reference" "R17" (id 0) (at 48.26 116.84 90))
     (property "Value" "0" (id 1) (at 52.07 116.84 90))
-    (property "Footprint" "Capacitor_SMD:C_0603_1608Metric" (id 2) (at 49.53 119.38 0)
+    (property "Footprint" "Resistor_SMD:R_0603_1608Metric" (id 2) (at 49.53 119.38 0)
       (effects (font (size 1.27 1.27)) hide)
     )
@@
     (property "Reference" "R24" (id 0) (at 49.53 78.74 90))
     (property "Value" "0" (id 1) (at 53.34 78.74 90))
-    (property "Footprint" "Capacitor_SMD:C_0603_1608Metric" (id 2) (at 50.8 81.28 0)
+    (property "Footprint" "Resistor_SMD:R_0603_1608Metric" (id 2) (at 50.8 81.28 0)
       (effects (font (size 1.27 1.27)) hide)
     )
@@
     (property "Reference" "R26" (id 0) (at 63.5 180.34 90))
     (property "Value" "10k" (id 1) (at 67.31 180.34 90))
-    (property "Footprint" "Capacitor_SMD:C_0603_1608Metric" (id 2) (at 64.77 182.88 0)
+    (property "Footprint" "Resistor_SMD:R_0603_1608Metric" (id 2) (at 64.77 182.88 0)
       (effects (font (size 1.27 1.27)) hide)
     )
@@
     (property "Reference" "R38" (id 0) (at 292.1 78.74 90))
     (property "Value" "0" (id 1) (at 295.91 78.74 90))
-    (property "Footprint" "Capacitor_SMD:C_0603_1608Metric" (id 2) (at 293.37 81.28 0)
+    (property "Footprint" "Resistor_SMD:R_0603_1608Metric" (id 2) (at 293.37 81.28 0)
       (effects (font (size 1.27 1.27)) hide)
     )
@@
     (property "Reference" "R39" (id 0) (at 292.1 83.82 90))
     (property "Value" "0" (id 1) (at 295.91 83.82 90))
-    (property "Footprint" "Capacitor_SMD:C_0603_1608Metric" (id 2) (at 293.37 86.36 0)
+    (property "Footprint" "Resistor_SMD:R_0603_1608Metric" (id 2) (at 293.37 86.36 0)
       (effects (font (size 1.27 1.27)) hide)
     )
@@
     (property "Reference" "R35" (id 0) (at 265.43 78.74 90))
     (property "Value" "0" (id 1) (at 269.24 78.74 90))
-    (property "Footprint" "Capacitor_SMD:C_0603_1608Metric" (id 2) (at 266.7 81.28 0)
+    (property "Footprint" "Resistor_SMD:R_0603_1608Metric" (id 2) (at 266.7 81.28 0)
       (effects (font (size 1.27 1.27)) hide)
     )
@@
     (property "Reference" "R25" (id 0) (at 49.53 86.36 90))
     (property "Value" "0" (id 1) (at 53.34 86.36 90))
-    (property "Footprint" "Capacitor_SMD:C_0603_1608Metric" (id 2) (at 50.8 88.9 0)
+    (property "Footprint" "Resistor_SMD:R_0603_1608Metric" (id 2) (at 50.8 88.9 0)
       (effects (font (size 1.27 1.27)) hide)
     )
@@
     (property "Reference" "R29" (id 0) (at 63.5 203.2 90))
     (property "Value" "10" (id 1) (at 67.31 203.2 90))
-    (property "Footprint" "Capacitor_SMD:C_0603_1608Metric" (id 2) (at 64.77 205.74 0)
+    (property "Footprint" "Resistor_SMD:R_0603_1608Metric" (id 2) (at 64.77 205.74 0)
       (effects (font (size 1.27 1.27)) hide)
     )
@@
     (property "Reference" "R36" (id 0) (at 265.43 85.09 90))
     (property "Value" "0" (id 1) (at 269.24 85.09 90))
-    (property "Footprint" "Capacitor_SMD:C_0603_1608Metric" (id 2) (at 266.7 87.63 0)
+    (property "Footprint" "Resistor_SMD:R_0603_1608Metric" (id 2) (at 266.7 87.63 0)
       (effects (font (size 1.27 1.27)) hide)
     )
@@
     (property "Reference" "R23" (id 0) (at 49.53 59.69 90))
     (property "Value" "0" (id 1) (at 53.34 59.69 90))
-    (property "Footprint" "Capacitor_SMD:C_0603_1608Metric" (id 2) (at 50.8 62.23 0)
+    (property "Footprint" "Resistor_SMD:R_0603_1608Metric" (id 2) (at 50.8 62.23 0)
       (effects (font (size 1.27 1.27)) hide)
     )
@@
     (property "Reference" "R40" (id 0) (at 292.1 88.9 90))
     (property "Value" "0" (id 1) (at 295.91 88.9 90))
-    (property "Footprint" "Capacitor_SMD:C_0603_1608Metric" (id 2) (at 293.37 91.44 0)
+    (property "Footprint" "Resistor_SMD:R_0603_1608Metric" (id 2) (at 293.37 91.44 0)
       (effects (font (size 1.27 1.27)) hide)
     )
@@
     (property "Reference" "R32" (id 0) (at 170.18 39.37 90))
     (property "Value" "0" (id 1) (at 173.99 39.37 90))
-    (property "Footprint" "" (id 2) (at 171.45 41.91 0)
+    (property "Footprint" "Resistor_SMD:R_0603_1608Metric" (id 2) (at 171.45 41.91 0)
       (effects (font (size 1.27 1.27)) hide)
     )
@@
     (property "Reference" "R33" (id 0) (at 170.18 46.99 90))
     (property "Value" "0" (id 1) (at 173.99 46.99 90))
-    (property "Footprint" "" (id 2) (at 171.45 49.53 0)
+    (property "Footprint" "Resistor_SMD:R_0603_1608Metric" (id 2) (at 171.45 49.53 0)
       (effects (font (size 1.27 1.27)) hide)
     )
@@
     (property "Reference" "R41" (id 0) (at 292.1 93.98 90))
     (property "Value" "0" (id 1) (at 295.91 93.98 90))
-    (property "Footprint" "Capacitor_SMD:C_0603_1608Metric" (id 2) (at 293.37 96.52 0)
+    (property "Footprint" "Resistor_SMD:R_0603_1608Metric" (id 2) (at 293.37 96.52 0)
       (effects (font (size 1.27 1.27)) hide)
     )
@@
     (property "Reference" "R28" (id 0) (at 63.5 195.58 90))
     (property "Value" "10" (id 1) (at 67.31 195.58 90))
-    (property "Footprint" "Capacitor_SMD:C_0603_1608Metric" (id 2) (at 64.77 198.12 0)
+    (property "Footprint" "Resistor_SMD:R_0603_1608Metric" (id 2) (at 64.77 198.12 0)
       (effects (font (size 1.27 1.27)) hide)
     )
@@
     (property "Reference" "R34" (id 0) (at 170.18 54.61 90))
     (property "Value" "0" (id 1) (at 173.99 54.61 90))
-    (property "Footprint" "" (id 2) (at 171.45 57.15 0)
+    (property "Footprint" "Resistor_SMD:R_0603_1608Metric" (id 2) (at 171.45 57.15 0)
       (effects (font (size 1.27 1.27)) hide)
     )
@@
     (property "Reference" "R31" (id 0) (at 78.74 78.74 90))
     (property "Value" "10k" (id 1) (at 82.55 78.74 90))
-    (property "Footprint" "Capacitor_SMD:C_0603_1608Metric" (id 2) (at 80.01 81.28 0)
+    (property "Footprint" "Resistor_SMD:R_0603_1608Metric" (id 2) (at 80.01 81.28 0)
       (effects (font (size 1.27 1.27)) hide)
     )
@@
     (property "Reference" "R30" (id 0) (at 63.5 210.82 90))
     (property "Value" "10" (id 1) (at 67.31 210.82 90))
-    (property "Footprint" "Capacitor_SMD:C_0603_1608Metric" (id 2) (at 64.77 213.36 0)
-      (effects (font (size 1.27 1.27)) hide)
-    )
+    (property "Footprint" "Resistor_SMD:R_0603_1608Metric" (id 2) (at 64.77 213.36 0)
+      (effects (font (size 1.27 1.27)) hide)
+    )

Commit message: .
.
Connections:
- net SCK renamed ISO_SCK
- net SDA renamed ISO_SDA
Changed lines of the file:
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@@
     (effects (font (size 1.27 1.27)) (justify left bottom))
   )
-  (label "SDA" (at 128.27 129.54 0)
+  (label "ISO_SDA" (at 128.27 129.54 0)
     (effects (font (size 1.27 1.27)) (justify left bottom))
   )
@@
     (effects (font (size 1.27 1.27)) (justify left bottom))
   )
-  (label "SCK" (at 128.27 132.08 0)
+  (label "ISO_SCK" (at 128.27 132.08 0)
     (effects (font (size 1.27 1.27)) (justify left bottom))
   )
@@
   (label "VDD_CPOUT" (at 60.96 105.41 0)
     (effects (font (size 1.27 1.27)) (justify left bottom))
+  )
+  (hierarchical_label "VDD_3.3V" (shape output) (at 147.32 49.53 180)
+    (effects (font (size 1.27 1.27)) (justify right))
   )
   (hierarchical_label "AVCC_GND" (shape input) (at 191.77 57.15 0)
     (effects (font (size 1.27 1.27)) (justify left))
   )
+  (hierarchical_label "ISO_SDA" (shape input) (at 125.73 129.54 180)
+    (effects (font (size 1.27 1.27)) (justify right))
+  )
   (hierarchical_label "VDD_GND" (shape input) (at 147.32 57.15 180)
     (effects (font (size 1.27 1.27)) (justify right))
@@
     (effects (font (size 1.27 1.27)) (justify left))
   )
+  (hierarchical_label "ISO_SCK" (shape input) (at 125.73 132.08 180)
+    (effects (font (size 1.27 1.27)) (justify right))
+  )
   (hierarchical_label "VDD_5V" (shape input) (at 147.32 41.91 180)

Commit message: .
.
Connections:
- net ISO_SDOUT renamed ISO_ADC
Changed lines of the file:
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@@
     (effects (font (size 1.27 1.27)) (justify left bottom))
   )
-  (label "ISO_SDOUT" (at 49.53 213.36 0)
+  (label "ISO_ADC" (at 49.53 213.36 0)
     (effects (font (size 1.27 1.27)) (justify left bottom))
   )
@@
     (effects (font (size 1.27 1.27)) (justify right))
   )
+  (hierarchical_label "ISO_ADC" (shape output) (at 46.99 213.36 180)
+    (effects (font (size 1.27 1.27)) (justify right))
+  )
+  (hierarchical_label "ISO_BCLK" (shape bidirectional) (at 46.99 198.12 180)
+    (effects (font (size 1.27 1.27)) (justify right))
+  )
   (hierarchical_label "VDD_GND" (shape input) (at 147.32 57.15 180)
     (effects (font (size 1.27 1.27)) (justify right))
@@
     (effects (font (size 1.27 1.27)) (justify right))
   )
+  (hierarchical_label "ISO_LRCK" (shape bidirectional) (at 46.99 205.74 180)
+    (effects (font (size 1.27 1.27)) (justify right))
+  )

Commit message: .
.
Parts:
- added C?: 0.1uF, Capacitor_SMD:C_0402_1005Metric, symbol Device:C_Small
- added X1: ASE-24.000MHz, Oscillator:Oscillator_SMD_Abracon_ASE-4Pin_3.2x2.5mm, symbol Oscillator:ASE-xxxMHz
- R35, R36, R37, R38, R39, R40, R41: footprint Resistor_SMD:R_0603_1608Metric -> Resistor_SMD:R_0402_1005Metric
Connections:
- net ISO_MCLK: now also X1.3 (OUT)
- net VDD_3.3V: now also C?.2, X1.1 (EN), X1.4 (Vdd)
- net VDD_GND: now also C?.1, X1.2 (GND)
- net AC108_3.3V: now reaches R35.2, R36.2, R38.1, R39.1, R40.1, R41.1
Other:
- note added: "MAIN_CLOCK"
Changed lines of the file:
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@@
   (junction (at 73.66 105.41) (diameter 0) (color 0 0 0 0)
   )
+  (junction (at 154.94 213.36) (diameter 0) (color 0 0 0 0)
+  )
   (junction (at 287.02 81.28) (diameter 0) (color 0 0 0 0)
   )
   (junction (at 287.02 91.44) (diameter 0) (color 0 0 0 0)
   )
+  (junction (at 170.18 234.95) (diameter 0) (color 0 0 0 0)
+  )
+  (junction (at 162.56 213.36) (diameter 0) (color 0 0 0 0)
+  )
   (junction (at 57.15 119.38) (diameter 0) (color 0 0 0 0)
   )
@@
     (stroke (width 0) (type default) (color 0 0 0 0))
   )
+  (wire (pts (xy 154.94 213.36) (xy 162.56 213.36))
+    (stroke (width 0) (type default) (color 0 0 0 0))
+  )
   (wire (pts (xy 204.47 104.14) (xy 222.25 104.14))
     (stroke (width 0) (type default) (color 0 0 0 0))
@@
     (stroke (width 0) (type default) (color 0 0 0 0))
   )
+  (wire (pts (xy 170.18 234.95) (xy 154.94 234.95))
+    (stroke (width 0) (type default) (color 0 0 0 0))
+  )
   (wire (pts (xy 125.73 104.14) (xy 143.51 104.14))
     (stroke (width 0) (type default) (color 0 0 0 0))
   )
+  (wire (pts (xy 162.56 220.98) (xy 162.56 213.36))
+    (stroke (width 0) (type default) (color 0 0 0 0))
+  )
   (polyline (pts (xy 242.57 129.54) (xy 242.57 140.97))
     (stroke (width 0) (type default) (color 0 0 0 0))
@@
     (stroke (width 0) (type default) (color 0 0 0 0))
   )
+  (wire (pts (xy 154.94 234.95) (xy 154.94 227.33))
+    (stroke (width 0) (type default) (color 0 0 0 0))
+  )
   (polyline (pts (xy 105.41 139.7) (xy 25.4 139.7))
     (stroke (width 0) (type default) (color 0 0 0 0))
@@
     (stroke (width 0) (type default) (color 0 0 0 0))
   )
+  (polyline (pts (xy 128.27 200.66) (xy 213.36 200.66))
+    (stroke (width 0) (type default) (color 0 0 0 0))
+  )
   (wire (pts (xy 82.55 97.79) (xy 100.33 97.79))
     (stroke (width 0) (type default) (color 0 0 0 0))
@@
     (stroke (width 0) (type default) (color 0 0 0 0))
   )
+  (polyline (pts (xy 128.27 200.66) (xy 128.27 246.38))
+    (stroke (width 0) (type default) (color 0 0 0 0))
+  )
   (wire (pts (xy 287.02 81.28) (xy 287.02 86.36))
     (stroke (width 0) (type default) (color 0 0 0 0))
@@
     (stroke (width 0) (type default) (color 0 0 0 0))
   )
+  (wire (pts (xy 154.94 222.25) (xy 154.94 213.36))
+    (stroke (width 0) (type default) (color 0 0 0 0))
+  )
   (wire (pts (xy 55.88 68.58) (xy 77.47 68.58))
     (stroke (width 0) (type default) (color 0 0 0 0))
@@
     (stroke (width 0) (type default) (color 0 0 0 0))
   )
+  (polyline (pts (xy 213.36 200.66) (xy 213.36 246.38))
+    (stroke (width 0) (type default) (color 0 0 0 0))
+  )
   (wire (pts (xy 57.15 127) (xy 77.47 127))
     (stroke (width 0) (type default) (color 0 0 0 0))
@@
     (stroke (width 0) (type default) (color 0 0 0 0))
   )
+  (wire (pts (xy 177.8 220.98) (xy 193.04 220.98))
+    (stroke (width 0) (type default) (color 0 0 0 0))
+  )
   (wire (pts (xy 295.91 91.44) (xy 317.5 91.44))
     (stroke (width 0) (type default) (color 0 0 0 0))
@@
     (stroke (width 0) (type default) (color 0 0 0 0))
   )
+  (wire (pts (xy 170.18 234.95) (xy 182.88 234.95))
+    (stroke (width 0) (type default) (color 0 0 0 0))
+  )
   (wire (pts (xy 82.55 68.58) (xy 100.33 68.58))
     (stroke (width 0) (type default) (color 0 0 0 0))
   )
+  (polyline (pts (xy 213.36 246.38) (xy 128.27 246.38))
+    (stroke (width 0) (type default) (color 0 0 0 0))
+  )
   (wire (pts (xy 53.34 62.23) (xy 77.47 62.23))
     (stroke (width 0) (type default) (color 0 0 0 0))
@@
     (stroke (width 0) (type default) (color 0 0 0 0))
   )
+  (wire (pts (xy 170.18 228.6) (xy 170.18 234.95))
+    (stroke (width 0) (type default) (color 0 0 0 0))
+  )
   (polyline (pts (xy 345.44 228.6) (xy 345.44 129.54))
     (stroke (width 0) (type default) (color 0 0 0 0))
@@
     (stroke (width 0) (type default) (color 0 0 0 0))
   )
+  (wire (pts (xy 162.56 213.36) (xy 170.18 213.36))
+    (stroke (width 0) (type default) (color 0 0 0 0))
+  )
   (wire (pts (xy 204.47 111.76) (xy 222.25 111.76))
     (stroke (width 0) (type default) (color 0 0 0 0))
@@
   )
   (wire (pts (xy 82.55 127) (xy 100.33 127))
+    (stroke (width 0) (type default) (color 0 0 0 0))
+  )
+  (wire (pts (xy 138.43 213.36) (xy 154.94 213.36))
     (stroke (width 0) (type default) (color 0 0 0 0))
   )
@@
     (effects (font (size 2.54 2.54)) (justify left bottom))
   )
+  (text "MAIN_CLOCK" (at 161.29 205.74 0)
+    (effects (font (size 2.54 2.54)) (justify left bottom))
+  )
   (text "ANALOG POWER" (at 280.67 24.13 0)
     (effects (font (size 2.54 2.54)) (justify left bottom))
@@
     (effects (font (size 1.27 1.27)) (justify left bottom))
   )
+  (label "VDD_3.3V" (at 142.24 213.36 0)
+    (effects (font (size 1.27 1.27)) (justify left bottom))
+  )
   (label "SDOUT1" (at 72.39 213.36 0)
     (effects (font (size 1.27 1.27)) (justify left bottom))
   )
+  (label "VDD_GND" (at 172.72 234.95 0)
+    (effects (font (size 1.27 1.27)) (justify left bottom))
+  )
   (label "AVCC_ANA1" (at 209.55 101.6 0)
     (effects (font (size 1.27 1.27)) (justify left bottom))
@@
   )
   (label "CP_VPN" (at 128.27 106.68 0)
+    (effects (font (size 1.27 1.27)) (justify left bottom))
+  )
+  (label "ISO_MCLK" (at 180.34 220.98 0)
+    (effects (font (size 1.27 1.27)) (justify left bottom))
+  )
+  (label "AC108_3.3V" (at 272.8351 81.28 0)
     (effects (font (size 1.27 1.27)) (justify left bottom))
   )
@@
     (property "Reference" "R37" (id 0) (at 289.56 71.12 90))
     (property "Value" "0" (id 1) (at 293.37 71.12 90))
-    (property "Footprint" "Resistor_SMD:R_0603_1608Metric" (id 2) (at 290.83 73.66 0)
+    (property "Footprint" "Resistor_SMD:R_0402_1005Metric" (id 2) (at 290.83 73.66 0)
       (effects (font (size 1.27 1.27)) hide)
     )
@@
     (property "Reference" "R38" (id 0) (at 292.1 78.74 90))
     (property "Value" "0" (id 1) (at 295.91 78.74 90))
-    (property "Footprint" "Resistor_SMD:R_0603_1608Metric" (id 2) (at 293.37 81.28 0)
+    (property "Footprint" "Resistor_SMD:R_0402_1005Metric" (id 2) (at 293.37 81.28 0)
       (effects (font (size 1.27 1.27)) hide)
     )
@@
     (property "Reference" "R39" (id 0) (at 292.1 83.82 90))
     (property "Value" "0" (id 1) (at 295.91 83.82 90))
-    (property "Footprint" "Resistor_SMD:R_0603_1608Metric" (id 2) (at 293.37 86.36 0)
+    (property "Footprint" "Resistor_SMD:R_0402_1005Metric" (id 2) (at 293.37 86.36 0)
       (effects (font (size 1.27 1.27)) hide)
     )
@@
     (property "Reference" "R35" (id 0) (at 265.43 78.74 90))
     (property "Value" "0" (id 1) (at 269.24 78.74 90))
-    (property "Footprint" "Resistor_SMD:R_0603_1608Metric" (id 2) (at 266.7 81.28 0)
+    (property "Footprint" "Resistor_SMD:R_0402_1005Metric" (id 2) (at 266.7 81.28 0)
       (effects (font (size 1.27 1.27)) hide)
     )
@@
     (property "Reference" "R36" (id 0) (at 265.43 85.09 90))
     (property "Value" "0" (id 1) (at 269.24 85.09 90))
-    (property "Footprint" "Resistor_SMD:R_0603_1608Metric" (id 2) (at 266.7 87.63 0)
+    (property "Footprint" "Resistor_SMD:R_0402_1005Metric" (id 2) (at 266.7 87.63 0)
       (effects (font (size 1.27 1.27)) hide)
     )
@@
     (property "Reference" "R40" (id 0) (at 292.1 88.9 90))
     (property "Value" "0" (id 1) (at 295.91 88.9 90))
-    (property "Footprint" "Resistor_SMD:R_0603_1608Metric" (id 2) (at 293.37 91.44 0)
+    (property "Footprint" "Resistor_SMD:R_0402_1005Metric" (id 2) (at 293.37 91.44 0)
       (effects (font (size 1.27 1.27)) hide)
     )
@@
     (pin "MP2")
   )
+  (symbol (lib_id "Oscillator:ASE-xxxMHz") (at 170.18 220.98 0) (unit 1)
+    (in_bom yes) (on_board yes)
+    (property "Reference" "X1" (id 0) (at 175.26 210.82 0))
+    (property "Value" "ASE-24.000MHz" (id 1) (at 181.61 213.36 0))
+    (property "Footprint" "Oscillator:Oscillator_SMD_Abracon_ASE-4Pin_3.2x2.5mm" (id 2) (at 187.96 229.87 0)
+      (effects (font (size 1.27 1.27)) hide)
+    )
+    (property "Datasheet" "http://www.abracon.com/Oscillators/ASV.pdf" (id 3) (at 167.64 220.98 0)
+      (effects (font (size 1.27 1.27)) hide)
+    )
+    (pin "1")
+    (pin "2")
+    (pin "3")
+    (pin "4")
+  )
   (symbol (lib_id "Device:R_Small_US") (at 171.45 41.91 90) (unit 1)
     (in_bom yes) (on_board yes)
@@
     (pin "2")
   )
+  (symbol (lib_id "Device:C_Small") (at 154.94 224.79 180) (unit 1)
+    (in_bom yes) (on_board yes)
+    (property "Reference" "C?" (id 0) (at 158.75 224.79 0))
+    (property "Value" "0.1uF" (id 1) (at 149.86 224.79 0))
+    (property "Footprint" "Capacitor_SMD:C_0402_1005Metric" (id 2) (at 154.94 224.79 0)
+      (effects (font (size 1.27 1.27)) hide)
+    )
+    (property "Datasheet" "~" (id 3) (at 154.94 224.79 0)
+      (effects (font (size 1.27 1.27)) hide)
+    )
+    (pin "1")
+    (pin "2")
+  )
   (symbol (lib_id "Device:R_Small_US") (at 293.37 96.52 90) (unit 1)
     (in_bom yes) (on_board yes)
     (property "Reference" "R41" (id 0) (at 292.1 93.98 90))
     (property "Value" "0" (id 1) (at 295.91 93.98 90))
-    (property "Footprint" "Resistor_SMD:R_0603_1608Metric" (id 2) (at 293.37 96.52 0)
-      (effects (font (size 1.27 1.27)) hide)
-    )
+    (property "Footprint" "Resistor_SMD:R_0402_1005Metric" (id 2) (at 293.37 96.52 0)
+      (effects (font (size 1.27 1.27)) hide)
+    )
