File: audio/4ch_mic.kicad_sch (KiCad schematic)
At the start: 67 parts, among them J11 MIC1, J12 MIC2, J13 MIC3, J14 MIC4, U10 ac108, U11 TCR3RM33, U12 TCR3RM33, X1 ASE-24.000MHz

Commit message: .
.
Parts:
- R25, R32, R33: value 0 -> NC
Connections:
- net DEV_ID0 is gone; now on net VDD_GND: U10.4 (DEV_ID0)
- net GND is gone; now on net AVCC_GND: U10.32 (VRN)
- net TEST is gone; now on net VDD_GND: U10.5 (TEST)
Changed lines of the file:
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@@
+    (effects (font (size 1.27 1.27)) (justify left bottom))
+  )
+  (label "VDD_GND" (at 128.27 137.16 0)
     (effects (font (size 1.27 1.27)) (justify left bottom))
   )
@@
     (effects (font (size 1.27 1.27)) (justify left bottom))
   )
+  (label "VDD_GND" (at 128.27 134.62 0)
+    (effects (font (size 1.27 1.27)) (justify left bottom))
+  )
   (label "AVCC_3.3V" (at 327.66 66.04 0)
     (effects (font (size 1.27 1.27)) (justify left bottom))
@@
     (effects (font (size 1.27 1.27)) (justify left bottom))
   )
-  (label "TEST" (at 128.27 137.16 0)
-    (effects (font (size 1.27 1.27)) (justify left bottom))
-  )
   (label "DLDOIN" (at 60.96 62.23 0)
     (effects (font (size 1.27 1.27)) (justify left bottom))
@@
     (effects (font (size 1.27 1.27)) (justify left bottom))
   )
-  (label "DEV_ID0" (at 128.27 134.62 0)
-    (effects (font (size 1.27 1.27)) (justify left bottom))
-  )
   (label "VCC_DIO" (at 60.96 119.38 0)
     (effects (font (size 1.27 1.27)) (justify left bottom))
@@
     (effects (font (size 1.27 1.27)) (justify left bottom))
   )
+  (label "AVCC_GND" (at 209.55 116.84 0)
+    (effects (font (size 1.27 1.27)) (justify left bottom))
+  )
   (label "MIC3N" (at 210.82 147.32 0)
     (effects (font (size 1.27 1.27)) (justify left bottom))
@@
   )
   (label "VDD_GND" (at 154.94 57.15 0)
-    (effects (font (size 1.27 1.27)) (justify left bottom))
-  )
-  (label "GND" (at 209.3526 116.84 0)
     (effects (font (size 1.27 1.27)) (justify left bottom))
   )
@@
     (in_bom yes) (on_board yes)
     (property "Reference" "R25" (id 0) (at 49.53 86.36 90))
-    (property "Value" "0" (id 1) (at 53.34 86.36 90))
+    (property "Value" "NC" (id 1) (at 53.34 86.36 90))
     (property "Footprint" "Resistor_SMD:R_0603_1608Metric" (id 2) (at 50.8 88.9 0)
       (effects (font (size 1.27 1.27)) hide)
@@
     (in_bom yes) (on_board yes)
     (property "Reference" "R32" (id 0) (at 170.18 39.37 90))
-    (property "Value" "0" (id 1) (at 173.99 39.37 90))
+    (property "Value" "NC" (id 1) (at 173.99 39.37 90))
     (property "Footprint" "Resistor_SMD:R_0603_1608Metric" (id 2) (at 171.45 41.91 0)
       (effects (font (size 1.27 1.27)) hide)
@@
     (in_bom yes) (on_board yes)
     (property "Reference" "R33" (id 0) (at 170.18 46.99 90))
-    (property "Value" "0" (id 1) (at 173.99 46.99 90))
+    (property "Value" "NC" (id 1) (at 173.99 46.99 90))
     (property "Footprint" "Resistor_SMD:R_0402_1005Metric" (id 2) (at 171.45 49.53 0)
       (effects (font (size 1.27 1.27)) hide)

Commit message: .
.
Parts:
- removed C102, C106, C108, C109, C112, C115, C80, C81, C83, C84, C85, C86, C87, C88, C89, C90, C91, C92, C93, C94, C95, C96, C97, C98, C99: 47u, Capacitor_SMD:C_0603_1608Metric, symbol Device:C
- removed C79: 1000u, Capacitor_Tantalum_SMD:CP_EIA-7360-38_Kemet-E, symbol Device:C
Other:
- moved on the sheet: C103

Commit message: .
.
Parts:
- added U15: MIC_4PIN_SMD, CM4IO:MIC_4PIN_SMD, symbol CM4IO:MIC_4PIN_SMD
Changed lines of the file:
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@@
     (pin "2")
+  )
+  (symbol (lib_id "CM4IO:MIC_4PIN_SMD") (at 322.58 151.13 0) (unit 1)
+    (in_bom yes) (on_board yes) (fields_autoplaced)
+    (property "Reference" "U15" (id 0) (at 328.93 146.05 0))
+    (property "Value" "MIC_4PIN_SMD" (id 1) (at 328.93 148.59 0))
+    (property "Footprint" "CM4IO:MIC_4PIN_SMD" (id 2) (at 322.58 151.13 0)
+      (effects (font (size 1.27 1.27)) hide)
+    )
+    (property "Datasheet" "" (id 3) (at 322.58 151.13 0)
+      (effects (font (size 1.27 1.27)) hide)
+    )
+    (pin "1")
+    (pin "2")
+    (pin "3")
+    (pin "4")
   )
   (symbol (lib_id "Device:C_Small") (at 276.86 52.07 90) (unit 1)

Commit message: .
.
Parts:
- added U16, U17, U18: MIC_4PIN_SMD, CM4IO:MIC_4PIN_SMD, symbol CM4IO:MIC_4PIN_SMD
Other:
- moved on the sheet: U15
Changed lines of the file:
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@@
     (pin "2")
+  )
+  (symbol (lib_id "CM4IO:MIC_4PIN_SMD") (at 322.58 190.5 0) (unit 1)
+    (in_bom yes) (on_board yes) (fields_autoplaced)
+    (property "Reference" "U17" (id 0) (at 328.93 185.42 0))
+    (property "Value" "MIC_4PIN_SMD" (id 1) (at 328.93 187.96 0))
+    (property "Footprint" "CM4IO:MIC_4PIN_SMD" (id 2) (at 322.58 190.5 0)
+      (effects (font (size 1.27 1.27)) hide)
+    )
+    (property "Datasheet" "" (id 3) (at 322.58 190.5 0)
+      (effects (font (size 1.27 1.27)) hide)
+    )
+    (pin "1")
+    (pin "2")
+    (pin "3")
+    (pin "4")
   )
   (symbol (lib_id "Device:C_Small") (at 67.31 46.99 90) (unit 1)
@@
     (pin "MP2")
   )
+  (symbol (lib_id "CM4IO:MIC_4PIN_SMD") (at 322.58 172.72 0) (unit 1)
+    (in_bom yes) (on_board yes) (fields_autoplaced)
+    (property "Reference" "U16" (id 0) (at 328.93 167.64 0))
+    (property "Value" "MIC_4PIN_SMD" (id 1) (at 328.93 170.18 0))
+    (property "Footprint" "CM4IO:MIC_4PIN_SMD" (id 2) (at 322.58 172.72 0)
+      (effects (font (size 1.27 1.27)) hide)
+    )
+    (property "Datasheet" "" (id 3) (at 322.58 172.72 0)
+      (effects (font (size 1.27 1.27)) hide)
+    )
+    (pin "1")
+    (pin "2")
+    (pin "3")
+    (pin "4")
+  )
   (symbol (lib_id "Device:C_Small") (at 80.01 68.58 90) (unit 1)
     (in_bom yes) (on_board yes)
@@
     (pin "2")
   )
+  (symbol (lib_id "CM4IO:MIC_4PIN_SMD") (at 322.58 209.55 0) (unit 1)
+    (in_bom yes) (on_board yes) (fields_autoplaced)
+    (property "Reference" "U18" (id 0) (at 328.93 204.47 0))
+    (property "Value" "MIC_4PIN_SMD" (id 1) (at 328.93 207.01 0))
+    (property "Footprint" "CM4IO:MIC_4PIN_SMD" (id 2) (at 322.58 209.55 0)
+      (effects (font (size 1.27 1.27)) hide)
+    )
+    (property "Datasheet" "" (id 3) (at 322.58 209.55 0)
+      (effects (font (size 1.27 1.27)) hide)
+    )
+    (pin "1")
+    (pin "2")
+    (pin "3")
+    (pin "4")
+  )
   (symbol (lib_id "Device:R_Small_US") (at 50.8 88.9 90) (unit 1)
     (in_bom yes) (on_board yes)
@@
     (pin "2")
   )
-  (symbol (lib_id "CM4IO:MIC_4PIN_SMD") (at 322.58 151.13 0) (unit 1)
-    (in_bom yes) (on_board yes) (fields_autoplaced)
-    (property "Reference" "U15" (id 0) (at 328.93 146.05 0))
-    (property "Value" "MIC_4PIN_SMD" (id 1) (at 328.93 148.59 0))
-    (property "Footprint" "CM4IO:MIC_4PIN_SMD" (id 2) (at 322.58 151.13 0)
-      (effects (font (size 1.27 1.27)) hide)
-    )
-    (property "Datasheet" "" (id 3) (at 322.58 151.13 0)
-      (effects (font (size 1.27 1.27)) hide)
-    )
+  (symbol (lib_id "CM4IO:MIC_4PIN_SMD") (at 322.58 149.86 0) (unit 1)
+    (in_bom yes) (on_board yes) (fields_autoplaced)
+    (property "Reference" "U15" (id 0) (at 328.93 144.78 0))
+    (property "Value" "MIC_4PIN_SMD" (id 1) (at 328.93 147.32 0))
+    (property "Footprint" "CM4IO:MIC_4PIN_SMD" (id 2) (at 322.58 149.86 0)
+      (effects (font (size 1.27 1.27)) hide)
+    )
+    (property "Datasheet" "" (id 3) (at 322.58 149.86 0)
+      (effects (font (size 1.27 1.27)) hide)
+    )
