File: audio/4ch_mic.kicad_sch (KiCad schematic)
At the start: 45 parts, among them J11 MIC1, J12 MIC2, J13 MIC3, J14 MIC4, U10 ac108, U11 TCR3RM33, U12 TCR3RM33, U15 MIC_4PIN_SMD, U16 MIC_4PIN_SMD, U17 MIC_4PIN_SMD, U18 MIC_4PIN_SMD, X1 ASE-24.000MHz

Commit message: .
.
Parts:
- removed J11: MIC1, CM4IO:GROVE_4PIN, symbol CM4IO:GROVE_4PIN
- removed J12: MIC2, CM4IO:GROVE_4PIN, symbol CM4IO:GROVE_4PIN
- removed J13: MIC3, CM4IO:GROVE_4PIN, symbol CM4IO:GROVE_4PIN
- removed J14: MIC4, CM4IO:GROVE_4PIN, symbol CM4IO:GROVE_4PIN
Connections:
- net AVCC_3.3V: now also U15.1 (VDD), U16.1 (VDD), U17.1 (VDD), U18.1 (VDD)
- net AVCC_GND: now also U15.2 (GND), U16.2 (GND), U17.2 (GND), U18.2 (GND)
- net MIC1N: now also U18.4 (MIC-)
- net MIC1P: now also U18.3 (MIC+)
- net MIC2N: now also U17.4 (MIC-)
- net MIC2P: now also U17.3 (MIC+)
- net MIC3N: now also U16.4 (MIC-)
- net MIC3P: now also U16.3 (MIC+)
- net MIC4N: now also U15.4 (MIC-)
- net MIC4P: now also U15.3 (MIC+)
Other:
- moved on the sheet: U15, U16, U17, U18

Commit message: .
.
Parts:
- added R37, R38, R39, R40, R41, R54, R55, R56, R57, R7, R8, R9: 0, Resistor_SMD:R_0402_1005Metric, symbol Device:R_Small_US
Connections:
- net AVCC_GND: now also R37.1, R39.1, R41.1, R8.1
- net MIC1N: now also R7.2, R8.2; no longer U18.4 (MIC-)
- net MIC1P: now also R54.2; no longer U18.3 (MIC+)
- net MIC2N: now also R37.2, R9.2; no longer U17.4 (MIC-)
- net MIC2P: now also R55.2; no longer U17.3 (MIC+)
- net MIC3N: now also R38.2, R39.2; no longer U16.4 (MIC-)
- net MIC3P: now also R56.2; no longer U16.3 (MIC+)
- net MIC4N: now also R40.2, R41.2; no longer U15.4 (MIC-)
- net MIC4P: now also R57.2; no longer U15.3 (MIC+)
- new net MIC1_CON_N: R7.1, U18.4 (MIC-)
- new net MIC1_CON_P: R54.1, U18.3 (MIC+)
- new net MIC2_CON_N: R9.1, U17.4 (MIC-)
- new net MIC2_CON_P: R55.1, U17.3 (MIC+)
- new net MIC3_CON_N: R38.1, U16.4 (MIC-)
- new net MIC3_CON_P: R56.1, U16.3 (MIC+)
- new net MIC4_CON_N: R40.1, U15.4 (MIC-)
- new net MIC4_CON_P: R57.1, U15.3 (MIC+)
Other:
- moved on the sheet: U15, U16, U17, U18

Commit message: ,
,
Parts:
- C103: value 47u -> 10u
Changed lines of the file:
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@@
       (effects (font (size 1.27 1.27)) (justify left))
     )
-    (property "Value" "47u" (at 371.221 30.353 0)
+    (property "Value" "10u" (at 371.221 30.353 0)
       (effects (font (size 1.27 1.27)) (justify left))
     )

Commit message: USB_OK
.
Parts:
- R37, R39, R41, R8: value 0 -> NC
Changed lines of the file:
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@@
   (junction (at 325.12 170.18) (diameter 0) (color 0 0 0 0)
-  )
-  (junction (at 295.91 74.93) (diameter 0) (color 0 0 0 0)
   )
   (junction (at 73.66 105.41) (diameter 0) (color 0 0 0 0)
@@
   )
   (wire (pts (xy 57.15 119.38) (xy 77.47 119.38))
-    (stroke (width 0) (type default))
-  )
-  (wire (pts (xy 295.91 74.93) (xy 298.45 74.93))
     (stroke (width 0) (type default))
   )
@@
       (effects (font (size 1.27 1.27)))
     )
-    (property "Value" "0" (at 327.66 185.42 90)
+    (property "Value" "NC" (at 327.66 185.42 90)
       (effects (font (size 1.27 1.27)))
     )
@@
       (effects (font (size 1.27 1.27)))
     )
-    (property "Value" "0" (at 327.66 204.47 90)
+    (property "Value" "NC" (at 327.66 204.47 90)
       (effects (font (size 1.27 1.27)))
     )
@@
       (effects (font (size 1.27 1.27)))
     )
-    (property "Value" "0" (at 327.66 167.64 90)
+    (property "Value" "NC" (at 327.66 167.64 90)
       (effects (font (size 1.27 1.27)))
     )
@@
       (effects (font (size 1.27 1.27)))
     )
-    (property "Value" "0" (at 327.66 148.59 90)
-      (effects (font (size 1.27 1.27)))
-    )
+    (property "Value" "NC" (at 327.66 148.59 90)
+      (effects (font (size 1.27 1.27)))
+    )
