File: audio/PCIe-USB3.kicad_sch (KiCad schematic)
At the start: 55 parts, among them J2 Conn_02x05_Odd_Even, J3 USB3_A, Q1 DMG1012T, U2 AP3429KTTR-G1, U3 VL805, U4 AP22653W6, Y1 25MHz

Commit message: .
.
Parts:
- removed J2: Conn_02x05_Odd_Even, Connector_PinHeader_2.54mm:PinHeader_2x05_P2.54mm_Vertical, symbol Connector_Generic:Conn_02x05_Odd_Even
Connections:
- no-connect marks 21 -> 19
Other:
- note removed: "Expansion USB connector"
Changed lines of the file:
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@@
   (no_connect (at 200.66 116.84))
   (no_connect (at 200.66 114.3))
-  (no_connect (at 253.2888 129.8702))
   (no_connect (at 100.965 34.925))
   (no_connect (at 100.965 45.085))
   (no_connect (at 131.445 57.785))
-  (no_connect (at 265.9888 129.8702))
   (no_connect (at 131.445 60.325))
   (no_connect (at 200.66 105.41))
@@
     (stroke (width 0) (type solid) (color 0 0 0 0))
   )
-  (wire (pts (xy 274.8788 124.7902) (xy 265.9888 124.7902))
-    (stroke (width 0) (type solid) (color 0 0 0 0))
-  )
   (wire (pts (xy 32.385 35.56) (xy 37.465 35.56))
     (stroke (width 0) (type solid) (color 0 0 0 0))
@@
     (stroke (width 0) (type solid) (color 0 0 0 0))
   )
-  (wire (pts (xy 274.8788 119.7102) (xy 265.9888 119.7102))
-    (stroke (width 0) (type solid) (color 0 0 0 0))
-  )
   (wire (pts (xy 113.157 154.813) (xy 116.967 154.813))
     (stroke (width 0) (type solid) (color 0 0 0 0))
@@
     (stroke (width 0) (type solid) (color 0 0 0 0))
   )
-  (wire (pts (xy 250.7488 127.3302) (xy 253.2888 127.3302))
-    (stroke (width 0) (type solid) (color 0 0 0 0))
-  )
   (wire (pts (xy 188.087 154.813) (xy 198.247 154.813))
     (stroke (width 0) (type solid) (color 0 0 0 0))
@@
     (stroke (width 0) (type solid) (color 0 0 0 0))
   )
-  (wire (pts (xy 244.3988 119.7102) (xy 253.2888 119.7102))
-    (stroke (width 0) (type solid) (color 0 0 0 0))
-  )
   (wire (pts (xy 137.287 162.433) (xy 146.177 162.433))
     (stroke (width 0) (type solid) (color 0 0 0 0))
@@
     (stroke (width 0) (type solid) (color 0 0 0 0))
   )
-  (wire (pts (xy 268.5288 127.3302) (xy 268.5288 131.1402))
-    (stroke (width 0) (type solid) (color 0 0 0 0))
-  )
   (wire (pts (xy 200.66 97.79) (xy 212.09 97.79))
     (stroke (width 0) (type solid) (color 0 0 0 0))
@@
     (stroke (width 0) (type solid) (color 0 0 0 0))
   )
-  (wire (pts (xy 244.3988 122.2502) (xy 253.2888 122.2502))
-    (stroke (width 0) (type solid) (color 0 0 0 0))
-  )
   (wire (pts (xy 69.469 115.697) (xy 75.819 115.697))
     (stroke (width 0) (type solid) (color 0 0 0 0))
@@
     (stroke (width 0) (type solid) (color 0 0 0 0))
   )
-  (wire (pts (xy 265.9888 127.3302) (xy 268.5288 127.3302))
-    (stroke (width 0) (type solid) (color 0 0 0 0))
-  )
   (wire (pts (xy 27.051 71.755) (xy 35.941 71.755))
     (stroke (width 0) (type solid) (color 0 0 0 0))
@@
     (stroke (width 0) (type solid) (color 0 0 0 0))
   )
-  (wire (pts (xy 274.8788 122.2502) (xy 265.9888 122.2502))
-    (stroke (width 0) (type solid) (color 0 0 0 0))
-  )
   (wire (pts (xy 98.425 67.945) (xy 98.425 69.215))
     (stroke (width 0) (type solid) (color 0 0 0 0))
@@
     (stroke (width 0) (type solid) (color 0 0 0 0))
   )
-  (wire (pts (xy 250.7488 127.3302) (xy 250.7488 131.1402))
-    (stroke (width 0) (type solid) (color 0 0 0 0))
-  )
   (wire (pts (xy 26.289 110.617) (xy 31.369 110.617))
     (stroke (width 0) (type solid) (color 0 0 0 0))
@@
   )
   (wire (pts (xy 208.28 53.34) (xy 212.09 53.34))
-    (stroke (width 0) (type solid) (color 0 0 0 0))
-  )
-  (wire (pts (xy 244.3988 124.7902) (xy 253.2888 124.7902))
     (stroke (width 0) (type solid) (color 0 0 0 0))
   )
@@
     (at 16.51 138.43 0)
     (effects (font (size 1.27 1.27)) (justify left bottom))
-  )
-  (text "Expansion USB connector" (at 269.5194 111.252 180)
-    (effects (font (size 1.27 1.27)) (justify right bottom))
   )
   (text "Stacked USB connectors" (at 279.3238 97.8662 180)
@@
     (effects (font (size 1.27 1.27)) (justify left bottom))
   )
-  (label "VBUS" (at 244.3988 119.7102 0)
-    (effects (font (size 1.27 1.27)) (justify left bottom))
-  )
   (label "C1_N" (at 201.93 22.86 0)
-    (effects (font (size 1.27 1.27)) (justify left bottom))
-  )
-  (label "PD4_N" (at 269.0622 122.2502 0)
     (effects (font (size 1.27 1.27)) (justify left bottom))
   )
@@
     (effects (font (size 1.27 1.27)) (justify left bottom))
   )
-  (label "VBUS" (at 274.8788 119.7102 180)
-    (effects (font (size 1.27 1.27)) (justify right bottom))
-  )
   (label "PD1_N" (at 201.93 40.64 0)
     (effects (font (size 1.27 1.27)) (justify left bottom))
@@
     (effects (font (size 1.27 1.27)) (justify right bottom))
   )
-  (label "PD3_P" (at 244.3988 124.7902 0)
-    (effects (font (size 1.27 1.27)) (justify left bottom))
-  )
   (label "A1.05v" (at 153.035 50.8 0)
     (effects (font (size 1.27 1.27)) (justify left bottom))
   )
   (label "SSRX1_N" (at 241.3 69.85 0)
-    (effects (font (size 1.27 1.27)) (justify left bottom))
-  )
-  (label "PD3_N" (at 244.3988 122.2502 0)
-    (effects (font (size 1.27 1.27)) (justify left bottom))
-  )
-  (label "PD4_P" (at 269.0876 124.7902 0)
     (effects (font (size 1.27 1.27)) (justify left bottom))
   )
@@
     (pin "1")
     (pin "2")
-  )
-  (symbol (lib_id "power:GND") (at 268.5288 131.1402 0) (mirror y) (unit 1)
-    (in_bom yes) (on_board yes)
-    (property "Reference" "#PWR0108" (id 0) (at 268.5288 137.4902 0)
-      (effects (font (size 1.27 1.27)) hide)
-    )
-    (property "Value" "GND" (id 1) (at 268.4018 135.5344 0))
-    (property "Footprint" "" (id 2) (at 268.5288 131.1402 0)
-      (effects (font (size 1.27 1.27)) hide)
-    )
-    (property "Datasheet" "" (id 3) (at 268.5288 131.1402 0)
-      (effects (font (size 1.27 1.27)) hide)
-    )
-    (pin "1")
   )
   (symbol (lib_id "Device:C") (at 128.27 184.15 0) (unit 1)
@@
     (pin "B9")
   )
-  (symbol (lib_id "power:GND") (at 250.7488 131.1402 0) (unit 1)
-    (in_bom yes) (on_board yes)
-    (property "Reference" "#PWR0107" (id 0) (at 250.7488 137.4902 0)
-      (effects (font (size 1.27 1.27)) hide)
-    )
-    (property "Value" "GND" (id 1) (at 250.8758 135.5344 0))
-    (property "Footprint" "" (id 2) (at 250.7488 131.1402 0)
-      (effects (font (size 1.27 1.27)) hide)
-    )
-    (property "Datasheet" "" (id 3) (at 250.7488 131.1402 0)
-      (effects (font (size 1.27 1.27)) hide)
-    )
-    (pin "1")
-  )
-  (symbol (lib_id "Connector_Generic:Conn_02x05_Odd_Even") (at 258.3688 124.7902 0) (unit 1)
-    (in_bom yes) (on_board yes)
-    (property "Reference" "J2" (id 0) (at 259.6386 114.1988 0))
-    (property "Value" "Conn_02x05_Odd_Even" (id 1) (at 259.6388 116.5098 0))
-    (property "Footprint" "Connector_PinHeader_2.54mm:PinHeader_2x05_P2.54mm_Vertical" (id 2) (at 258.3688 124.7902 0)
-      (effects (font (size 1.27 1.27)) hide)
-    )
-    (property "Datasheet" "https://www.toby.co.uk/uploads/publications/1673.pdf" (id 3) (at 258.3688 124.7902 0)
-      (effects (font (size 1.27 1.27)) hide)
-    )
-    (property "Field4" "Toby" (id 4) (at 258.3688 124.7902 0)
-      (effects (font (size 1.27 1.27)) hide)
-    )
-    (property "Field5" "THD-05-R" (id 5) (at 258.3688 124.7902 0)
-      (effects (font (size 1.27 1.27)) hide)
-    )
-    (property "Field6" "THD-05-R" (id 6) (at 258.3688 124.7902 0)
-      (effects (font (size 1.27 1.27)) hide)
-    )
-    (property "Field7" "Toby" (id 7) (at 258.3688 124.7902 0)
-      (effects (font (size 1.27 1.27)) hide)
-    )
-    (property "Part Description" "PinHeader_2x05_P2.54mm_Vertical" (id 8) (at 258.3688 124.7902 0)
-      (effects (font (size 1.27 1.27)) hide)
-    )
-    (pin "1")
-    (pin "10")
-    (pin "2")
-    (pin "3")
-    (pin "4")
-    (pin "5")
-    (pin "6")
-    (pin "7")
-    (pin "8")
-    (pin "9")
-  )
   (symbol (lib_id "CM4:VL805") (at 118.745 56.515 0) (unit 4)

Commit message: .
.
Parts:
- removed U2: AP3429KTTR-G1, Package_TO_SOT_SMD:TSOT-23-5, symbol CM4:AP3429KTTR-G1
- added C40: 22u, Capacitor_SMD:C_0805_2012Metric, symbol Device:C
- added U8: AP3402, Package_TO_SOT_SMD:TSOT-23-6, symbol Regulator_Switching:AP3402
- C17, C7: value 10u -> 22u
- L2: value 2.2uH -> 1.0uH
Connections:
- net +5v: now also U8.4 (VIN)
- net GND: now also C40.2, U8.2 (GND)
- net at C12.1, C17.1, C21.1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: now also C40.1
- net at C12.2, R6.2, R7.1: now also U8.6 (FB)
- net at R1.2, R2.1: now also U8.1 (EN)
- net at L2.1: now also U8.3 (LX)
Other:
- moved on the sheet: C21, C24, C26, C28, C29, C30, C31, C32, C33, C34, C7, L3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

Commit message: .
.
Connections:
- net SW_OUT: now reaches C12.1, C17.1, C21.1, C40.1, L2.2, L3.1, R6.1
- net FB: now reaches C12.2, R6.2, R7.1, U8.6 (FB)
- net EN: now reaches R1.2, R2.1, U8.1 (EN)
- net clock2: now reaches C16.1, U3.48 (SSX0), Y1.3
- net clock1: now reaches C11.1, U3.47 (SSXI), Y1.1
- net LX: now reaches L2.1, U8.3 (LX)
- net PG: now reaches U8.5 (PG)
Changed lines of the file:
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@@
     (stroke (width 0) (type solid) (color 0 0 0 0))
+  )
+  (wire (pts (xy 40.767 157.353) (xy 45.847 157.353))
+    (stroke (width 0) (type default) (color 0 0 0 0))
   )
   (wire (pts (xy 33.02 187.96) (xy 57.15 187.96))
@@
     (effects (font (size 1.27 1.27)) (justify left bottom))
   )
+  (label "SW_OUT" (at 92.6289 154.813 0)
+    (effects (font (size 1.27 1.27)) (justify left bottom))
+  )
   (label "C2_N" (at 201.93 50.8 0)
     (effects (font (size 1.27 1.27)) (justify left bottom))
@@
     (effects (font (size 1.27 1.27)) (justify left bottom))
   )
+  (label "FB" (at 67.31 159.893 0)
+    (effects (font (size 1.27 1.27)) (justify left bottom))
+  )
   (label "PD1_N" (at 201.93 40.64 0)
     (effects (font (size 1.27 1.27)) (justify left bottom))
@@
     (effects (font (size 1.27 1.27)) (justify left bottom))
   )
+  (label "clock2" (at 92.71 67.945 0)
+    (effects (font (size 1.27 1.27)) (justify left bottom))
+  )
   (label "PEXTX_N" (at 52.705 33.02 180)
     (effects (font (size 1.27 1.27)) (justify right bottom))
@@
     (effects (font (size 1.27 1.27)) (justify left bottom))
   )
+  (label "EN" (at 41.91 159.893 0)
+    (effects (font (size 1.27 1.27)) (justify left bottom))
+  )
   (label "SSRX1_N" (at 241.3 69.85 0)
     (effects (font (size 1.27 1.27)) (justify left bottom))
@@
     (effects (font (size 1.27 1.27)) (justify left bottom))
   )
+  (label "clock1" (at 80.5151 67.945 0)
+    (effects (font (size 1.27 1.27)) (justify left bottom))
+  )
   (label "SSRX1_P" (at 201.93 29.21 0)
     (effects (font (size 1.27 1.27)) (justify left bottom))
@@
     (effects (font (size 1.27 1.27)) (justify left bottom))
   )
+  (label "PG" (at 42.0329 157.353 0)
+    (effects (font (size 1.27 1.27)) (justify left bottom))
+  )
   (label "SSTX1_N" (at 241.3 77.47 0)
     (effects (font (size 1.27 1.27)) (justify left bottom))
@@
     (effects (font (size 1.27 1.27)) (justify left bottom))
   )
+  (label "LX" (at 67.6064 154.813 0)
+    (effects (font (size 1.27 1.27)) (justify left bottom))
+  )

Commit message: .
.
Connections:
- net ILIM: now reaches R5.1, U4.5 (ILIM)
Changed lines of the file:
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@@
+    (effects (font (size 1.27 1.27)) (justify left bottom))
+  )
+  (label "ILIM" (at 72.1835 113.157 0)
     (effects (font (size 1.27 1.27)) (justify left bottom))
   )

Commit message: .
.
Parts:
- added C72: 100n, Capacitor_SMD:C_0402_1005Metric, symbol Device:C
Connections:
- net A1.05v: now also C72.1
- net GND: now also C72.2
Changed lines of the file:
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@@
   (junction (at 123.952 162.433) (diameter 1.016) (color 0 0 0 0)
   )
+  (junction (at 229.8474 154.807) (diameter 0) (color 0 0 0 0)
+  )
   (junction (at 87.63 187.96) (diameter 1.016) (color 0 0 0 0)
   )
@@
   (junction (at 161.925 20.32) (diameter 1.016) (color 0 0 0 0)
   )
+  (junction (at 219.202 162.433) (diameter 0) (color 0 0 0 0)
+  )
   (junction (at 78.105 67.945) (diameter 1.016) (color 0 0 0 0)
   )
@@
   (junction (at 148.082 162.433) (diameter 1.016) (color 0 0 0 0)
   )
+  (junction (at 219.202 162.427) (diameter 0) (color 0 0 0 0)
+  )
   (junction (at 78.867 154.813) (diameter 1.016) (color 0 0 0 0)
   )
@@
     (stroke (width 0) (type solid) (color 0 0 0 0))
   )
+  (wire (pts (xy 229.8474 154.807) (xy 237.8233 154.807))
+    (stroke (width 0) (type solid) (color 0 0 0 0))
+  )
   (wire (pts (xy 35.941 79.375) (xy 35.941 84.455))
     (stroke (width 0) (type solid) (color 0 0 0 0))
   )
+  (wire (pts (xy 219.202 162.427) (xy 219.202 162.433))
+    (stroke (width 0) (type default) (color 0 0 0 0))
+  )
   (wire (pts (xy 200.66 38.1) (xy 212.09 38.1))
     (stroke (width 0) (type solid) (color 0 0 0 0))
@@
     (stroke (width 0) (type solid) (color 0 0 0 0))
   )
-  (wire (pts (xy 219.202 154.813) (xy 229.362 154.813))
+  (wire (pts (xy 227.6633 154.807) (xy 229.8474 154.807))
     (stroke (width 0) (type solid) (color 0 0 0 0))
   )
@@
     (stroke (width 0) (type solid) (color 0 0 0 0))
   )
+  (wire (pts (xy 227.6633 154.807) (xy 219.202 154.813))
+    (stroke (width 0) (type default) (color 0 0 0 0))
+  )
   (wire (pts (xy 254 83.82) (xy 254 86.36))
     (stroke (width 0) (type solid) (color 0 0 0 0))
@@
     (stroke (width 0) (type default) (color 0 0 0 0))
   )
+  (wire (pts (xy 229.8474 162.427) (xy 219.202 162.427))
+    (stroke (width 0) (type default) (color 0 0 0 0))
+  )
   (wire (pts (xy 33.02 187.96) (xy 57.15 187.96))
     (stroke (width 0) (type solid) (color 0 0 0 0))
@@
     (effects (font (size 1.27 1.27)) (justify left bottom))
   )
-  (label "A1.05v" (at 223.012 154.813 0)
+  (label "A1.05v" (at 231.4733 154.807 0)
     (effects (font (size 1.27 1.27)) (justify left bottom))
   )
@@
       (effects (font (size 1.27 1.27)) hide)
     )
+    (pin "1")
+    (pin "2")
+  )
+  (symbol (lib_id "Device:C") (at 229.8474 158.617 0) (unit 1)
+    (in_bom yes) (on_board yes)
+    (property "Reference" "C72" (id 0) (at 232.7684 157.4486 0)
+      (effects (font (size 1.27 1.27)) (justify left))
+    )
+    (property "Value" "100n" (id 1) (at 232.7684 159.76 0)
+      (effects (font (size 1.27 1.27)) (justify left))
+    )
+    (property "Footprint" "Capacitor_SMD:C_0402_1005Metric" (id 2) (at 230.8126 162.427 0)
+      (effects (font (size 1.27 1.27)) hide)
+    )
+    (property "Datasheet" "https://search.murata.co.jp/Ceramy/image/img/A01X/G101/ENG/GRM155R71C104KA88-01.pdf" (id 3) (at 229.8474 158.617 0)
+      (effects (font (size 1.27 1.27)) hide)
+    )
+    (property "Field4" "Farnell" (id 4) (at 229.8474 158.617 0)
+      (effects (font (size 1.27 1.27)) hide)
+    )
+    (property "Field5" "2611911" (id 5) (at 229.8474 158.617 0)
+      (effects (font (size 1.27 1.27)) hide)
+    )
+    (property "Field6" "RM EMK105 B7104KV-F" (id 6) (at 229.8474 158.617 0)
+      (effects (font (size 1.27 1.27)) hide)
+    )
+    (property "Field7" "TAIYO YUDEN EUROPE GMBH" (id 7) (at 229.8474 158.617 0)
+      (effects (font (size 1.27 1.27)) hide)
+    )
+    (property "Field8" "110091611" (id 8) (at 229.8474 158.617 0)
+      (effects (font (size 1.27 1.27)) hide)
+    )
+    (property "Part Description" "	0.1uF 10% 16V Ceramic Capacitor X7R 0402 (1005 Metric)" (id 9) (at 229.8474 158.617 0)
+      (effects (font (size 1.27 1.27)) hide)
+    )

Commit message: .
.
Parts:
- C14: footprint Capacitor_Tantalum_SMD:CP_EIA-7343-31_Kemet-D -> Capacitor_Tantalum_SMD:CP_EIA-3528-21_Kemet-B
Connections:
- net SSREXT: now reaches R8.1, U3.50 (SSREXT)
Other:
- moved on the sheet: R8
Changed lines of the file:
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@@
-    (stroke (width 0) (type solid) (color 0 0 0 0))
-  )
-  (wire (pts (xy 132.715 62.865) (xy 132.715 64.135))
     (stroke (width 0) (type solid) (color 0 0 0 0))
   )
@@
     (stroke (width 0) (type solid) (color 0 0 0 0))
   )
-  (wire (pts (xy 131.445 62.865) (xy 132.715 62.865))
+  (wire (pts (xy 131.445 62.865) (xy 144.7717 62.865))
     (stroke (width 0) (type solid) (color 0 0 0 0))
   )
@@
   )
   (label "SSRX1_N" (at 241.3 69.85 0)
+    (effects (font (size 1.27 1.27)) (justify left bottom))
+  )
+  (label "SSREXT" (at 133.9575 62.865 0)
     (effects (font (size 1.27 1.27)) (justify left bottom))
   )
@@
     (pin "1")
   )
-  (symbol (lib_id "Device:R") (at 132.715 67.945 0) (unit 1)
-    (in_bom yes) (on_board yes)
-    (property "Reference" "R8" (id 0) (at 134.493 66.7766 0)
-      (effects (font (size 1.27 1.27)) (justify left))
-    )
-    (property "Value" "6.04K" (id 1) (at 134.493 69.088 0)
-      (effects (font (size 1.27 1.27)) (justify left))
-    )
-    (property "Footprint" "Resistor_SMD:R_0402_1005Metric" (id 2) (at 130.937 67.945 90)
-      (effects (font (size 1.27 1.27)) hide)
-    )
-    (property "Datasheet" "https://fscdn.rohm.com/en/products/databook/datasheet/passive/resistor/chip_resistor/mcr-e.pdf" (id 3) (at 132.715 67.945 0)
-      (effects (font (size 1.27 1.27)) hide)
-    )
-    (property "Field4" "Farnell" (id 4) (at 132.715 67.945 0)
-      (effects (font (size 1.27 1.27)) hide)
-    )
-    (property "Field6" "MCR01MZPF6041" (id 5) (at 132.715 67.945 0)
-      (effects (font (size 1.27 1.27)) hide)
-    )
-    (property "Field7" "Rohm" (id 6) (at 132.715 67.945 0)
-      (effects (font (size 1.27 1.27)) hide)
-    )
-    (property "Part Description" "Resistor 6.04K M1005 1% 63mW" (id 7) (at 132.715 67.945 0)
+  (symbol (lib_id "Device:R") (at 144.7717 66.675 0) (unit 1)
+    (in_bom yes) (on_board yes)
+    (property "Reference" "R8" (id 0) (at 146.5497 65.5066 0)
+      (effects (font (size 1.27 1.27)) (justify left))
+    )
+    (property "Value" "6.04K" (id 1) (at 146.5497 67.818 0)
+      (effects (font (size 1.27 1.27)) (justify left))
+    )
+    (property "Footprint" "Resistor_SMD:R_0402_1005Metric" (id 2) (at 142.9937 66.675 90)
+      (effects (font (size 1.27 1.27)) hide)
+    )
+    (property "Datasheet" "https://fscdn.rohm.com/en/products/databook/datasheet/passive/resistor/chip_resistor/mcr-e.pdf" (id 3) (at 144.7717 66.675 0)
+      (effects (font (size 1.27 1.27)) hide)
+    )
+    (property "Field4" "Farnell" (id 4) (at 144.7717 66.675 0)
+      (effects (font (size 1.27 1.27)) hide)
+    )
+    (property "Field6" "MCR01MZPF6041" (id 5) (at 144.7717 66.675 0)
+      (effects (font (size 1.27 1.27)) hide)
+    )
+    (property "Field7" "Rohm" (id 6) (at 144.7717 66.675 0)
+      (effects (font (size 1.27 1.27)) hide)
+    )
+    (property "Part Description" "Resistor 6.04K M1005 1% 63mW" (id 7) (at 144.7717 66.675 0)
       (effects (font (size 1.27 1.27)) hide)
     )
@@
       (effects (font (size 1.27 1.27)) (justify left))
     )
-    (property "Footprint" "Capacitor_Tantalum_SMD:CP_EIA-7343-31_Kemet-D" (id 2) (at 89.9922 120.777 0)
-      (effects (font (size 1.27 1.27)) hide)
-    )
+    (property "Footprint" "Capacitor_Tantalum_SMD:CP_EIA-3528-21_Kemet-B" (id 2) (at 89.9922 120.777 0))
     (property "Datasheet" "~" (id 3) (at 89.027 116.967 0)
       (effects (font (size 1.27 1.27)) hide)
@@
     (pin "2")
   )
-  (symbol (lib_id "power:GND") (at 132.715 71.755 0) (unit 1)
-    (in_bom yes) (on_board yes)
-    (property "Reference" "#PWR0120" (id 0) (at 132.715 78.105 0)
-      (effects (font (size 1.27 1.27)) hide)
-    )
-    (property "Value" "GND" (id 1) (at 132.842 76.1492 0))
-    (property "Footprint" "" (id 2) (at 132.715 71.755 0)
-      (effects (font (size 1.27 1.27)) hide)
-    )
-    (property "Datasheet" "" (id 3) (at 132.715 71.755 0)
-      (effects (font (size 1.27 1.27)) hide)
-    )
+  (symbol (lib_id "power:GND") (at 144.7717 70.485 0) (unit 1)
+    (in_bom yes) (on_board yes)
+    (property "Reference" "#PWR0120" (id 0) (at 144.7717 76.835 0)
+      (effects (font (size 1.27 1.27)) hide)
+    )
+    (property "Value" "GND" (id 1) (at 144.8987 74.8792 0))
+    (property "Footprint" "" (id 2) (at 144.7717 70.485 0)
+      (effects (font (size 1.27 1.27)) hide)
+    )
+    (property "Datasheet" "" (id 3) (at 144.7717 70.485 0)
+      (effects (font (size 1.27 1.27)) hide)
+    )

Commit message: .
.
Parts:
- L2: value 1.0uH -> 2.2uH
- R6: value 12K 1% -> 120K 1%
- R7: value 16K -> 160K
Changed lines of the file:
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@@
       (effects (font (size 1.27 1.27)) (justify left))
     )
-    (property "Value" "16K" (id 1) (at 89.535 168.656 0)
+    (property "Value" "160K" (id 1) (at 89.535 168.656 0)
       (effects (font (size 1.27 1.27)) (justify left))
     )
@@
       (effects (font (size 1.27 1.27)) (justify left))
     )
-    (property "Value" "12K 1%" (id 1) (at 89.535 159.766 0)
+    (property "Value" "120K 1%" (id 1) (at 89.535 159.766 0)
       (effects (font (size 1.27 1.27)) (justify left))
     )
@@
     (in_bom yes) (on_board yes)
     (property "Reference" "L2" (id 0) (at 75.057 149.987 90))
-    (property "Value" "1.0uH" (id 1) (at 75.057 152.2984 90))
+    (property "Value" "2.2uH" (id 1) (at 75.057 152.2984 90))
     (property "Footprint" "Inductor_SMD:L_1008_2520Metric" (id 2) (at 75.057 154.813 0)
       (effects (font (size 1.27 1.27)) hide)
@@
   (symbol (lib_id "Regulator_Switching:AP3402") (at 56.007 157.353 0) (unit 1)
     (in_bom yes) (on_board yes) (fields_autoplaced)
-    (property "Reference" "U8" (id 0) (at 56.007 147.193 0))
-    (property "Value" "AP3402" (id 1) (at 56.007 149.733 0))
+    (property "Reference" "U8" (id 0) (at 56.007 147.32 0))
+    (property "Value" "AP3402" (id 1) (at 56.007 149.86 0))
     (property "Footprint" "Package_TO_SOT_SMD:TSOT-23-6" (id 2) (at 56.007 157.353 0)
       (effects (font (size 1.27 1.27)) hide)

Commit message: .
.
Parts:
- removed C10, C13, C15, C19, C21, C22, C23, C27, C28, C29, C30, C31, C32, C33, C34, C35, C36, C37, C38, C5, C6, C72, C9: 100n, Capacitor_SMD:C_0402_1005Metric, symbol Device:C
- removed C11, C12, C16: 22pF, Capacitor_SMD:C_0402_1005Metric, symbol Device:C
- removed C14: 100uF, Capacitor_Tantalum_SMD:CP_EIA-3528-21_Kemet-B, symbol Device:CP
- removed C17, C40, C7: 22u, Capacitor_SMD:C_0805_2012Metric, symbol Device:C
- removed C18, C20, C24, C25, C26, C3, C4, C8: 10u, Capacitor_SMD:C_0805_2012Metric, symbol Device:C
- removed J3: USB3_A, CM4IO:MTCONN_UBAF30-D2011, symbol CM4:USB3_A
- removed L1, L3: BLM18AG221SN1, Inductor_SMD:L_0603_1608Metric, symbol Device:L
- removed L2: 2.2uH, Inductor_SMD:L_1008_2520Metric, symbol Device:L
- removed Q1: DMG1012T, Package_TO_SOT_SMD:SOT-523, symbol Transistor_FET:DMG1012T
- removed R1, R2, R3, R4, R5, R9: 15K 1%, Resistor_SMD:R_0402_1005Metric, symbol Device:R
- removed R6: 120K 1%, Resistor_SMD:R_0402_1005Metric, symbol Device:R
- removed R7: 160K, Resistor_SMD:R_0402_1005Metric, symbol Device:R
- removed R8: 6.04K, Resistor_SMD:R_0402_1005Metric, symbol Device:R
- removed U3: VL805, Package_DFN_QFN:QFN-68-1EP_8x8mm_P0.4mm_EP5.2x5.2mm_ThermalVias, symbol CM4:VL805
- removed U4: AP22653W6, Package_TO_SOT_SMD:SOT-23-6, symbol CM4IO:AP2553W6
- removed U8: AP3402, Package_TO_SOT_SMD:TSOT-23-6, symbol Regulator_Switching:AP3402
- removed Y1: 25MHz, Crystal:Crystal_SMD_SeikoEpson_FA238-4Pin_3.2x2.5mm, symbol Device:Crystal_GND24_Small
Connections:
- no-connect marks 19 -> 0
Other:
- note removed: "CLK PN swap to help routing"
- note removed: "Current Limit switch"
- note removed: "EN pin <0.4v Ouput off EN pin >1.5v Output on."
- note removed: "Make sure the power switch is disabled during power up"
- note removed: "Potential divider sets 1.05v to start when 3.3v rail is somewhere between 0.8v and 3v"
- note removed: "Stacked USB connectors"
- note removed: "TX2 RX2 P/N swapped to help routing"
