File: audio/POWER_sch.kicad_sch (KiCad schematic)
At the start: 5 parts, among them J5 1054500101

Commit message: .
.
Parts:
- gave numbers to parts that had none: 4
Changed lines of the file:
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@@
   (symbol (lib_id "Device:R") (at 134.62 85.09 0) (unit 1)
     (in_bom yes) (on_board yes)
-    (property "Reference" "R?" (id 0) (at 136.398 83.9216 0)
+    (property "Reference" "R20" (id 0) (at 136.398 83.9216 0)
       (effects (font (size 1.27 1.27)) (justify left))
     )
@@
   (symbol (lib_id "Device:R") (at 148.59 73.66 0) (unit 1)
     (in_bom yes) (on_board yes)
-    (property "Reference" "R?" (id 0) (at 150.368 72.4916 0)
+    (property "Reference" "R21" (id 0) (at 150.368 72.4916 0)
       (effects (font (size 1.27 1.27)) (justify left))
     )
@@
   (symbol (lib_id "Device:R") (at 134.62 73.66 0) (unit 1)
     (in_bom yes) (on_board yes)
-    (property "Reference" "R?" (id 0) (at 136.398 72.4916 0)
+    (property "Reference" "R19" (id 0) (at 136.398 72.4916 0)
       (effects (font (size 1.27 1.27)) (justify left))
     )
@@
   (symbol (lib_id "Device:R") (at 148.59 85.09 0) (unit 1)
     (in_bom yes) (on_board yes)
-    (property "Reference" "R?" (id 0) (at 150.368 83.9216 0)
+    (property "Reference" "R22" (id 0) (at 150.368 83.9216 0)
       (effects (font (size 1.27 1.27)) (justify left))
     )

Commit message: .
.
Parts:
- added C73: 100uF, Capacitor_Tantalum_SMD:CP_EIA-3528-21_Kemet-B, symbol Device:CP
Connections:
- net 5V: now also C73.1
- net GND: now also C73.2
Changed lines of the file:
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@@
   (junction (at 134.62 78.74) (diameter 0) (color 0 0 0 0)
   )
+  (wire (pts (xy 182.88 66.04) (xy 182.88 55.88))
+    (stroke (width 0) (type default) (color 0 0 0 0))
+  )
   (wire (pts (xy 35.56 100.33) (xy 50.8 100.33))
     (stroke (width 0) (type default) (color 0 0 0 0))
@@
     (stroke (width 0) (type default) (color 0 0 0 0))
   )
+  (wire (pts (xy 182.88 81.28) (xy 193.04 81.28))
+    (stroke (width 0) (type default) (color 0 0 0 0))
+  )
   (wire (pts (xy 50.8 100.33) (xy 50.8 102.87))
     (stroke (width 0) (type default) (color 0 0 0 0))
@@
     (stroke (width 0) (type default) (color 0 0 0 0))
   )
+  (wire (pts (xy 182.88 55.88) (xy 193.04 55.88))
+    (stroke (width 0) (type default) (color 0 0 0 0))
+  )
   (wire (pts (xy 41.91 72.39) (xy 50.8 72.39))
     (stroke (width 0) (type default) (color 0 0 0 0))
@@
     (stroke (width 0) (type default) (color 0 0 0 0))
   )
+  (wire (pts (xy 182.88 73.66) (xy 182.88 81.28))
+    (stroke (width 0) (type default) (color 0 0 0 0))
+  )
   (wire (pts (xy 134.62 77.47) (xy 134.62 78.74))
     (stroke (width 0) (type default) (color 0 0 0 0))
@@
     (effects (font (size 1.27 1.27)) (justify left bottom))
   )
+  (label "GND" (at 185.42 81.28 0)
+    (effects (font (size 1.27 1.27)) (justify left bottom))
+  )
   (label "5V" (at 45.72 58.42 0)
     (effects (font (size 1.27 1.27)) (justify left bottom))
@@
   )
   (label "GND" (at 41.91 100.33 0)
+    (effects (font (size 1.27 1.27)) (justify left bottom))
+  )
+  (label "5V" (at 185.42 55.88 0)
     (effects (font (size 1.27 1.27)) (justify left bottom))
   )
@@
       (effects (font (size 1.27 1.27)) hide)
     )
+    (pin "1")
+    (pin "2")
+  )
+  (symbol (lib_id "Device:CP") (at 182.88 69.85 0) (unit 1)
+    (in_bom yes) (on_board yes)
+    (property "Reference" "C73" (id 0) (at 185.8772 68.707 0)
+      (effects (font (size 1.27 1.27)) (justify left))
+    )
+    (property "Value" "100uF" (id 1) (at 185.8772 70.993 0)
+      (effects (font (size 1.27 1.27)) (justify left))
+    )
+    (property "Footprint" "Capacitor_Tantalum_SMD:CP_EIA-3528-21_Kemet-B" (id 2) (at 183.8452 73.66 0)
+      (effects (font (size 1.27 1.27)) hide)
+    )
+    (property "Datasheet" "~" (id 3) (at 182.88 69.85 0)
+      (effects (font (size 1.27 1.27)) hide)
+    )
+    (property "Field4" "Mouser" (id 4) (at 182.88 69.85 0)
+      (effects (font (size 1.27 1.27)) hide)
+    )
+    (property "Field5" "667-EEF-CX0J101R" (id 5) (at 182.88 69.85 0)
+      (effects (font (size 1.27 1.27)) hide)
+    )
+    (property "Part Description" "Capacitor, SP-Cap, 100u, 6.3V, 15mR ESR" (id 6) (at 182.88 69.85 0)
+      (effects (font (size 1.27 1.27)) hide)
+    )

Commit message: .
.
Parts:
- added R3, R4: 2.2K 1%, Resistor_SMD:R_0402_1005Metric, symbol Device:R
- added U3: TPD4EUSB30, Package_SON:USON-10_2.5x1.0mm_P0.5mm, symbol CM4IO:TPD4EUSB30
Connections:
- net 5V: now also R4.1
- net GND: now also R3.1, U3.3 (GND), U3.8 (GND)
- net USB2_P: now reaches J5.A6 (D1+)
- net USB2_P: now also U3.1 (D1+), U3.10
- net USB2_N: now reaches J5.A7 (D1-)
- net USB2_N: now also U3.2 (D1-), U3.9
- new net: U3.4 (D2+), U3.7
- new net: U3.5 (D2-), U3.6
- new net USBOTG: R3.2, R4.2
