File: audio/POWER_sch.kicad_sch (KiCad schematic)
At the start: 9 parts, among them J5 1054500101, U3 TPD4EUSB30

Commit message: .
.
Connections:
- net USB2_N: now also J5.B7 (D2-)
- net USB2_P: now also J5.B6 (D2+)
Changed lines of the file:
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@@
+    (stroke (width 0) (type default))
+  )
+  (wire (pts (xy 95.25 74.93) (xy 106.68 74.93))
+    (stroke (width 0) (type default))
+  )
+  (wire (pts (xy 95.25 77.47) (xy 106.68 77.47))
     (stroke (width 0) (type default))
   )
@@
     (effects (font (size 1.27 1.27)) (justify left bottom))
   )
+  (label "D+" (at 104.14 77.47 180) (fields_autoplaced)
+    (effects (font (size 1.27 1.27)) (justify right bottom))
+  )
   (label "CC2" (at 152.4 78.74 0) (fields_autoplaced)
     (effects (font (size 1.27 1.27)) (justify left bottom))
@@
   (label "5V" (at 96.5724 60.96 0) (fields_autoplaced)
     (effects (font (size 1.27 1.27)) (justify left bottom))
+  )
+  (label "D-" (at 104.14 74.93 180) (fields_autoplaced)
+    (effects (font (size 1.27 1.27)) (justify right bottom))
   )
   (label "5V" (at 118.11 130.81 0) (fields_autoplaced)
@@
     (effects (font (size 1.27 1.27)) (justify right))
   )
+  (hierarchical_label "USB2_N" (shape output) (at 106.68 74.93 0) (fields_autoplaced)
+    (effects (font (size 1.27 1.27)) (justify left))
+  )
   (hierarchical_label "USBOTG" (shape output) (at 107.95 157.48 270) (fields_autoplaced)
     (effects (font (size 1.27 1.27)) (justify right))
@@
     (effects (font (size 1.27 1.27)) (justify left))
   )
+  (hierarchical_label "USB2_P" (shape output) (at 106.68 77.47 0) (fields_autoplaced)
+    (effects (font (size 1.27 1.27)) (justify left))
+  )

Commit message: .
.
Parts:
- R19, R20, R21, R22: value 5.1K 5% -> NC
- R3, R4: value 2.2K 1% -> NC
Changed lines of the file:
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@@
       (effects (font (size 1.27 1.27)) (justify left))
     )
-    (property "Value" "5.1K 5%" (at 136.398 86.233 0)
+    (property "Value" "NC" (at 136.398 86.233 0)
       (effects (font (size 1.27 1.27)) (justify left))
     )
@@
       (effects (font (size 1.27 1.27)) (justify left))
     )
-    (property "Value" "5.1K 5%" (at 150.368 74.803 0)
+    (property "Value" "NC" (at 150.368 74.803 0)
       (effects (font (size 1.27 1.27)) (justify left))
     )
@@
       (effects (font (size 1.27 1.27)) (justify left))
     )
-    (property "Value" "5.1K 5%" (at 136.398 74.803 0)
+    (property "Value" "NC" (at 136.398 74.803 0)
       (effects (font (size 1.27 1.27)) (justify left))
     )
@@
       (effects (font (size 1.27 1.27)) (justify left))
     )
-    (property "Value" "2.2K 1%" (at 104.648 144.653 0)
+    (property "Value" "NC" (at 104.648 144.653 0)
       (effects (font (size 1.27 1.27)) (justify left))
     )
@@
       (effects (font (size 1.27 1.27)) (justify left))
     )
-    (property "Value" "5.1K 5%" (at 150.368 86.233 0)
+    (property "Value" "NC" (at 150.368 86.233 0)
       (effects (font (size 1.27 1.27)) (justify left))
     )
@@
       (effects (font (size 1.27 1.27)) (justify left))
     )
-    (property "Value" "2.2K 1%" (at 117.348 144.653 0)
-      (effects (font (size 1.27 1.27)) (justify left))
-    )
+    (property "Value" "NC" (at 117.348 144.653 0)
+      (effects (font (size 1.27 1.27)) (justify left))
+    )

Commit message: USB_OK
.
Parts:
- R20, R22: value NC -> 5.1k
Changed lines of the file:
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@@
       (effects (font (size 1.27 1.27)) (justify left))
     )
-    (property "Value" "NC" (at 136.398 86.233 0)
+    (property "Value" "5.1k" (at 136.398 86.233 0)
       (effects (font (size 1.27 1.27)) (justify left))
     )
@@
       (effects (font (size 1.27 1.27)) (justify left))
     )
-    (property "Value" "NC" (at 150.368 86.233 0)
-      (effects (font (size 1.27 1.27)) (justify left))
-    )
+    (property "Value" "5.1k" (at 150.368 86.233 0)
+      (effects (font (size 1.27 1.27)) (justify left))
+    )
